File: JK330-1-BF/Filtre Passe Bas.sch (KiCad schematic (older format))
At the start: 32 parts, among them P7 CAVALIER, U1 MF10, U2 74HC4059, U3 74HC377, U4 74HC74, U5 OSC

Commit message: MAJ  composants
Parts:
- C7: value C -> 1U
- R14, R15, R16, R17, R18, R19, R20, R21: value R -> 10k
- U5: value OSC -> 16Mhz
Changed lines of the file:
@@
-EESchema Schematic File Version 2  date 2013-03-25 22:18:17
+EESchema Schematic File Version 2  date 29/04/2013 22:12:34
 LIBS:power
 LIBS:CEN-SCHEMA
@@
 Sheet 4 6
 Title "F4DEB"
-Date "25 mar 2013"
+Date "29 apr 2013"
 Rev "V 3.00"
 Comp "RACKANOUS"
@@
 U 1 1 4AA40E69
 P 9550 1100
-F 0 "C7" H 9600 1200 50  0000 L CNN
-F 1 "C" H 9600 1000 50  0000 L CNN
+F 0 "C7" V 9500 950 50  0000 L CNN
+F 1 "1U" V 9500 1200 50  0000 L CNN
 F 2 "" H 9550 1100 60  0001 C CNN
 F 3 "" H 9550 1100 60  0001 C CNN
@@
 U 1 1 4A9D825E
 P 8350 900
-F 0 "R6" V 8300 1000 50  0000 C CNN
-F 1 "10k" V 8400 1000 50  0000 C CNN
+F 0 "R6" V 8300 700 50  0000 C CNN
+F 1 "10k" V 8300 900 50  0000 C CNN
 F 2 "" H 8350 900 60  0001 C CNN
 F 3 "" H 8350 900 60  0001 C CNN
@@
 U 1 1 5150BF96
 P 6850 2150
-F 0 "C8" H 6900 2250 50  0000 L CNN
-F 1 "10U" H 6900 2050 50  0000 L CNN
+F 0 "C8" H 6650 2150 50  0000 L CNN
+F 1 "10U" H 6600 2050 50  0000 L CNN
 F 2 "" H 6850 2150 60  0001 C CNN
 F 3 "" H 6850 2150 60  0001 C CNN
@@
 U 1 1 5150BF90
 P 8900 1500
-F 0 "R12" V 8900 1700 50  0000 C CNN
+F 0 "R12" V 8850 1300 50  0000 C CNN
 F 1 "39k//39k" V 8950 1350 50  0000 C CNN
 F 2 "" H 8900 1500 60  0001 C CNN
@@
 U 1 1 5150BF8F
 P 8900 1400
-F 0 "R10" V 8900 1600 50  0000 C CNN
-F 1 "10k" V 8850 1300 50  0000 C CNN
+F 0 "R10" V 8850 1200 50  0000 C CNN
+F 1 "10k" V 8850 1400 50  0000 C CNN
 F 2 "" H 8900 1400 60  0001 C CNN
 F 3 "" H 8900 1400 60  0001 C CNN
@@
 U 1 1 5150BF8E
 P 8900 1300
-F 0 "R8" V 8900 1500 50  0000 C CNN
-F 1 "10k" V 8850 1200 50  0000 C CNN
+F 0 "R8" V 8850 1100 50  0000 C CNN
+F 1 "10k" V 8850 1300 50  0000 C CNN
 F 2 "" H 8900 1300 60  0001 C CNN
 F 3 "" H 8900 1300 60  0001 C CNN
@@
 U 1 1 5150BF8C
 P 7450 1400
-F 0 "R9" V 7450 1000 50  0000 C CNN
-F 1 "10k" V 7400 1300 50  0000 C CNN
+F 0 "R9" V 7400 1250 50  0000 C CNN
+F 1 "10k" V 7400 1400 50  0000 C CNN
 F 2 "" H 7450 1400 60  0001 C CNN
 F 3 "" H 7450 1400 60  0001 C CNN
@@
 U 1 1 5150BF8B
 P 7450 1500
-F 0 "R11" V 7450 1100 50  0000 C CNN
+F 0 "R11" V 7400 1350 50  0000 C CNN
 F 1 "39k//39k" V 7500 1450 50  0000 C CNN
 F 2 "" H 7450 1500 60  0001 C CNN
@@
 U 1 1 5150BF8A
 P 7450 1300
-F 0 "R7" V 7450 900 50  0000 C CNN
-F 1 "10k" V 7400 1200 50  0000 C CNN
+F 0 "R7" V 7400 1150 50  0000 C CNN
+F 1 "10k" V 7400 1300 50  0000 C CNN
 F 2 "" H 7450 1300 60  0001 C CNN
 F 3 "" H 7450 1300 60  0001 C CNN
@@
 P 4800 6250
 F 0 "U5" H 4700 6200 60  0000 C CNN
-F 1 "OSC" H 5050 6200 60  0000 C CNN
+F 1 "16Mhz" H 5050 6200 60  0000 C CNN
 F 2 "" H 4800 6250 60  0001 C CNN
 F 3 "" H 4800 6250 60  0001 C CNN
@@
 U 1 1 514F37D4
 P 3050 3950
-F 0 "R14" V 3000 4050 50  0000 C CNN
-F 1 "R" V 3100 4050 50  0000 C CNN
+F 0 "R14" V 3000 3800 50  0000 C CNN
+F 1 "10k" V 3000 4000 50  0000 C CNN
 F 2 "" H 3050 3950 60  0000 C CNN
 F 3 "" H 3050 3950 60  0000 C CNN
@@
 U 1 1 514F37ED
 P 3150 3950
-F 0 "R15" V 3100 4050 50  0000 C CNN
-F 1 "R" V 3200 4050 50  0000 C CNN
+F 0 "R15" V 3100 3800 50  0000 C CNN
+F 1 "10k" V 3100 4000 50  0000 C CNN
 F 2 "" H 3150 3950 60  0000 C CNN
 F 3 "" H 3150 3950 60  0000 C CNN
@@
 U 1 1 514F37FA
 P 3250 3950
-F 0 "R16" V 3200 4050 50  0000 C CNN
-F 1 "R" V 3300 4050 50  0000 C CNN
+F 0 "R16" V 3200 3800 50  0000 C CNN
+F 1 "10k" V 3200 4000 50  0000 C CNN
 F 2 "" H 3250 3950 60  0000 C CNN
 F 3 "" H 3250 3950 60  0000 C CNN
@@
 U 1 1 514F3800
 P 3350 3950
-F 0 "R17" V 3300 4050 50  0000 C CNN
-F 1 "R" V 3400 4050 50  0000 C CNN
+F 0 "R17" V 3300 3800 50  0000 C CNN
+F 1 "10k" V 3300 4000 50  0000 C CNN
 F 2 "" H 3350 3950 60  0000 C CNN
 F 3 "" H 3350 3950 60  0000 C CNN
@@
 U 1 1 514F3806
 P 3450 3950
-F 0 "R18" V 3400 4050 50  0000 C CNN
-F 1 "R" V 3500 4050 50  0000 C CNN
+F 0 "R18" V 3400 3800 50  0000 C CNN
+F 1 "10k" V 3400 4000 50  0000 C CNN
 F 2 "" H 3450 3950 60  0000 C CNN
 F 3 "" H 3450 3950 60  0000 C CNN
@@
 U 1 1 514F380C
 P 3550 3950
-F 0 "R19" V 3500 4050 50  0000 C CNN
-F 1 "R" V 3600 4050 50  0000 C CNN
+F 0 "R19" V 3500 3800 50  0000 C CNN
+F 1 "10k" V 3500 4000 50  0000 C CNN
 F 2 "" H 3550 3950 60  0000 C CNN
 F 3 "" H 3550 3950 60  0000 C CNN
@@
 U 1 1 514F3812
 P 3650 3950
-F 0 "R20" V 3600 4050 50  0000 C CNN
-F 1 "R" V 3700 4050 50  0000 C CNN
+F 0 "R20" V 3600 3800 50  0000 C CNN
+F 1 "10k" V 3600 4000 50  0000 C CNN
 F 2 "" H 3650 3950 60  0000 C CNN
 F 3 "" H 3650 3950 60  0000 C CNN
@@
 U 1 1 514F3818
 P 3750 3950
-F 0 "R21" V 3700 4050 50  0000 C CNN
-F 1 "R" V 3800 4050 50  0000 C CNN
+F 0 "R21" V 3700 3800 50  0000 C CNN
+F 1 "10k" V 3700 4000 50  0000 C CNN
 F 2 "" H 3750 3950 60  0000 C CNN
 F 3 "" H 3750 3950 60  0000 C CNN
@@
 	6650 650  8150 650
 Connection ~ 6650 1650
-Text Notes 8050 800  0    60   ~ 0
+Text Notes 8650 600  0    60   ~ 0
 NO FILTER\n
 $Comp

Commit message: Reste 2 pistes a router
Parts:
- C16: value C -> 100n
Connections:
- net labels removed: +5V
- wire segments 134 -> 135
Other:
- note removed: "U1"
- note removed: "U2"
- note removed: "U3"
- note removed: "U4"
- moved on the sheet: C16
Changed lines of the file:
@@
-EESchema Schematic File Version 2  date 09/06/2013 23:13:58
+EESchema Schematic File Version 2  date 11/06/2013 22:16:43
 LIBS:power
 LIBS:CEN-SCHEMA
@@
 Sheet 4 6
 Title "F4DEB"
-Date "9 jun 2013"
+Date "11 jun 2013"
 Rev "V 3.00"
 Comp "RACKANOUS"
@@
 	8550 1400 8650 1400
 Wire Wire Line
-	6750 1650 6550 1650
+	6550 1650 6750 1650
 Connection ~ 7150 1400
 Wire Wire Line
@@
 	4300 6750 4500 6750
 Wire Wire Line
-	5350 7100 5350 7150
+	5550 6500 5550 6550
 Wire Wire Line
 	5850 6750 5850 5100
@@
 Connection ~ 4650 4100
 Wire Wire Line
-	4750 4100 4650 4100
+	4650 4100 4750 4100
 Connection ~ 4650 3900
 Wire Wire Line
@@
 	4750 5200 4650 5200
 Wire Wire Line
-	4750 5000 2600 5000
-Wire Wire Line
-	4750 4800 2600 4800
-Wire Wire Line
-	4750 4600 2600 4600
-Wire Wire Line
-	4750 4400 2600 4400
+	2600 5000 4750 5000
+Wire Wire Line
+	2600 4800 4750 4800
+Wire Wire Line
+	2600 4600 4750 4600
+Wire Wire Line
+	2600 4400 4750 4400
 Wire Wire Line
 	2600 4300 4750 4300
@@
 	2150 5350 2150 5450
 Wire Wire Line
-	5350 6450 5350 6500
+	5350 6150 5350 6500
 Wire Wire Line
 	5350 6500 5250 6500
-Wire Wire Line
-	5350 6800 5350 6750
-Connection ~ 5350 6750
 Wire Wire Line
 	5250 6750 6150 6750
@@
 	0    1    1    0
 $EndComp
-Text Notes 4000 2700 0    60   ~ 0
-U4
-Text Notes 3650 2700 0    60   ~ 0
-U3
-Text Notes 3300 2700 0    60   ~ 0
-U2
-Text Notes 2950 2700 0    60   ~ 0
-U1
 Text Label 1450 4850 0    60   ~ 0
 D7
@@
 $EndComp
 $Comp
-L +5V #PWR039
-U 1 1 49948FF2
-P 6400 4650
-F 0 "#PWR039" H 6400 4740 20  0001 C CNN
-F 1 "+5V" H 6400 4740 30  0000 C CNN
-F 2 "" H 6400 4650 60  0001 C CNN
-F 3 "" H 6400 4650 60  0001 C CNN
-	1    6400 4650
-	0    -1   -1   0
-$EndComp
-$Comp
-L +5V #PWR040
-U 1 1 49948FF0
-P 6400 4300
-F 0 "#PWR040" H 6400 4390 20  0001 C CNN
-F 1 "+5V" H 6400 4390 30  0000 C CNN
-F 2 "" H 6400 4300 60  0001 C CNN
-F 3 "" H 6400 4300 60  0001 C CNN
-	1    6400 4300
-	0    -1   -1   0
-$EndComp
-$Comp
-L GND #PWR041
+L GND #PWR039
 U 1 1 49948FE7
 P 6950 5050
-F 0 "#PWR041" H 6950 5050 30  0001 C CNN
+F 0 "#PWR039" H 6950 5050 30  0001 C CNN
 F 1 "GND" H 6950 4980 30  0001 C CNN
 F 2 "" H 6950 5050 60  0001 C CNN
@@
 $EndComp
 $Comp
-L GND #PWR042
+L GND #PWR040
 U 1 1 49948ECF
-P 5350 7150
-F 0 "#PWR042" H 5350 7150 30  0001 C CNN
-F 1 "GND" H 5350 7080 30  0001 C CNN
-F 2 "" H 5350 7150 60  0001 C CNN
-F 3 "" H 5350 7150 60  0001 C CNN
-	1    5350 7150
-	1    0    0    -1
-$EndComp
-$Comp
-L GND #PWR043
+P 5550 6550
+F 0 "#PWR040" H 5550 6550 30  0001 C CNN
+F 1 "GND" H 5550 6480 30  0001 C CNN
+F 2 "" H 5550 6550 60  0001 C CNN
+F 3 "" H 5550 6550 60  0001 C CNN
+	1    5550 6550
+	1    0    0    -1
+$EndComp
+$Comp
+L GND #PWR041
 U 1 1 49948EB9
 P 4300 6750
-F 0 "#PWR043" H 4300 6750 30  0001 C CNN
+F 0 "#PWR041" H 4300 6750 30  0001 C CNN
 F 1 "GND" H 4300 6680 30  0001 C CNN
 F 2 "" H 4300 6750 60  0001 C CNN
@@
 $EndComp
 $Comp
-L GND #PWR044
+L GND #PWR042
 U 1 1 49948DAB
 P 2150 5450
-F 0 "#PWR044" H 2150 5450 30  0001 C CNN
+F 0 "#PWR042" H 2150 5450 30  0001 C CNN
 F 1 "GND" H 2150 5380 30  0001 C CNN
 F 2 "" H 2150 5450 60  0001 C CNN
@@
 $EndComp
 $Comp
-L GND #PWR045
+L GND #PWR043
 U 1 1 5150BF84
 P 1600 5150
-F 0 "#PWR045" H 1600 5150 30  0001 C CNN
+F 0 "#PWR043" H 1600 5150 30  0001 C CNN
 F 1 "GND" H 1600 5080 30  0001 C CNN
 F 2 "" H 1600 5150 60  0001 C CNN
@@
 	1250 4750 1350 4850
 $Comp
-L GND #PWR046
+L GND #PWR044
 U 1 1 5150BF83
 P 5350 3500
-F 0 "#PWR046" H 5350 3500 30  0001 C CNN
+F 0 "#PWR044" H 5350 3500 30  0001 C CNN
 F 1 "GND" H 5350 3430 30  0001 C CNN
 F 2 "" H 5350 3500 60  0001 C CNN
@@
 $EndComp
 $Comp
-L GND #PWR047
+L GND #PWR045
 U 1 1 5150BF82
 P 5900 4950
-F 0 "#PWR047" H 5900 4950 30  0001 C CNN
+F 0 "#PWR045" H 5900 4950 30  0001 C CNN
 F 1 "GND" H 5900 4880 30  0001 C CNN
 F 2 "" H 5900 4950 60  0001 C CNN
@@
 $EndComp
 $Comp
-L +5V #PWR048
-U 1 1 499351CC
-P 5250 5850
-F 0 "#PWR048" H 5250 5940 20  0001 C CNN
-F 1 "+5V" H 5250 5940 30  0000 C CNN
-F 2 "" H 5250 5850 60  0001 C CNN
-F 3 "" H 5250 5850 60  0001 C CNN
-	1    5250 5850
-	-1   0    0    1
-$EndComp
-$Comp
-L GND #PWR049
+L GND #PWR046
 U 1 1 499351AF
 P 4650 3700
-F 0 "#PWR049" H 4650 3700 30  0001 C CNN
+F 0 "#PWR046" H 4650 3700 30  0001 C CNN
 F 1 "GND" H 4650 3630 30  0001 C CNN
 F 2 "" H 4650 3700 60  0001 C CNN
@@
 $EndComp
 $Comp
-L GND #PWR050
+L GND #PWR047
 U 1 1 5150BF80
 P 4650 5550
-F 0 "#PWR050" H 4650 5550 30  0001 C CNN
+F 0 "#PWR047" H 4650 5550 30  0001 C CNN
 F 1 "GND" H 4650 5480 30  0001 C CNN
 F 2 "" H 4650 5550 60  0001 C CNN
@@
 L C C16
 U 1 1 49934E07
-P 5350 6950
-F 0 "C16" H 5400 7050 50  0000 L CNN
-F 1 "C" H 5400 6850 50  0000 L CNN
-F 2 "" H 5350 6950 60  0001 C CNN
-F 3 "" H 5350 6950 60  0001 C CNN
-	1    5350 6950
+P 5550 6350
+F 0 "C16" H 5600 6450 50  0000 L CNN
+F 1 "100n" H 5600 6250 50  0000 L CNN
+F 2 "" H 5550 6350 60  0001 C CNN
+F 3 "" H 5550 6350 60  0001 C CNN
+	1    5550 6350
 	-1   0    0    1
 $EndComp
@@
 F 3 "" H 3450 2800 60  0001 C CNN
 	1    3450 2800
-	1    0    0    -1
-$EndComp
-$Comp
-L C C12
-U 1 1 5150BF7B
-P 3100 2800
-F 0 "C12" H 3150 2900 50  0000 L CNN
-F 1 "100n" H 3150 2700 50  0000 L CNN
-F 2 "" H 3100 2800 60  0001 C CNN
-F 3 "" H 3100 2800 60  0001 C CNN
-	1    3100 2800
 	1    0    0    -1
 $EndComp
@@
 	3050 3900 3050 3750
 Wire Wire Line
-	3750 3900 3750 3750
-Wire Wire Line
-	3750 3750 3050 3750
+	3750 3750 3750 3900
+Wire Wire Line
+	3050 3750 3750 3750
 Wire Wire Line
 	3150 3900 3150 3750
@@
 NO FILTER\n
 $Comp
-L +5VA #PWR051
+L +5VA #PWR048
 U 1 1 514F8423
 P 6700 2000
-F 0 "#PWR051" H 6700 2130 20  0001 C CNN
+F 0 "#PWR048" H 6700 2130 20  0001 C CNN
 F 1 "+5VA" H 6700 2100 30  0000 C CNN
 F 2 "" H 6700 2000 60  0000 C CNN
@@
 $EndComp
 $Comp
-L +5VD #PWR052
+L +5VD #PWR049
 U 1 1 514F8648
 P 2150 3800
-F 0 "#PWR052" H 2150 3750 20  0001 C CNN
+F 0 "#PWR049" H 2150 3750 20  0001 C CNN
 F 1 "+5VD" H 2150 3900 30  0000 C CNN
 F 2 "" H 2150 3800 60  0000 C CNN
@@
 $EndComp
 $Comp
-L +5VD #PWR053
+L +5VD #PWR050
 U 1 1 514F8657
 P 3350 3650
-F 0 "#PWR053" H 3350 3600 20  0001 C CNN
+F 0 "#PWR050" H 3350 3600 20  0001 C CNN
 F 1 "+5VD" H 3350 3750 30  0000 C CNN
 F 2 "" H 3350 3650 60  0000 C CNN
@@
 $EndComp
 $Comp
-L +5VD #PWR054
+L +5VD #PWR051
 U 1 1 514F8666
 P 5150 3500
-F 0 "#PWR054" H 5150 3450 20  0001 C CNN
+F 0 "#PWR051" H 5150 3450 20  0001 C CNN
 F 1 "+5VD" H 5150 3600 30  0000 C CNN
 F 2 "" H 5150 3500 60  0000 C CNN
@@
 $EndComp
 $Comp
-L +5VD #PWR055
+L +5VD #PWR052
 U 1 1 514F8675
 P 6950 3900
-F 0 "#PWR055" H 6950 3850 20  0001 C CNN
+F 0 "#PWR052" H 6950 3850 20  0001 C CNN
 F 1 "+5VD" H 6950 4000 30  0000 C CNN
 F 2 "" H 6950 3900 60  0000 C CNN
@@
 $EndComp
 $Comp
-L +5VD #PWR056
+L +5VD #PWR053
 U 1 1 514F8686
 P 3450 2500
-F 0 "#PWR056" H 3450 2450 20  0001 C CNN
+F 0 "#PWR053" H 3450 2450 20  0001 C CNN
 F 1 "+5VD" H 3450 2600 30  0000 C CNN
 F 2 "" H 3450 2500 60  0000 C CNN
@@
 $EndComp
 $Comp
+L +5VD #PWR054
+U 1 1 514F8695
+P 5550 6100
+F 0 "#PWR054" H 5550 6050 20  0001 C CNN
+F 1 "+5VD" H 5550 6200 30  0000 C CNN
+F 2 "" H 5550 6100 60  0000 C CNN
+F 3 "" H 5550 6100 60  0000 C CNN
+	1    5550 6100
+	1    0    0    -1
+$EndComp
+Wire Wire Line
+	5350 6150 5550 6150
+Wire Wire Line
+	5550 6100 5550 6200
+Connection ~ 5550 6150
+$Comp
+L C C12
+U 1 1 5150BF7B
+P 3100 2800
+F 0 "C12" H 3150 2900 50  0000 L CNN
+F 1 "100n" H 3150 2700 50  0000 L CNN
+F 2 "" H 3100 2800 60  0001 C CNN
+F 3 "" H 3100 2800 60  0001 C CNN
+	1    3100 2800
+	1    0    0    -1
+$EndComp
+$Comp
+L +5VD #PWR055
+U 1 1 51B78931
+P 5250 5850
+F 0 "#PWR055" H 5250 5800 20  0001 C CNN
+F 1 "+5VD" H 5250 5950 30  0000 C CNN
+F 2 "" H 5250 5850 60  0000 C CNN
+F 3 "" H 5250 5850 60  0000 C CNN
+	1    5250 5850
+	-1   0    0    1
+$EndComp
+$Comp
+L +5VD #PWR056
+U 1 1 51B78B9B
+P 6400 4300
+F 0 "#PWR056" H 6400 4250 20  0001 C CNN
+F 1 "+5VD" H 6400 4400 30  0000 C CNN
+F 2 "" H 6400 4300 60  0000 C CNN
+F 3 "" H 6400 4300 60  0000 C CNN
+	1    6400 4300
+	0    -1   -1   0
+$EndComp
+$Comp
 L +5VD #PWR057
-U 1 1 514F8695
-P 5350 6450
-F 0 "#PWR057" H 5350 6400 20  0001 C CNN
-F 1 "+5VD" H 5350 6550 30  0000 C CNN
-F 2 "" H 5350 6450 60  0000 C CNN
-F 3 "" H 5350 6450 60  0000 C CNN
-	1    5350 6450
-	1    0    0    -1
+U 1 1 51B78BAA
+P 6400 4650
+F 0 "#PWR057" H 6400 4600 20  0001 C CNN
+F 1 "+5VD" H 6400 4750 30  0000 C CNN
+F 2 "" H 6400 4650 60  0000 C CNN
+F 3 "" H 6400 4650 60  0000 C CNN
+	1    6400 4650
+	0    -1   -1   0
 $EndComp
 $EndSCHEMATC
