File: JK330-1-BF/Filtre Passe Bas.sch (KiCad schematic (older format))
At the start: 32 parts, among them P7 CAVALIER, U1 MF10, U2 74HC4059, U3 74HC377, U4 74HC74, U5 16Mhz

Commit message: Ajout carte power
Parts:
- C13, C15: value C -> 100n
- C7: value 1U -> 10U
Changed lines of the file:
@@
 Sheet 4 6
 Title "JK330 "
-Date "18 jun 2013"
+Date "18 jul 2013"
 Rev "V0.10"
 Comp "F4DEB 2013"
@@
 P 9550 1100
 F 0 "C7" V 9500 950 50  0000 L CNN
-F 1 "1U" V 9500 1200 50  0000 L CNN
+F 1 "10U" V 9500 1200 50  0000 L CNN
 F 2 "" H 9550 1100 60  0001 C CNN
 F 3 "" H 9550 1100 60  0001 C CNN
@@
 P 4150 2800
 F 0 "C15" H 4200 2900 50  0000 L CNN
-F 1 "C" H 4200 2700 50  0000 L CNN
+F 1 "100n" H 4200 2700 50  0000 L CNN
 F 2 "" H 4150 2800 60  0001 C CNN
 F 3 "" H 4150 2800 60  0001 C CNN
@@
 P 3450 2800
 F 0 "C13" H 3500 2900 50  0000 L CNN
-F 1 "C" H 3500 2700 50  0000 L CNN
+F 1 "100n" H 3500 2700 50  0000 L CNN
 F 2 "" H 3450 2800 60  0001 C CNN
 F 3 "" H 3450 2800 60  0001 C CNN
