File: JK330-1-BF/HP.sch (KiCad schematic (older format))
At the start: 14 parts, among them U10 TDA2003

Commit message: MAJ  composants
Changed lines of the file:
@@
-EESchema Schematic File Version 2  date 2013-03-25 22:18:17
+EESchema Schematic File Version 2  date 29/04/2013 22:12:34
 LIBS:power
 LIBS:CEN-SCHEMA
@@
 Sheet 6 6
 Title "F4DEB"
-Date "25 mar 2013"
+Date "29 apr 2013"
 Rev "V 3.00"
 Comp "RACKANOUS"
@@
 U 1 1 49949B00
 P 7150 4200
-F 0 "R45" V 7100 4300 50  0000 C CNN
-F 1 "1" V 7200 4300 50  0000 C CNN
+F 0 "R45" V 7100 4050 50  0000 C CNN
+F 1 "1" V 7100 4250 50  0000 C CNN
 F 2 "" H 7150 4200 60  0001 C CNN
 F 3 "" H 7150 4200 60  0001 C CNN
@@
 U 1 1 49949ADD
 P 5750 4600
-F 0 "C32" H 5800 4700 50  0000 L CNN
-F 1 "NC" H 5800 4500 50  0000 L CNN
+F 0 "C32" V 5700 4400 50  0000 L CNN
+F 1 "NC" V 5700 4650 50  0000 L CNN
 F 2 "" H 5750 4600 60  0001 C CNN
 F 3 "" H 5750 4600 60  0001 C CNN
@@
 U 1 1 49949AD8
 P 6350 4600
-F 0 "R48" V 6300 4700 50  0000 C CNN
-F 1 "NC" V 6400 4700 50  0000 C CNN
+F 0 "R48" V 6300 4400 50  0000 C CNN
+F 1 "NC" V 6300 4600 50  0000 C CNN
 F 2 "" H 6350 4600 60  0001 C CNN
 F 3 "" H 6350 4600 60  0001 C CNN
@@
 U 1 1 49949AC5
 P 6350 4300
-F 0 "R47" V 6300 4400 50  0000 C CNN
-F 1 "470" V 6400 4400 50  0000 C CNN
+F 0 "R47" V 6300 4100 50  0000 C CNN
+F 1 "470" V 6300 4300 50  0000 C CNN
 F 2 "" H 6350 4300 60  0001 C CNN
 F 3 "" H 6350 4300 60  0001 C CNN
@@
 U 1 1 49949AC0
 P 5850 4300
-F 0 "R46" V 5800 4400 50  0000 C CNN
-F 1 "10" V 5900 4400 50  0000 C CNN
+F 0 "R46" V 5800 4150 50  0000 C CNN
+F 1 "10" V 5800 4300 50  0000 C CNN
 F 2 "" H 5850 4300 60  0001 C CNN
 F 3 "" H 5850 4300 60  0001 C CNN
@@
 U 1 1 49949AB6
 P 6350 3650
-F 0 "U10" H 6450 3900 60  0000 L CNN
-F 1 "TDA2003" H 6450 3500 60  0000 L CNN
+F 0 "U10" H 6150 3950 60  0000 L CNN
+F 1 "TDA2003" H 6450 3950 60  0000 L CNN
 F 2 "" H 6350 3650 60  0001 C CNN
 F 3 "" H 6350 3650 60  0001 C CNN
@@
 U 1 1 499499EB
 P 6550 2500
-F 0 "C25" H 6600 2600 50  0000 L CNN
-F 1 "1000U" H 6600 2400 50  0000 L CNN
+F 0 "C25" V 6700 2550 50  0000 L CNN
+F 1 "1000U" V 6650 2200 50  0000 L CNN
 F 2 "" H 6550 2500 60  0001 C CNN
 F 3 "" H 6550 2500 60  0001 C CNN
@@
 U 1 1 499499E8
 P 6550 2850
-F 0 "C26" H 6600 2950 50  0000 L CNN
-F 1 "100n" H 6600 2750 50  0000 L CNN
+F 0 "C26" V 6500 2650 50  0000 L CNN
+F 1 "100n" V 6500 2900 50  0000 L CNN
 F 2 "" H 6550 2850 60  0001 C CNN
 F 3 "" H 6550 2850 60  0001 C CNN
@@
 U 1 1 499499E2
 P 6000 4050
-F 0 "C31" H 6050 4150 50  0000 L CNN
-F 1 "100U" H 6050 3950 50  0000 L CNN
+F 0 "C31" H 6050 3950 50  0000 L CNN
+F 1 "100U" H 5750 3950 50  0000 L CNN
 F 2 "" H 6000 4050 60  0001 C CNN
 F 3 "" H 6000 4050 60  0001 C CNN
@@
 U 1 1 499499D2
 P 4900 3550
-F 0 "C28" H 4950 3650 50  0000 L CNN
-F 1 "15n" H 4950 3450 50  0000 L CNN
+F 0 "C28" V 4950 3650 50  0000 L CNN
+F 1 "15n" V 4950 3350 50  0000 L CNN
 F 2 "" H 4900 3550 60  0001 C CNN
 F 3 "" H 4900 3550 60  0001 C CNN
@@
 U 1 1 514F756F
 P 4050 3700
-F 0 "RVAR2" V 4000 3800 50  0000 C CNN
-F 1 "RVAR" V 4100 3800 50  0000 C CNN
+F 0 "RVAR2" V 3950 3700 50  0000 C CNN
+F 1 "RVAR" V 4150 3600 50  0000 C CNN
 F 2 "" H 4050 3700 60  0000 C CNN
 F 3 "" H 4050 3700 60  0000 C CNN

Commit message: Routage  PCB
Parts:
- removed RVAR2: RVAR, symbol RVAR
Connections:
- net BFIN: now reaches C28.1
Changed lines of the file:
@@
-EESchema Schematic File Version 2  date 04/06/2013 21:43:31
+EESchema Schematic File Version 2  date 09/06/2013 23:13:58
 LIBS:power
 LIBS:CEN-SCHEMA
@@
 Sheet 6 6
 Title "F4DEB"
-Date "4 jun 2013"
+Date "9 jun 2013"
 Rev "V 3.00"
 Comp "RACKANOUS"
@@
 HP1
 $Comp
-L GND #PWR081
+L GND #PWR083
 U 1 1 49AAEFDB
 P 6350 3900
-F 0 "#PWR081" H 6350 3900 30  0001 C CNN
+F 0 "#PWR083" H 6350 3900 30  0001 C CNN
 F 1 "GND" H 6350 3830 30  0001 C CNN
 F 2 "" H 6350 3900 60  0001 C CNN
@@
 $EndComp
 $Comp
-L +12V #PWR082
+L +12V #PWR084
 U 1 1 49949CCF
 P 6350 2150
-F 0 "#PWR082" H 6350 2100 20  0001 C CNN
+F 0 "#PWR084" H 6350 2100 20  0001 C CNN
 F 1 "+12V" H 6350 2250 30  0000 C CNN
 F 2 "" H 6350 2150 60  0001 C CNN
@@
 $EndComp
 $Comp
-L GND #PWR083
+L GND #PWR085
 U 1 1 49949B5F
 P 7150 4550
-F 0 "#PWR083" H 7150 4550 30  0001 C CNN
+F 0 "#PWR085" H 7150 4550 30  0001 C CNN
 F 1 "GND" H 7150 4480 30  0001 C CNN
 F 2 "" H 7150 4550 60  0001 C CNN
@@
 $EndComp
 $Comp
-L GND #PWR084
+L GND #PWR086
 U 1 1 49949B5C
 P 6950 2850
-F 0 "#PWR084" H 6950 2850 30  0001 C CNN
+F 0 "#PWR086" H 6950 2850 30  0001 C CNN
 F 1 "GND" H 6950 2780 30  0001 C CNN
 F 2 "" H 6950 2850 60  0001 C CNN
@@
 $EndComp
 $Comp
-L GND #PWR085
+L GND #PWR087
 U 1 1 49949B58
 P 6950 2500
-F 0 "#PWR085" H 6950 2500 30  0001 C CNN
+F 0 "#PWR087" H 6950 2500 30  0001 C CNN
 F 1 "GND" H 6950 2430 30  0001 C CNN
 F 2 "" H 6950 2500 60  0001 C CNN
@@
 $EndComp
 $Comp
-L GND #PWR086
+L GND #PWR088
 U 1 1 49949B51
 P 5750 3100
-F 0 "#PWR086" H 5750 3100 30  0001 C CNN
+F 0 "#PWR088" H 5750 3100 30  0001 C CNN
 F 1 "GND" H 5750 3030 30  0001 C CNN
 F 2 "" H 5750 3100 60  0001 C CNN
@@
 $EndComp
 $Comp
-L GND #PWR087
+L GND #PWR089
 U 1 1 49949B48
 P 5500 4300
-F 0 "#PWR087" H 5500 4300 30  0001 C CNN
+F 0 "#PWR089" H 5500 4300 30  0001 C CNN
 F 1 "GND" H 5500 4230 30  0001 C CNN
 F 2 "" H 5500 4300 60  0001 C CNN
@@
 Wire Wire Line
 	4800 3550 4150 3550
-Text HLabel 3850 3400 0    60   Input ~ 0
-AFRN
-$Comp
-L RVAR RVAR2
-U 1 1 514F756F
-P 4050 3700
-F 0 "RVAR2" V 3950 3700 50  0000 C CNN
-F 1 "RVAR" V 4150 3600 50  0000 C CNN
-F 2 "" H 4050 3700 60  0000 C CNN
-F 3 "" H 4050 3700 60  0000 C CNN
-	1    4050 3700
-	-1   0    0    1
-$EndComp
-Wire Wire Line
-	3850 3400 4050 3400
-Wire Wire Line
-	4050 3400 4050 3450
-Wire Wire Line
-	4050 3750 4050 3850
-$Comp
-L GND #PWR088
-U 1 1 514F75CD
-P 4050 3850
-F 0 "#PWR088" H 4050 3850 30  0001 C CNN
-F 1 "GND" H 4050 3780 30  0001 C CNN
-F 2 "" H 4050 3850 60  0000 C CNN
-F 3 "" H 4050 3850 60  0000 C CNN
-	1    4050 3850
-	1    0    0    -1
-$EndComp
+Text HLabel 4150 3550 0    60   Input ~ 0
+BFIN
 Wire Wire Line
 	7450 3650 7450 3950

Commit message: Fin Routage PCb V0-10
Parts:
- removed C31: 100U, symbol C
- added C31: 100u, symbol CP
Connections:
- net at R46.1, R47.2: now also C31.1
- net at U10.2 (-): now also C31.2
Changed lines of the file:
@@
-EESchema Schematic File Version 2  date 16/06/2013 19:24:33
+EESchema Schematic File Version 2
 LIBS:power
 LIBS:CEN-SCHEMA
@@
 encoding utf-8
 Sheet 6 6
-Title "F4DEB"
-Date "16 jun 2013"
-Rev "V 3.00"
-Comp "RACKANOUS"
-Comment1 "Carte  Audio"
+Title "JK330 "
+Date "18 jun 2013"
+Rev "V0.10"
+Comp "F4DEB 2013"
+Comment1 "CARTE FI 9Mhz FILTRE BF"
 Comment2 "AMPLIFICATEUR AUDIO"
 Comment3 ""
@@
 	6050 3750 6000 3750
 Wire Wire Line
-	6000 3750 6000 3900
-Wire Wire Line
-	6000 4200 6000 4300
+	6000 3750 6000 3950
+Wire Wire Line
+	6000 4150 6000 4300
 Connection ~ 6000 4300
 Wire Wire Line
@@
 $EndComp
 $Comp
-L C C31
-U 1 1 499499E2
-P 6000 4050
-F 0 "C31" H 6050 3950 50  0000 L CNN
-F 1 "100U" H 5750 3950 50  0000 L CNN
-F 2 "" H 6000 4050 60  0001 C CNN
-F 3 "" H 6000 4050 60  0001 C CNN
-	1    6000 4050
-	-1   0    0    1
-$EndComp
-$Comp
 L CP C28
 U 1 1 499499D2
@@
 Text HLabel 7600 3950 2    60   Input ~ 0
 HP2
+$Comp
+L CP C31
+U 1 1 51C0C83B
+P 6000 4050
+F 0 "C31" H 6050 4150 50  0000 L CNN
+F 1 "100u" H 6050 3950 50  0000 L CNN
+F 2 "" H 6000 4050 60  0000 C CNN
+F 3 "" H 6000 4050 60  0000 C CNN
+	1    6000 4050
+	-1   0    0    1
+$EndComp
 $EndSCHEMATC
