File: JK330-1-BF/HP.sch (KiCad schematic (older format))
At the start: 13 parts, among them U10 TDA2003

Commit message: Ajout carte power
Parts:
- C28: value 15n -> 47U
Changed lines of the file:
@@
 Sheet 6 6
 Title "JK330 "
-Date "18 jun 2013"
+Date "18 jul 2013"
 Rev "V0.10"
 Comp "F4DEB 2013"
@@
 P 4900 3550
 F 0 "C28" V 4950 3650 50  0000 L CNN
-F 1 "15n" V 4950 3350 50  0000 L CNN
+F 1 "47U" V 4950 3350 50  0000 L CNN
 F 2 "" H 4900 3550 60  0001 C CNN
 F 3 "" H 4900 3550 60  0001 C CNN
