File: JK330-1-BF/MIC.sch (KiCad schematic (older format))
At the start: 4 parts, among them Q1 BSS123

Commit message: Rajout commande PTT
+12VTV
+12VRX
Parts:
- removed Q1: BSS123, symbol BSS123
- removed R5: R, symbol R
- added C? (x3): CP, symbol CP
- added Q? (x3): BC847, symbol BC847
- added Q? (x2): BSP250, symbol BSP250
- added R? (x7): R, symbol R
Connections:
- net labels added: +12VRX, +12VTX, +5V
- wire segments 8 -> 37
Other:
- moved on the sheet: C6, R4

Commit message: maj EMPREINTE
Parts:
- gave numbers to parts that had none: 15
Changed lines of the file:
@@
-EESchema Schematic File Version 2  date 30/04/2013 22:23:42
+EESchema Schematic File Version 2  date 20/05/2013 22:53:17
 LIBS:power
 LIBS:CEN-SCHEMA
@@
 Sheet 3 6
 Title ""
-Date "30 apr 2013"
+Date "20 may 2013"
 Rev ""
 Comp ""
@@
 	3100 3600 3100 3450
 $Comp
-L +12V #PWR020
+L +12V #PWR018
 U 1 1 514F9C6A
 P 3100 3450
-F 0 "#PWR020" H 3100 3400 20  0001 C CNN
+F 0 "#PWR018" H 3100 3400 20  0001 C CNN
 F 1 "+12V" H 3100 3550 30  0000 C CNN
 F 2 "" H 3100 3450 60  0000 C CNN
@@
 AFE
 $Comp
-L BC847 Q?
+L BC847 Q1
 U 1 1 518025F5
 P 6400 4850
-F 0 "Q?" H 6550 4850 50  0000 C CNN
+F 0 "Q1" H 6550 4850 50  0000 C CNN
 F 1 "BC847" H 6200 4950 50  0000 C CNN
 F 2 "" H 6400 4850 60  0000 C CNN
@@
 $EndComp
 $Comp
-L R R?
+L R R5
 U 1 1 51802604
 P 6100 4550
-F 0 "R?" V 6050 4650 50  0000 C CNN
+F 0 "R5" V 6050 4650 50  0000 C CNN
 F 1 "R" V 6150 4650 50  0000 C CNN
 F 2 "" H 6100 4550 60  0000 C CNN
@@
 	6500 5050 6500 5100
 $Comp
-L GND #PWR?
+L GND #PWR019
 U 1 1 5180264F
 P 6500 5100
-F 0 "#PWR?" H 6500 5100 30  0001 C CNN
+F 0 "#PWR019" H 6500 5100 30  0001 C CNN
 F 1 "GND" H 6500 5030 30  0001 C CNN
 F 2 "" H 6500 5100 60  0000 C CNN
@@
 $EndComp
 $Comp
-L +5V #PWR?
+L +5V #PWR020
 U 1 1 5180265E
 P 6100 4400
-F 0 "#PWR?" H 6100 4490 20  0001 C CNN
+F 0 "#PWR020" H 6100 4490 20  0001 C CNN
 F 1 "+5V" H 6100 4490 30  0000 C CNN
 F 2 "" H 6100 4400 60  0000 C CNN
@@
 	6500 4550 6500 4650
 $Comp
-L R R?
+L R R49
 U 1 1 5180267F
 P 6500 4300
-F 0 "R?" V 6450 4400 50  0000 C CNN
+F 0 "R49" V 6450 4400 50  0000 C CNN
 F 1 "R" V 6550 4400 50  0000 C CNN
 F 2 "" H 6500 4300 60  0000 C CNN
@@
 Connection ~ 6500 4600
 $Comp
-L BC847 Q?
+L BC847 Q2
 U 1 1 518026E8
 P 7400 4600
-F 0 "Q?" H 7550 4600 50  0000 C CNN
+F 0 "Q2" H 7550 4600 50  0000 C CNN
 F 1 "BC847" H 7200 4700 50  0000 C CNN
 F 2 "" H 7400 4600 60  0000 C CNN
@@
 $EndComp
 $Comp
-L R R?
+L R R51
 U 1 1 5180275B
 P 7100 4750
-F 0 "R?" V 7050 4850 50  0000 C CNN
+F 0 "R51" V 7050 4850 50  0000 C CNN
 F 1 "R" V 7150 4850 50  0000 C CNN
 F 2 "" H 7100 4750 60  0000 C CNN
@@
 	7500 4800 7500 4850
 $Comp
-L GND #PWR?
+L GND #PWR021
 U 1 1 518027C2
 P 7100 5050
-F 0 "#PWR?" H 7100 5050 30  0001 C CNN
+F 0 "#PWR021" H 7100 5050 30  0001 C CNN
 F 1 "GND" H 7100 4980 30  0001 C CNN
 F 2 "" H 7100 5050 60  0000 C CNN
@@
 $EndComp
 $Comp
-L GND #PWR?
+L GND #PWR022
 U 1 1 518027D1
 P 7500 4850
-F 0 "#PWR?" H 7500 4850 30  0001 C CNN
+F 0 "#PWR022" H 7500 4850 30  0001 C CNN
 F 1 "GND" H 7500 4780 30  0001 C CNN
 F 2 "" H 7500 4850 60  0000 C CNN
@@
 $EndComp
 $Comp
-L BSP250 Q?
+L BSP250 Q5
 U 1 1 5180281C
 P 9200 3650
-F 0 "Q?" H 9200 3840 60  0000 R CNN
+F 0 "Q5" H 9200 3840 60  0000 R CNN
 F 1 "BSP250" H 9200 3470 60  0000 R CNN
 F 2 "" H 9200 3650 60  0000 C CNN
@@
 $EndComp
 $Comp
-L BSP250 Q?
+L BSP250 Q3
 U 1 1 5180282B
 P 7500 3650
-F 0 "Q?" H 7500 3840 60  0000 R CNN
+F 0 "Q3" H 7500 3840 60  0000 R CNN
 F 1 "BSP250" H 7500 3470 60  0000 R CNN
 F 2 "" H 7500 3650 60  0000 C CNN
@@
 $EndComp
 $Comp
-L R R?
+L R R52
 U 1 1 51802867
 P 7800 3750
-F 0 "R?" V 7750 3850 50  0000 C CNN
+F 0 "R52" V 7750 3850 50  0000 C CNN
 F 1 "R" V 7850 3850 50  0000 C CNN
 F 2 "" H 7800 3750 60  0000 C CNN
@@
 $EndComp
 $Comp
-L R R?
+L R R54
 U 1 1 51802876
 P 8800 3750
-F 0 "R?" V 8750 3850 50  0000 C CNN
+F 0 "R54" V 8750 3850 50  0000 C CNN
 F 1 "R" V 8850 3850 50  0000 C CNN
 F 2 "" H 8800 3750 60  0000 C CNN
@@
 $EndComp
 $Comp
-L +12V #PWR?
+L +12V #PWR023
 U 1 1 5180289C
 P 6500 4150
-F 0 "#PWR?" H 6500 4100 20  0001 C CNN
+F 0 "#PWR023" H 6500 4100 20  0001 C CNN
 F 1 "+12V" H 6500 4250 30  0000 C CNN
 F 2 "" H 6500 4150 60  0000 C CNN
@@
 Connection ~ 7800 3550
 $Comp
-L BC847 Q?
+L BC847 Q4
 U 1 1 51802936
 P 9100 4600
-F 0 "Q?" H 9250 4600 50  0000 C CNN
+F 0 "Q4" H 9250 4600 50  0000 C CNN
 F 1 "BC847" H 8900 4700 50  0000 C CNN
 F 2 "" H 9100 4600 60  0000 C CNN
@@
 $EndComp
 $Comp
-L R R?
+L R R53
 U 1 1 51802945
 P 8550 4600
-F 0 "R?" V 8500 4700 50  0000 C CNN
+F 0 "R53" V 8500 4700 50  0000 C CNN
 F 1 "R" V 8600 4700 50  0000 C CNN
 F 2 "" H 8550 4600 60  0000 C CNN
@@
 	7100 4600 7100 4700
 $Comp
-L R R?
+L R R50
 U 1 1 5180295E
 P 6750 4600
-F 0 "R?" V 6700 4700 50  0000 C CNN
+F 0 "R50" V 6700 4700 50  0000 C CNN
 F 1 "R" V 6800 4700 50  0000 C CNN
 F 2 "" H 6750 4600 60  0000 C CNN
@@
 Connection ~ 8300 3550
 $Comp
-L +12V #PWR?
+L +12V #PWR024
 U 1 1 51802A84
 P 8300 3450
-F 0 "#PWR?" H 8300 3400 20  0001 C CNN
+F 0 "#PWR024" H 8300 3400 20  0001 C CNN
 F 1 "+12V" H 8300 3550 30  0000 C CNN
 F 2 "" H 8300 3450 60  0000 C CNN
@@
 Connection ~ 7100 3500
 $Comp
-L CP C?
+L CP C35
 U 1 1 51802BC2
 P 9600 3750
-F 0 "C?" H 9650 3850 50  0000 L CNN
+F 0 "C35" H 9650 3850 50  0000 L CNN
 F 1 "CP" H 9650 3650 50  0000 L CNN
 F 2 "" H 9600 3750 60  0000 C CNN
@@
 $EndComp
 $Comp
-L CP C?
+L CP C33
 U 1 1 51802BD1
 P 7100 3750
-F 0 "C?" H 7150 3850 50  0000 L CNN
+F 0 "C33" H 7150 3850 50  0000 L CNN
 F 1 "CP" H 7150 3650 50  0000 L CNN
 F 2 "" H 7100 3750 60  0000 C CNN
@@
 	7100 3850 7100 3900
 $Comp
-L GND #PWR?
+L GND #PWR025
 U 1 1 51802C41
 P 9600 3900
-F 0 "#PWR?" H 9600 3900 30  0001 C CNN
+F 0 "#PWR025" H 9600 3900 30  0001 C CNN
 F 1 "GND" H 9600 3830 30  0001 C CNN
 F 2 "" H 9600 3900 60  0000 C CNN
@@
 $EndComp
 $Comp
-L GND #PWR?
+L GND #PWR026
 U 1 1 51802C50
 P 7100 3900
-F 0 "#PWR?" H 7100 3900 30  0001 C CNN
+F 0 "#PWR026" H 7100 3900 30  0001 C CNN
 F 1 "GND" H 7100 3830 30  0001 C CNN
 F 2 "" H 7100 3900 60  0000 C CNN
@@
 	9200 4800 9200 4850
 $Comp
-L GND #PWR?
+L GND #PWR027
 U 1 1 51802C91
 P 9200 4850
-F 0 "#PWR?" H 9200 4850 30  0001 C CNN
+F 0 "#PWR027" H 9200 4850 30  0001 C CNN
 F 1 "GND" H 9200 4780 30  0001 C CNN
 F 2 "" H 9200 4850 60  0000 C CNN
@@
 $EndComp
 $Comp
-L CP C?
+L CP C34
 U 1 1 51802CA0
 P 8300 3750
-F 0 "C?" H 8350 3850 50  0000 L CNN
+F 0 "C34" H 8350 3850 50  0000 L CNN
 F 1 "CP" H 8350 3650 50  0000 L CNN
 F 2 "" H 8300 3750 60  0000 C CNN
@@
 	8300 3850 8300 3900
 $Comp
-L GND #PWR?
+L GND #PWR028
 U 1 1 51802D14
 P 8300 3900
-F 0 "#PWR?" H 8300 3900 30  0001 C CNN
+F 0 "#PWR028" H 8300 3900 30  0001 C CNN
 F 1 "GND" H 8300 3830 30  0001 C CNN
 F 2 "" H 8300 3900 60  0000 C CNN

Commit message: Routage  PCB
Other:
- moved on the sheet: R53
Changed lines of the file:
@@
-EESchema Schematic File Version 2  date 04/06/2013 21:43:31
+EESchema Schematic File Version 2  date 09/06/2013 23:13:58
 LIBS:power
 LIBS:CEN-SCHEMA
@@
 Sheet 3 6
 Title ""
-Date "4 jun 2013"
+Date "9 jun 2013"
 Rev ""
 Comp ""
@@
 Comment4 ""
 $EndDescr
-Text HLabel 6000 4850 0    60   Input ~ 0
+Text HLabel 5550 4850 0    60   Input ~ 0
 PTT
 $Comp
@@
 	3100 3600 3100 3450
 $Comp
-L +12V #PWR018
+L +12V #PWR020
 U 1 1 514F9C6A
 P 3100 3450
-F 0 "#PWR018" H 3100 3400 20  0001 C CNN
+F 0 "#PWR020" H 3100 3400 20  0001 C CNN
 F 1 "+12V" H 3100 3550 30  0000 C CNN
 F 2 "" H 3100 3450 60  0000 C CNN
@@
 Text HLabel 3700 4200 2    60   Input ~ 0
 AFE
-$Comp
-L BC847 Q1
-U 1 1 518025F5
-P 6400 4850
-F 0 "Q1" H 6550 4850 50  0000 C CNN
-F 1 "BC847" H 6200 4950 50  0000 C CNN
-F 2 "" H 6400 4850 60  0000 C CNN
-F 3 "" H 6400 4850 60  0000 C CNN
-	1    6400 4850
-	1    0    0    -1
-$EndComp
 $Comp
 L R R5
@@
 	6500 5050 6500 5100
 $Comp
-L GND #PWR019
+L GND #PWR021
 U 1 1 5180264F
 P 6500 5100
-F 0 "#PWR019" H 6500 5100 30  0001 C CNN
+F 0 "#PWR021" H 6500 5100 30  0001 C CNN
 F 1 "GND" H 6500 5030 30  0001 C CNN
 F 2 "" H 6500 5100 60  0000 C CNN
@@
 $EndComp
 $Comp
-L +5V #PWR020
+L +5V #PWR022
 U 1 1 5180265E
 P 6100 4400
-F 0 "#PWR020" H 6100 4490 20  0001 C CNN
+F 0 "#PWR022" H 6100 4490 20  0001 C CNN
 F 1 "+5V" H 6100 4490 30  0000 C CNN
 F 2 "" H 6100 4400 60  0000 C CNN
@@
 	7500 4800 7500 4850
 $Comp
-L GND #PWR021
+L GND #PWR023
 U 1 1 518027C2
 P 7100 5050
-F 0 "#PWR021" H 7100 5050 30  0001 C CNN
+F 0 "#PWR023" H 7100 5050 30  0001 C CNN
 F 1 "GND" H 7100 4980 30  0001 C CNN
 F 2 "" H 7100 5050 60  0000 C CNN
@@
 $EndComp
 $Comp
-L GND #PWR022
+L GND #PWR024
 U 1 1 518027D1
 P 7500 4850
-F 0 "#PWR022" H 7500 4850 30  0001 C CNN
+F 0 "#PWR024" H 7500 4850 30  0001 C CNN
 F 1 "GND" H 7500 4780 30  0001 C CNN
 F 2 "" H 7500 4850 60  0000 C CNN
@@
 $EndComp
 $Comp
-L +12V #PWR023
+L +12V #PWR025
 U 1 1 5180289C
 P 6500 4150
-F 0 "#PWR023" H 6500 4100 20  0001 C CNN
+F 0 "#PWR025" H 6500 4100 20  0001 C CNN
 F 1 "+12V" H 6500 4250 30  0000 C CNN
 F 2 "" H 6500 4150 60  0000 C CNN
@@
 L R R53
 U 1 1 51802945
-P 8550 4600
-F 0 "R53" V 8500 4700 50  0000 C CNN
-F 1 "R" V 8600 4700 50  0000 C CNN
-F 2 "" H 8550 4600 60  0000 C CNN
-F 3 "" H 8550 4600 60  0000 C CNN
-	1    8550 4600
+P 5750 4850
+F 0 "R53" V 5700 4950 50  0000 C CNN
+F 1 "R" V 5800 4950 50  0000 C CNN
+F 2 "" H 5750 4850 60  0000 C CNN
+F 3 "" H 5750 4850 60  0000 C CNN
+	1    5750 4850
 	0    -1   -1   0
 $EndComp
@@
 	8300 5250 8300 4600
 Wire Wire Line
-	8300 4600 8500 4600
-Wire Wire Line
-	8800 4600 8900 4600
-Wire Wire Line
-	9200 4400 9200 3850
+	8300 4600 8900 4600
+Wire Wire Line
+	9200 3850 9200 4400
 Wire Wire Line
 	8800 4000 9200 4000
@@
 Connection ~ 8300 3550
 $Comp
-L +12V #PWR024
+L +12V #PWR026
 U 1 1 51802A84
 P 8300 3450
-F 0 "#PWR024" H 8300 3400 20  0001 C CNN
+F 0 "#PWR026" H 8300 3400 20  0001 C CNN
 F 1 "+12V" H 8300 3550 30  0000 C CNN
 F 2 "" H 8300 3450 60  0000 C CNN
@@
 	7100 3850 7100 3900
 $Comp
-L GND #PWR025
+L GND #PWR027
 U 1 1 51802C41
 P 9600 3900
-F 0 "#PWR025" H 9600 3900 30  0001 C CNN
+F 0 "#PWR027" H 9600 3900 30  0001 C CNN
 F 1 "GND" H 9600 3830 30  0001 C CNN
 F 2 "" H 9600 3900 60  0000 C CNN
@@
 $EndComp
 $Comp
-L GND #PWR026
+L GND #PWR028
 U 1 1 51802C50
 P 7100 3900
-F 0 "#PWR026" H 7100 3900 30  0001 C CNN
+F 0 "#PWR028" H 7100 3900 30  0001 C CNN
 F 1 "GND" H 7100 3830 30  0001 C CNN
 F 2 "" H 7100 3900 60  0000 C CNN
@@
 	9200 4800 9200 4850
 $Comp
-L GND #PWR027
+L GND #PWR029
 U 1 1 51802C91
 P 9200 4850
-F 0 "#PWR027" H 9200 4850 30  0001 C CNN
+F 0 "#PWR029" H 9200 4850 30  0001 C CNN
 F 1 "GND" H 9200 4780 30  0001 C CNN
 F 2 "" H 9200 4850 60  0000 C CNN
@@
 	8300 3850 8300 3900
 $Comp
-L GND #PWR028
+L GND #PWR030
 U 1 1 51802D14
 P 8300 3900
-F 0 "#PWR028" H 8300 3900 30  0001 C CNN
+F 0 "#PWR030" H 8300 3900 30  0001 C CNN
 F 1 "GND" H 8300 3830 30  0001 C CNN
 F 2 "" H 8300 3900 60  0000 C CNN
@@
 	1    0    0    -1
 $EndComp
+Wire Wire Line
+	5550 4850 5700 4850
+$Comp
+L BC847 Q1
+U 1 1 518025F5
+P 6400 4850
+F 0 "Q1" H 6550 4850 50  0000 C CNN
+F 1 "BC847" H 6200 4950 50  0000 C CNN
+F 2 "" H 6400 4850 60  0000 C CNN
+F 3 "" H 6400 4850 60  0000 C CNN
+	1    6400 4850
+	1    0    0    -1
+$EndComp

Commit message: Reste 2 pistes a router
Connections:
- net labels added: +5VD
- net labels removed: +5V
Changed lines of the file:
@@
-EESchema Schematic File Version 2  date 09/06/2013 23:13:58
+EESchema Schematic File Version 2  date 11/06/2013 22:16:43
 LIBS:power
 LIBS:CEN-SCHEMA
@@
 Sheet 3 6
 Title ""
-Date "9 jun 2013"
+Date "11 jun 2013"
 Rev ""
 Comp ""
@@
 	1    0    0    -1
 $EndComp
-$Comp
-L +5V #PWR022
-U 1 1 5180265E
-P 6100 4400
-F 0 "#PWR022" H 6100 4490 20  0001 C CNN
-F 1 "+5V" H 6100 4490 30  0000 C CNN
-F 2 "" H 6100 4400 60  0000 C CNN
-F 3 "" H 6100 4400 60  0000 C CNN
-	1    6100 4400
-	1    0    0    -1
-$EndComp
 Wire Wire Line
 	6500 4550 6500 4650
@@
 	1    0    0    -1
 $EndComp
+$Comp
+L +5VD #PWR?
+U 1 1 51B7A81B
+P 6100 4400
+F 0 "#PWR?" H 6100 4350 20  0001 C CNN
+F 1 "+5VD" H 6100 4500 30  0000 C CNN
+F 2 "" H 6100 4400 60  0000 C CNN
+F 3 "" H 6100 4400 60  0000 C CNN
+	1    6100 4400
+	1    0    0    -1
+$EndComp

Commit message: Fin PCB
Parts:
- added D3, D4, D5, D6, D7, D8, D9: LED, symbol LED
- added R55, R56, R57, R58, R59, R60, R61: 1k, symbol R
Connections:
- net +12V: now also D3.1 (A)
- net +12VRX: now also D9.1 (A)
- net +12VTX: now also D8.1 (A)
- net +5VD: now also D4.1 (A)
- net GND: now also R55.2, R56.2, R57.2, R58.2, R59.2, R60.2, R61.2
- new net: D3.2 (K), R55.1
- new net: D4.2 (K), R56.1
- new net: D5.2 (K), R57.1
- new net: D6.2 (K), R58.1
- new net: D7.2 (K), R59.1
- new net: D8.2 (K), R60.1
- new net: D9.2 (K), R61.1
- new net +3.3V: D7.1 (A)
- new net +5VA: D5.1 (A)
- new net -5VA: D6.1 (A)
