File: JK330-1-BF/MIC.sch (KiCad schematic (older format))
At the start: 31 parts, among them Q1 BC847, Q2 BC847, Q3 BSP250, Q4 BC847, Q5 BSP250

Commit message: Ajout carte power
Parts:
- C33, C34, C35: value CP -> 10U
- D8: value LED -> ROUGE
- D9: value LED -> VERT
- R49, R5: value R -> 10k
- R50: value R -> 0
- R51: value R -> NC
- R52, R54: value R -> 4.7k
- R53: value R -> 1.5k
- R55: value 1k -> 3.3k
- R59: value 1k -> 470
- R60, R61: value 1k -> 3k3
Other:
- note added: "A CABLER"
Changed lines of the file:
@@
 Sheet 3 6
 Title "JK330 "
-Date "18 jun 2013"
+Date "18 jul 2013"
 Rev "V0.10"
 Comp "F4DEB 2013"
@@
 P 6100 4550
 F 0 "R5" V 6050 4650 50  0000 C CNN
-F 1 "R" V 6150 4650 50  0000 C CNN
+F 1 "10k" V 6150 4650 50  0000 C CNN
 F 2 "" H 6100 4550 60  0000 C CNN
 F 3 "" H 6100 4550 60  0000 C CNN
@@
 P 6500 4300
 F 0 "R49" V 6450 4400 50  0000 C CNN
-F 1 "R" V 6550 4400 50  0000 C CNN
+F 1 "10k" V 6550 4400 50  0000 C CNN
 F 2 "" H 6500 4300 60  0000 C CNN
 F 3 "" H 6500 4300 60  0000 C CNN
@@
 P 7100 4750
 F 0 "R51" V 7050 4850 50  0000 C CNN
-F 1 "R" V 7150 4850 50  0000 C CNN
+F 1 "NC" V 7150 4850 50  0000 C CNN
 F 2 "" H 7100 4750 60  0000 C CNN
 F 3 "" H 7100 4750 60  0000 C CNN
@@
 P 7800 3750
 F 0 "R52" V 7750 3850 50  0000 C CNN
-F 1 "R" V 7850 3850 50  0000 C CNN
+F 1 "4.7k" V 7850 3850 50  0000 C CNN
 F 2 "" H 7800 3750 60  0000 C CNN
 F 3 "" H 7800 3750 60  0000 C CNN
@@
 P 8800 3750
 F 0 "R54" V 8750 3850 50  0000 C CNN
-F 1 "R" V 8850 3850 50  0000 C CNN
+F 1 "4.7k" V 8850 3850 50  0000 C CNN
 F 2 "" H 8800 3750 60  0000 C CNN
 F 3 "" H 8800 3750 60  0000 C CNN
@@
 P 5750 4850
 F 0 "R53" V 5700 4950 50  0000 C CNN
-F 1 "R" V 5800 4950 50  0000 C CNN
+F 1 "1.5k" V 5800 4950 50  0000 C CNN
 F 2 "" H 5750 4850 60  0000 C CNN
 F 3 "" H 5750 4850 60  0000 C CNN
@@
 P 6750 4600
 F 0 "R50" V 6700 4700 50  0000 C CNN
-F 1 "R" V 6800 4700 50  0000 C CNN
+F 1 "0" V 6800 4700 50  0000 C CNN
 F 2 "" H 6750 4600 60  0000 C CNN
 F 3 "" H 6750 4600 60  0000 C CNN
@@
 P 9600 3750
 F 0 "C35" H 9650 3850 50  0000 L CNN
-F 1 "CP" H 9650 3650 50  0000 L CNN
+F 1 "10U" H 9650 3650 50  0000 L CNN
 F 2 "" H 9600 3750 60  0000 C CNN
 F 3 "" H 9600 3750 60  0000 C CNN
@@
 P 7100 3750
 F 0 "C33" H 7150 3850 50  0000 L CNN
-F 1 "CP" H 7150 3650 50  0000 L CNN
+F 1 "10U" H 7150 3650 50  0000 L CNN
 F 2 "" H 7100 3750 60  0000 C CNN
 F 3 "" H 7100 3750 60  0000 C CNN
@@
 P 8300 3750
 F 0 "C34" H 8350 3850 50  0000 L CNN
-F 1 "CP" H 8350 3650 50  0000 L CNN
+F 1 "10U" H 8350 3650 50  0000 L CNN
 F 2 "" H 8300 3750 60  0000 C CNN
 F 3 "" H 8300 3750 60  0000 C CNN
@@
 U 1 1 51BE01D5
 P 4350 2150
-F 0 "R55" V 4300 2000 50  0000 C CNN
-F 1 "1k" V 4300 2150 50  0000 C CNN
+F 0 "R55" V 4300 2050 50  0000 C CNN
+F 1 "3.3k" V 4450 2050 50  0000 C CNN
 F 2 "" H 4350 2150 60  0000 C CNN
 F 3 "" H 4350 2150 60  0000 C CNN
@@
 U 1 1 51BE01E4
 P 4650 2150
-F 0 "R56" V 4600 2000 50  0000 C CNN
-F 1 "1k" V 4600 2150 50  0000 C CNN
+F 0 "R56" V 4600 2050 50  0000 C CNN
+F 1 "1k" V 4750 2050 50  0000 C CNN
 F 2 "" H 4650 2150 60  0000 C CNN
 F 3 "" H 4650 2150 60  0000 C CNN
@@
 U 1 1 51BE01F3
 P 4950 2150
-F 0 "R57" V 4900 2000 50  0000 C CNN
-F 1 "1k" V 4900 2150 50  0000 C CNN
+F 0 "R57" V 4900 2050 50  0000 C CNN
+F 1 "1k" V 5050 2050 50  0000 C CNN
 F 2 "" H 4950 2150 60  0000 C CNN
 F 3 "" H 4950 2150 60  0000 C CNN
@@
 U 1 1 51BE0202
 P 5250 2150
-F 0 "R58" V 5200 2000 50  0000 C CNN
-F 1 "1k" V 5200 2150 50  0000 C CNN
+F 0 "R58" V 5200 2050 50  0000 C CNN
+F 1 "1k" V 5350 2050 50  0000 C CNN
 F 2 "" H 5250 2150 60  0000 C CNN
 F 3 "" H 5250 2150 60  0000 C CNN
@@
 U 1 1 51BE0211
 P 5550 2150
-F 0 "R59" V 5500 2000 50  0000 C CNN
-F 1 "1k" V 5500 2150 50  0000 C CNN
+F 0 "R59" V 5500 2050 50  0000 C CNN
+F 1 "470" V 5650 2050 50  0000 C CNN
 F 2 "" H 5550 2150 60  0000 C CNN
 F 3 "" H 5550 2150 60  0000 C CNN
@@
 P 6850 3600
 F 0 "R60" V 6800 3450 50  0000 C CNN
-F 1 "1k" V 6800 3600 50  0000 C CNN
+F 1 "3k3" V 6800 3600 50  0000 C CNN
 F 2 "" H 6850 3600 60  0000 C CNN
 F 3 "" H 6850 3600 60  0000 C CNN
@@
 P 6850 3300
 F 0 "D8" H 6850 3400 50  0000 C CNN
-F 1 "LED" H 6850 3200 50  0000 C CNN
+F 1 "ROUGE" H 6850 3200 50  0000 C CNN
 F 2 "" H 6850 3300 60  0000 C CNN
 F 3 "" H 6850 3300 60  0000 C CNN
@@
 P 9900 3600
 F 0 "R61" V 9850 3450 50  0000 C CNN
-F 1 "1k" V 9850 3600 50  0000 C CNN
+F 1 "3k3" V 9850 3600 50  0000 C CNN
 F 2 "" H 9900 3600 60  0000 C CNN
 F 3 "" H 9900 3600 60  0000 C CNN
@@
 P 9900 3300
 F 0 "D9" H 9900 3400 50  0000 C CNN
-F 1 "LED" H 9900 3200 50  0000 C CNN
+F 1 "VERT" H 9900 3200 50  0000 C CNN
 F 2 "" H 9900 3300 60  0000 C CNN
 F 3 "" H 9900 3300 60  0000 C CNN
@@
 	9900 3150 9600 3150
 Connection ~ 9600 3150
+Wire Notes Line
+	2200 2950 4250 2950
+Wire Notes Line
+	4250 2950 4250 4650
+Wire Notes Line
+	4250 4650 2200 4650
+Wire Notes Line
+	2200 4650 2200 2950
+Text Notes 3600 3750 0    60   ~ 0
+A CABLER
 $EndSCHEMATC
