File: JK330-1-BF/NOTCH.sch (KiCad schematic (older format))
At the start: 37 parts, among them P8 CAVALIER, U4 74HC74, U6 MC33172, U7 MF10, U8 74HC4059, U9 74HC377

Commit message: MAJ  composants
Changed lines of the file:
@@
-EESchema Schematic File Version 2  date 2013-03-25 22:18:17
+EESchema Schematic File Version 2  date 29/04/2013 22:12:34
 LIBS:power
 LIBS:CEN-SCHEMA
@@
 Sheet 5 6
 Title "F4DEB"
-Date "25 mar 2013"
+Date "29 apr 2013"
 Rev "V 3.00"
 Comp "RACKANOUS"
@@
 U 1 1 4994977B
 P 8650 2150
-F 0 "R28" V 8600 2250 50  0000 C CNN
-F 1 "11k5" V 8700 2250 50  0000 C CNN
+F 0 "R28" V 8700 2200 50  0000 C CNN
+F 1 "11k5" V 8700 2000 50  0000 C CNN
 F 2 "" H 8650 2150 60  0001 C CNN
 F 3 "" H 8650 2150 60  0001 C CNN
@@
 U 1 1 49949778
 P 9650 1750
-F 0 "R27" V 9600 1850 50  0000 C CNN
-F 1 "11k5" V 9700 1850 50  0000 C CNN
+F 0 "R27" V 9550 1550 50  0000 C CNN
+F 1 "11k5" V 9550 1800 50  0000 C CNN
 F 2 "" H 9650 1750 60  0001 C CNN
 F 3 "" H 9650 1750 60  0001 C CNN
@@
 U 1 1 49949776
 P 8850 1750
-F 0 "R26" V 8800 1850 50  0000 C CNN
-F 1 "11.5k" V 8900 1850 50  0000 C CNN
+F 0 "R26" V 8750 1550 50  0000 C CNN
+F 1 "11.5k" V 8750 1800 50  0000 C CNN
 F 2 "" H 8850 1750 60  0001 C CNN
 F 3 "" H 8850 1750 60  0001 C CNN
@@
 U 1 1 499496DB
 P 7550 1500
-F 0 "R25" V 7500 1600 50  0000 C CNN
-F 1 "11.5k" V 7600 1600 50  0000 C CNN
+F 0 "R25" V 7500 1300 50  0000 C CNN
+F 1 "11.5k" V 7500 1550 50  0000 C CNN
 F 2 "" H 7550 1500 60  0001 C CNN
 F 3 "" H 7550 1500 60  0001 C CNN
@@
 U 1 1 499496CF
 P 6950 1000
-F 0 "R23" V 6900 1100 50  0000 C CNN
-F 1 "11.5k" V 7000 1100 50  0000 C CNN
+F 0 "R23" V 6900 800 50  0000 C CNN
+F 1 "11.5k" V 6900 1050 50  0000 C CNN
 F 2 "" H 6950 1000 60  0001 C CNN
 F 3 "" H 6950 1000 60  0001 C CNN
@@
 U 1 1 499496CD
 P 6300 1400
-F 0 "R24" V 6250 1500 50  0000 C CNN
-F 1 "11.5k" V 6350 1500 50  0000 C CNN
+F 0 "R24" V 6250 1200 50  0000 C CNN
+F 1 "11.5k" V 6250 1450 50  0000 C CNN
 F 2 "" H 6300 1400 60  0001 C CNN
 F 3 "" H 6300 1400 60  0001 C CNN
@@
 U 1 1 499496C8
 P 6300 1000
-F 0 "R22" V 6250 1100 50  0000 C CNN
-F 1 "11.5k" V 6350 1100 50  0000 C CNN
+F 0 "R22" V 6250 800 50  0000 C CNN
+F 1 "11.5k" V 6250 1050 50  0000 C CNN
 F 2 "" H 6300 1000 60  0001 C CNN
 F 3 "" H 6300 1000 60  0001 C CNN
@@
 U 2 1 4994968B
 P 9550 2250
-F 0 "U6" H 9650 2500 60  0000 L CNN
-F 1 "MC33172" H 9650 2100 60  0000 L CNN
+F 0 "U6" H 9550 2500 60  0000 L CNN
+F 1 "MC33172" H 9400 2000 60  0000 L CNN
 F 2 "" H 9550 2250 60  0001 C CNN
 F 3 "" H 9550 2250 60  0001 C CNN
@@
 U 1 1 4994967F
 P 6850 1500
-F 0 "U6" H 6950 1750 60  0000 L CNN
-F 1 "MC33172" H 6950 1350 60  0000 L CNN
+F 0 "U6" H 6650 1250 60  0000 L CNN
+F 1 "MC33172" H 6350 1800 60  0000 L CNN
 F 2 "" H 6850 1500 60  0001 C CNN
 F 3 "" H 6850 1500 60  0001 C CNN
@@
 U 1 1 499491D7
 P 10250 2250
-F 0 "R29" V 10200 2150 50  0000 C CNN
-F 1 "R" V 10300 2150 50  0000 C CNN
+F 0 "R29" V 10200 2050 50  0000 C CNN
+F 1 "R" V 10200 2200 50  0000 C CNN
 F 2 "" H 10250 2250 60  0001 C CNN
 F 3 "" H 10250 2250 60  0001 C CNN
@@
 U 1 1 499491D4
 P 7800 2650
-F 0 "R35" V 7750 2750 50  0000 C CNN
-F 1 "11.5k" V 7850 2750 50  0000 C CNN
+F 0 "R35" V 7750 2450 50  0000 C CNN
+F 1 "11.5k" V 7750 2650 50  0000 C CNN
 F 2 "" H 7800 2650 60  0001 C CNN
 F 3 "" H 7800 2650 60  0001 C CNN
@@
 U 1 1 499491D1
 P 7800 2550
-F 0 "R33" V 7750 2650 50  0000 C CNN
-F 1 "100k" V 7850 2650 50  0000 C CNN
+F 0 "R33" V 7750 2350 50  0000 C CNN
+F 1 "100k" V 7750 2550 50  0000 C CNN
 F 2 "" H 7800 2550 60  0001 C CNN
 F 3 "" H 7800 2550 60  0001 C CNN
@@
 U 1 1 499491CC
 P 7800 2450
-F 0 "R31" V 7750 2550 50  0000 C CNN
-F 1 "11.5k" V 7850 2550 50  0000 C CNN
+F 0 "R31" V 7750 2250 50  0000 C CNN
+F 1 "11.5k" V 7750 2450 50  0000 C CNN
 F 2 "" H 7800 2450 60  0001 C CNN
 F 3 "" H 7800 2450 60  0001 C CNN
@@
 U 1 1 499491C1
 P 5100 2800
-F 0 "R36" V 5050 2900 50  0000 C CNN
-F 1 "11.5k" V 5150 2900 50  0000 C CNN
+F 0 "R36" V 5050 2600 50  0000 C CNN
+F 1 "11.5k" V 5050 2800 50  0000 C CNN
 F 2 "" H 5100 2800 60  0001 C CNN
 F 3 "" H 5100 2800 60  0001 C CNN
@@
 U 1 1 499491B9
 P 5550 2550
-F 0 "R32" V 5500 2650 50  0000 C CNN
-F 1 "100k" V 5600 2650 50  0000 C CNN
+F 0 "R32" V 5500 2350 50  0000 C CNN
+F 1 "100k" V 5500 2600 50  0000 C CNN
 F 2 "" H 5550 2550 60  0001 C CNN
 F 3 "" H 5550 2550 60  0001 C CNN
@@
 U 1 1 499491AC
 P 5550 2650
-F 0 "R34" V 5500 2750 50  0000 C CNN
-F 1 "11.5k" V 5600 2750 50  0000 C CNN
+F 0 "R34" V 5500 2450 50  0000 C CNN
+F 1 "11.5k" V 5500 2700 50  0000 C CNN
 F 2 "" H 5550 2650 60  0001 C CNN
 F 3 "" H 5550 2650 60  0001 C CNN
@@
 U 1 1 499491A8
 P 5550 2450
-F 0 "R30" V 5500 2550 50  0000 C CNN
-F 1 "11.5k" V 5600 2550 50  0000 C CNN
+F 0 "R30" V 5500 2250 50  0000 C CNN
+F 1 "11.5k" V 5500 2500 50  0000 C CNN
 F 2 "" H 5550 2450 60  0001 C CNN
 F 3 "" H 5550 2450 60  0001 C CNN
@@
 U 1 1 514F7067
 P 10550 2250
-F 0 "C17" H 10600 2350 50  0000 L CNN
-F 1 "C" H 10600 2150 50  0000 L CNN
+F 0 "C17" V 10650 2050 50  0000 L CNN
+F 1 "C" V 10450 2150 50  0000 L CNN
 F 2 "" H 10550 2250 60  0000 C CNN
 F 3 "" H 10550 2250 60  0000 C CNN
@@
 U 1 1 514F72E5
 P 7650 750
-F 0 "P8" H 7800 750 60  0000 C CNN
+F 0 "P8" H 7750 950 60  0000 C CNN
 F 1 "CAVALIER" H 7800 850 60  0000 C CNN
 F 2 "" H 7650 750 60  0000 C CNN

Commit message: Reste 2 pistes a router
Connections:
- net labels removed: +5V
Changed lines of the file:
@@
-EESchema Schematic File Version 2  date 09/06/2013 23:13:58
+EESchema Schematic File Version 2  date 11/06/2013 22:16:43
 LIBS:power
 LIBS:CEN-SCHEMA
@@
 Sheet 5 6
 Title "F4DEB"
-Date "9 jun 2013"
+Date "11 jun 2013"
 Rev "V 3.00"
 Comp "RACKANOUS"
@@
 Comment4 ""
 $EndDescr
-$Comp
-L +5V #PWR058
-U 1 1 4A9EC139
-P 4700 7000
-F 0 "#PWR058" H 4700 7090 20  0001 C CNN
-F 1 "+5V" H 4700 7090 30  0000 C CNN
-F 2 "" H 4700 7000 60  0001 C CNN
-F 3 "" H 4700 7000 60  0001 C CNN
-	1    4700 7000
-	-1   0    0    1
-$EndComp
 Text Notes 3100 3850 0    60   ~ 0
 U9
@@
 $EndComp
 $Comp
-L +5V #PWR069
-U 1 1 5150BF88
-P 5850 5950
-F 0 "#PWR069" H 5850 6040 20  0001 C CNN
-F 1 "+5V" H 5850 6040 30  0000 C CNN
-F 2 "" H 5850 5950 60  0001 C CNN
-F 3 "" H 5850 5950 60  0001 C CNN
-	1    5850 5950
-	0    -1   -1   0
-$EndComp
-$Comp
-L +5V #PWR070
-U 1 1 5150BF87
-P 5850 5600
-F 0 "#PWR070" H 5850 5690 20  0001 C CNN
-F 1 "+5V" H 5850 5690 30  0000 C CNN
-F 2 "" H 5850 5600 60  0001 C CNN
-F 3 "" H 5850 5600 60  0001 C CNN
-	1    5850 5600
-	0    -1   -1   0
-$EndComp
-$Comp
 L 74HC74 U4
 U 2 1 5150BF86
@@
 	1    0    0    -1
 $EndComp
+$Comp
+L +5VD #PWR?
+U 1 1 51B7AA1A
+P 4700 7000
+F 0 "#PWR?" H 4700 6950 20  0001 C CNN
+F 1 "+5VD" H 4700 7100 30  0000 C CNN
+F 2 "" H 4700 7000 60  0000 C CNN
+F 3 "" H 4700 7000 60  0000 C CNN
+	1    4700 7000
+	-1   0    0    1
+$EndComp
+$Comp
+L +5VD #PWR?
+U 1 1 51B7AA29
+P 5850 5600
+F 0 "#PWR?" H 5850 5550 20  0001 C CNN
+F 1 "+5VD" H 5850 5700 30  0000 C CNN
+F 2 "" H 5850 5600 60  0000 C CNN
+F 3 "" H 5850 5600 60  0000 C CNN
+	1    5850 5600
+	0    -1   -1   0
+$EndComp
+$Comp
+L +5VD #PWR?
+U 1 1 51B7AA38
+P 5850 5950
+F 0 "#PWR?" H 5850 5900 20  0001 C CNN
+F 1 "+5VD" H 5850 6050 30  0000 C CNN
+F 2 "" H 5850 5950 60  0000 C CNN
+F 3 "" H 5850 5950 60  0000 C CNN
+	1    5850 5950
+	0    -1   -1   0
+$EndComp
 $EndSCHEMATC
