File: JK330-1-BF/NOTCH.sch (KiCad schematic (older format))
At the start: 37 parts, among them P8 CAVALIER, U4 74HC74, U6 MC33172, U7 MF10, U8 74HC4059, U9 74HC377

Commit message: Ajout carte power
Parts:
- C17: value C -> 100n
- R22, R23, R24, R25, R26, R30, R31, R34, R35, R36: value 11.5k -> 11.3k
- R27, R28: value 11k5 -> 11.3k
- R29: value R -> 47k
Changed lines of the file:
@@
 Sheet 5 6
 Title "JK330 "
-Date "18 jun 2013"
+Date "18 jul 2013"
 Rev "V0.10"
 Comp "F4DEB 2013"
@@
 P 8650 2150
 F 0 "R28" V 8700 2200 50  0000 C CNN
-F 1 "11k5" V 8700 2000 50  0000 C CNN
+F 1 "11.3k" V 8700 2000 50  0000 C CNN
 F 2 "" H 8650 2150 60  0001 C CNN
 F 3 "" H 8650 2150 60  0001 C CNN
@@
 P 9650 1750
 F 0 "R27" V 9550 1550 50  0000 C CNN
-F 1 "11k5" V 9550 1800 50  0000 C CNN
+F 1 "11.3k" V 9550 1800 50  0000 C CNN
 F 2 "" H 9650 1750 60  0001 C CNN
 F 3 "" H 9650 1750 60  0001 C CNN
@@
 P 8850 1750
 F 0 "R26" V 8750 1550 50  0000 C CNN
-F 1 "11.5k" V 8750 1800 50  0000 C CNN
+F 1 "11.3k" V 8750 1800 50  0000 C CNN
 F 2 "" H 8850 1750 60  0001 C CNN
 F 3 "" H 8850 1750 60  0001 C CNN
@@
 P 7550 1500
 F 0 "R25" V 7500 1300 50  0000 C CNN
-F 1 "11.5k" V 7500 1550 50  0000 C CNN
+F 1 "11.3k" V 7500 1550 50  0000 C CNN
 F 2 "" H 7550 1500 60  0001 C CNN
 F 3 "" H 7550 1500 60  0001 C CNN
@@
 P 6950 1000
 F 0 "R23" V 6900 800 50  0000 C CNN
-F 1 "11.5k" V 6900 1050 50  0000 C CNN
+F 1 "11.3k" V 6900 1050 50  0000 C CNN
 F 2 "" H 6950 1000 60  0001 C CNN
 F 3 "" H 6950 1000 60  0001 C CNN
@@
 P 6300 1400
 F 0 "R24" V 6250 1200 50  0000 C CNN
-F 1 "11.5k" V 6250 1450 50  0000 C CNN
+F 1 "11.3k" V 6250 1450 50  0000 C CNN
 F 2 "" H 6300 1400 60  0001 C CNN
 F 3 "" H 6300 1400 60  0001 C CNN
@@
 P 6300 1000
 F 0 "R22" V 6250 800 50  0000 C CNN
-F 1 "11.5k" V 6250 1050 50  0000 C CNN
+F 1 "11.3k" V 6250 1050 50  0000 C CNN
 F 2 "" H 6300 1000 60  0001 C CNN
 F 3 "" H 6300 1000 60  0001 C CNN
@@
 P 10250 2250
 F 0 "R29" V 10200 2050 50  0000 C CNN
-F 1 "R" V 10200 2200 50  0000 C CNN
+F 1 "47k" V 10200 2200 50  0000 C CNN
 F 2 "" H 10250 2250 60  0001 C CNN
 F 3 "" H 10250 2250 60  0001 C CNN
@@
 P 7800 2650
 F 0 "R35" V 7750 2450 50  0000 C CNN
-F 1 "11.5k" V 7750 2650 50  0000 C CNN
+F 1 "11.3k" V 7750 2650 50  0000 C CNN
 F 2 "" H 7800 2650 60  0001 C CNN
 F 3 "" H 7800 2650 60  0001 C CNN
@@
 P 7800 2450
 F 0 "R31" V 7750 2250 50  0000 C CNN
-F 1 "11.5k" V 7750 2450 50  0000 C CNN
+F 1 "11.3k" V 7750 2450 50  0000 C CNN
 F 2 "" H 7800 2450 60  0001 C CNN
 F 3 "" H 7800 2450 60  0001 C CNN
@@
 P 5100 2800
 F 0 "R36" V 5050 2600 50  0000 C CNN
-F 1 "11.5k" V 5050 2800 50  0000 C CNN
+F 1 "11.3k" V 5050 2800 50  0000 C CNN
 F 2 "" H 5100 2800 60  0001 C CNN
 F 3 "" H 5100 2800 60  0001 C CNN
@@
 P 5550 2650
 F 0 "R34" V 5500 2450 50  0000 C CNN
-F 1 "11.5k" V 5500 2700 50  0000 C CNN
+F 1 "11.3k" V 5500 2700 50  0000 C CNN
 F 2 "" H 5550 2650 60  0001 C CNN
 F 3 "" H 5550 2650 60  0001 C CNN
@@
 P 5550 2450
 F 0 "R30" V 5500 2250 50  0000 C CNN
-F 1 "11.5k" V 5500 2500 50  0000 C CNN
+F 1 "11.3k" V 5500 2500 50  0000 C CNN
 F 2 "" H 5550 2450 60  0001 C CNN
 F 3 "" H 5550 2450 60  0001 C CNN
@@
 P 10550 2250
 F 0 "C17" V 10650 2050 50  0000 L CNN
-F 1 "C" V 10450 2150 50  0000 L CNN
+F 1 "100n" V 10450 2150 50  0000 L CNN
 F 2 "" H 10550 2250 60  0000 C CNN
 F 3 "" H 10550 2250 60  0000 C CNN
