File: JK330-1-BF/Mixer9Mhz.sch (KiCad schematic (older format))
At the start: 12 parts

Commit message: Ajout carte power
Parts:
- C1, C2: value 10U -> 220U
Changed lines of the file:
@@
 Sheet 2 6
 Title "JK330 "
-Date "18 jun 2013"
+Date "18 jul 2013"
 Rev "V0.10"
 Comp "F4DEB 2013"
@@
 P 5025 2600
 F 0 "C1" H 5075 2700 50  0000 L CNN
-F 1 "10U" H 5075 2500 50  0000 L CNN
+F 1 "220U" H 5075 2500 50  0000 L CNN
 F 2 "" H 5025 2600 60  0001 C CNN
 F 3 "" H 5025 2600 60  0001 C CNN
@@
 P 4525 3000
 F 0 "C2" V 4625 3075 50  0000 L CNN
-F 1 "10U" V 4625 2825 50  0000 L CNN
+F 1 "220U" V 4625 2725 50  0000 L CNN
 F 2 "" H 4525 3000 60  0001 C CNN
 F 3 "" H 4525 3000 60  0001 C CNN
