File: JK330-1-BF/_autosave-JK330-1-BF.kicad_pcb (KiCad board)
At the start: 2 copper layers, 280 parts, among them K1 CONN_2, K10 COLONETTE, K11 CONN_3, K2 CONN_2, K3 CONN_3, K5 COLONETTE, K6 COLONETTE, K7 COLONETTE, K8 COLONETTE, K9 COLONETTE, P1 U.FL, P2 U.FL, P3 U.FL, P4 CONN_5, P5 HE10-16, P6 CONN_6, P7 CAVALIER, P8 CAVALIER, Q1 BC847, Q2 BC847, Q3 BSP250, Q4 BC847, Q5 BSP250, U1 MF10, U10 TDA2003, U2 74HC4059, U3 74HC377, U4 74HC74, U5 16Mhz, U6 MC33172, U7 MF10, U8 74HC4059, U9 74HC377

Commit message: Ajout carte power
Parts:
- removed the C1 at (108.8, 141.9)
- removed the C10 at (91.1, 117.0)
- removed the C11 at (92.3, 120.5)
- removed the C12 at (69.5, 123.6)
- removed the C13 at (76.8, 138.0)
- removed the C14 at (71.0, 119.3)
- removed the C15 at (78.6, 102.5)
- removed the C16 at (67.7, 86.2)
- removed the C17 at (106.8, 84.5)
- removed the C18 at (89.5, 110.6)
- removed the C19 at (89.8, 106.8)
- removed the C2 at (113.9, 141.9)
- removed the C20 at (93.9, 83.2)
- removed the C21 at (89.3, 90.8)
- removed the C22 at (99.9, 99.4)
- removed the C23 at (76.6, 88.3)
- removed the C24 at (77.1, 53.2)
- removed the C25 at (95.1, 51.2)
- removed the C26 at (99.4, 51.9)
- removed the C27 at (108.1, 70.5)
- removed the C28 at (105.5, 77.9)
- removed the C29 at (102.2, 44.1)
- removed the C3 at (112.0, 161.5)
- removed the C30 at (97.4, 42.0)
- removed the C31 at (104.3, 58.8)
- removed the C32 at (107.1, 64.9)
- removed the C33 at (73.0, 148.5)
- removed the C34 at (89.0, 148.5)
- removed the C35 at (83.2, 148.5)
- removed the C4 at (105.7, 155.2)
- removed the C5 at (112.0, 153.3)
- removed the C6 at (118.7, 139.6)
- removed the C7 at (104.4, 120.5)
- removed the C8 at (89.3, 139.8)
- removed the C9 at (92.3, 135.8)
- removed the D1 at (108.8, 160.3)
- removed the D2 at (108.8, 154.6)
- removed the D3 at (99.4, 69.7)
- removed the D4 at (97.2, 69.7)
- removed the D5 at (94.6, 69.7)
- removed the D6 at (92.3, 69.7)
- removed the D7 at (89.8, 69.7)
- removed the D8 at (71.0, 168.3)
- removed the D9 at (67.9, 168.3)
- removed the K1 at (114.2, 73.0)
- removed the K10 at (117.5, 115.2)
- removed the K11 at (114.4, 84.5)
- removed the K2 at (103.3, 34.7)
- removed the K3 at (74.8, 170.1)
- removed the K5 at (117.7, 34.9)
- removed the K6 at (60.3, 34.9)
- removed the K7 at (60.6, 170.6)
- removed the K8 at (60.3, 80.4)
- removed the K9 at (117.7, 170.3)
- removed the MX1 at (99.3, 157.7)
- removed the P1 at (117.1, 160.9)
- removed the P2 at (117.1, 152.7)
- removed the P3 at (97.4, 171.1)
- removed the P4 at (117.5, 131.4)
- removed the P5 at (80.1, 34.7)
- removed the P6 at (60.6, 128.7)
- removed the P7 at (103.8, 129.4)
- removed the P8 at (112.4, 101.0)
- removed the Q1 at (65.9, 143.4)
- removed the Q2 at (69.7, 141.1)
- removed the Q3 at (74.5, 158.1)
- removed the Q4 at (78.6, 142.1)
- removed the Q5 at (84.2, 158.1)
- removed the R1 at (108.8, 165.4)
- removed the R10 at (99.9, 119.3)
- removed the R11 at (98.7, 137.0)
- removed the R12 at (98.2, 119.3)
- removed the R13 at (99.3, 139.6)
- removed the R14 at (85.0, 133.0)
- removed the R15 at (85.0, 131.7)
- removed the R16 at (85.0, 130.4)
- removed the R17 at (85.0, 129.2)
- removed the R18 at (85.0, 127.9)
- removed the R19 at (85.0, 126.6)
- removed the R2 at (112.0, 157.7)
- removed the R20 at (85.0, 125.3)
- removed the R21 at (85.0, 124.1)
- removed the R22 at (104.3, 106.3)
- removed the R23 at (108.6, 106.3)
- removed the R24 at (106.0, 106.3)
- removed the R25 at (108.6, 101.7)
- removed the R26 at (100.7, 93.3)
- removed the R27 at (103.8, 93.3)
- removed the R28 at (100.7, 91.6)
- removed the R29 at (104.5, 90.3)
- removed the R3 at (108.8, 150.1)
- removed the R30 at (101.2, 111.1)
- removed the R31 at (98.2, 90.8)
- removed the R32 at (99.4, 111.1)
- removed the R33 at (96.4, 90.8)
- removed the R34 at (97.7, 111.1)
- removed the R35 at (94.6, 90.8)
- removed the R36 at (106.0, 110.1)
- removed the R37 at (85.0, 83.7)
- removed the R38 at (85.0, 82.4)
- removed the R39 at (85.0, 81.2)
- removed the R4 at (119.5, 144.1)
- removed the R40 at (85.0, 79.9)
- removed the R41 at (85.0, 78.6)
- removed the R42 at (85.0, 77.3)
- removed the R43 at (85.0, 76.1)
- removed the R44 at (85.0, 74.5)
- removed the R45 at (94.4, 42.0)
- removed the R46 at (104.3, 62.9)
- removed the R47 at (104.3, 60.8)
- removed the R48 at (107.1, 61.6)
- removed the R49 at (64.1, 146.7)
- removed the R5 at (61.8, 144.1)
- removed the R50 at (65.9, 146.7)
- removed the R51 at (67.7, 146.7)
- removed the R52 at (77.1, 150.2)
- removed the R53 at (61.8, 142.1)
- removed the R54 at (79.1, 150.2)
- removed the R55 at (99.4, 66.7)
- removed the R56 at (97.2, 66.7)
- removed the R57 at (94.6, 66.7)
- removed the R58 at (92.3, 66.7)
- removed the R59 at (89.8, 66.7)
- removed the R6 at (104.4, 137.0)
- removed the R60 at (71.0, 165.0)
- removed the R61 at (67.9, 165.0)
- removed the R7 at (102.5, 137.0)
- removed the R8 at (101.7, 119.3)
- removed the R9 at (100.6, 137.0)
- removed the RVAR1 at (101.9, 141.2)
- removed the U1 at (95.5, 128.1)
- removed the U10 at (111.1, 54.0)
- removed the U2 at (76.7, 128.5)
- removed the U3 at (76.7, 111.4)
- removed the U4 at (79.1, 95.9)
- removed the U5 at (64.9, 95.6)
- removed the U6 at (103.8, 99.7)
- removed the U7 at (92.3, 99.7)
- removed the U8 at (76.8, 79.1)
- removed the U9 at (76.8, 60.8)
Routing:
- net (no net): track 4.78 -> 2445.8 mm, vias 8 -> 4
- net GND: track 1481.2 -> 740.6 mm, vias 44 -> 22
- net +5VD: track 863.0 -> 431.5 mm, vias 24 -> 12
- net +12V: track 539.7 -> 269.9 mm, vias 18 -> 9
- net +3.3V: track 373.7 -> 186.9 mm, vias 2 -> 1
- net +5VA: track 342.6 -> 171.3 mm, vias 8 -> 4
- net -5VA: track 327.1 -> 163.5 mm, vias 12 -> 6
- net /BD7: track 246.3 -> 123.1 mm, vias 4 -> 2
- net /HP/HP1: track 239.6 -> 119.8 mm, vias 2 -> 1
- net /BD0: track 229.8 -> 114.9 mm, vias 4 -> 2
- net /BD1: track 216.6 -> 108.3 mm, vias 4 -> 2
- net /BD6: track 205.8 -> 102.9 mm, vias 4 -> 2
- net /BD2: track 195.7 -> 97.9 mm, vias 4 -> 2
- net /BD4: track 194.1 -> 97.1 mm, vias 4 -> 2
- net /BD3: track 182.2 -> 91.1 mm, vias 4 -> 2
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
Commit message: MAJ
Parts:
- added C1: 10U, SM2112L, B.Cu at (108.8, 141.9)
- added C10: 10U, SM2112L, B.Cu at (91.1, 117.0)
- added C11: 100n, SM0603_Capa, B.Cu at (92.3, 120.5)
- added C12: 100n, SM0603_Capa, B.Cu at (69.5, 123.6)
- added C13: C, SM0603_Capa, B.Cu at (76.8, 138.0)
- added C14: 100n, SM0603_Capa, B.Cu at (71.0, 119.3)
- added C15: C, SM0603_Capa, B.Cu at (78.6, 102.5)
- added C16: 100n, SM0603_Capa, B.Cu at (67.7, 86.2)
- added C17: C, SM0603_Capa, B.Cu at (106.8, 84.5)
- added C18: CP, SM2112L, B.Cu at (89.5, 110.6)
- added C19: 100n, SM0603_Capa, B.Cu at (89.8, 106.8)
- added C2: 10U, SM2112L, B.Cu at (113.9, 141.9)
- added C20: CP, SM2112L, B.Cu at (93.9, 83.2)
- added C21: 100n, SM0603_Capa, B.Cu at (89.3, 90.8)
- added C22: 100n, SM0603_Capa, B.Cu at (99.9, 99.4)
- added C23: 100n, SM0603_Capa, B.Cu at (76.6, 88.3)
- added C24: 100n, SM0603_Capa, B.Cu at (77.1, 53.2)
- added C25: 1000U, SM2112L, B.Cu at (95.1, 51.2)
- added C26: 100n, SM0603_Capa, B.Cu at (99.4, 51.9)
- added C27: 470p, SM0603_Capa, B.Cu at (108.1, 70.5)
- added C28: 15n, SM2112L, B.Cu at (105.5, 77.9)
- added C29: 470U, SM2112L, B.Cu at (102.2, 44.1)
- added C3: 1n, SM0603_Capa, B.Cu at (112.0, 161.5)
- added C30: 100n, SM0603_Capa, B.Cu at (97.4, 42.0)
- added C31: 100u, SM0603_Capa, B.Cu at (104.3, 58.8)
- added C32: NC, SM0603_Capa, B.Cu at (107.1, 64.9)
- added C33: CP, SM2112L, B.Cu at (73.0, 148.5)
- added C34: CP, SM2112L, B.Cu at (89.0, 148.5)
- added C35: CP, SM2112L, B.Cu at (83.2, 148.5)
- added C4: 1n, SM0603_Capa, B.Cu at (105.7, 155.2)
- added C5: 1n, SM0603_Capa, B.Cu at (112.0, 153.3)
- added C6: C, SM0603_Capa, B.Cu at (118.7, 139.6)
- added C7: 1U, SM1206, B.Cu at (104.4, 120.5)
- added C8: 10U, SM2112L, B.Cu at (89.3, 139.8)
- added C9: 100n, SM0603_Capa, B.Cu at (92.3, 135.8)
- added D1: MA4P1250, SM1206, B.Cu at (108.8, 160.3)
- added D2: MA4P1250, SM1206, B.Cu at (108.8, 154.6)
- added D3: LED, SM0603, B.Cu at (99.4, 69.7)
- added D4: LED, SM0603, B.Cu at (97.2, 69.7)
- added D5: LED, SM0603, B.Cu at (94.6, 69.7)
- added D6: LED, SM0603, B.Cu at (92.3, 69.7)
- added D7: LED, SM0603, B.Cu at (89.8, 69.7)
- added D8: LED, SM0603, B.Cu at (71.0, 168.3)
- added D9: LED, SM0603, B.Cu at (67.9, 168.3)
- added K1: CONN_2, KK-2, B.Cu at (114.2, 73.0)
- added K10: COLONETTE, COLONETTE, B.Cu at (117.5, 115.2)
- added K11: CONN_3, KK-3, B.Cu at (114.4, 84.5)
- added K2: CONN_2, KK-2, B.Cu at (103.3, 34.7)
- added K3: CONN_3, KK-3, B.Cu at (74.8, 170.1)
- added K5: COLONETTE, COLONETTE, B.Cu at (117.7, 34.9)
- added K6: COLONETTE, COLONETTE, B.Cu at (60.3, 34.9)
- added K7: COLONETTE, COLONETTE, B.Cu at (60.6, 170.6)
- added K8: COLONETTE, COLONETTE, B.Cu at (60.3, 80.4)
- added K9: COLONETTE, COLONETTE, B.Cu at (117.7, 170.3)
- added MX1: SBL-1, SBL1, B.Cu at (99.3, 157.7)
- added P1: U.FL, UFL, B.Cu at (117.1, 160.9)
- added P2: U.FL, UFL, B.Cu at (117.1, 152.7)
- added P3: U.FL, UFL, B.Cu at (97.4, 171.1)
- added P4: CONN_5, KK-5, B.Cu at (117.5, 131.4)
- added P5: HE10-16, he10-16d, B.Cu at (80.1, 34.7)
- added P6: CONN_6, KK-6, B.Cu at (60.6, 128.7)
- added P7: CAVALIER, CAVALIER, B.Cu at (103.8, 129.4)
- added P8: CAVALIER, CAVALIER, B.Cu at (112.4, 101.0)
- added Q1: BC847, SOT23EBC, B.Cu at (65.9, 143.4)
- added Q2: BC847, SOT23EBC, B.Cu at (69.7, 141.1)
- added Q3: BSP250, SOT223, B.Cu at (74.5, 158.1)
- added Q4: BC847, SOT23EBC, B.Cu at (78.6, 142.1)
- added Q5: BSP250, SOT223, B.Cu at (84.2, 158.1)
- added R1: 1k, SM0603_Resistor, B.Cu at (108.8, 165.4)
- added R10: 10k, SM0603_Resistor, B.Cu at (99.9, 119.3)
- added R11: 39k//39k, SM0603_Resistor, B.Cu at (98.7, 137.0)
- added R12: 39k//39k, SM0603_Resistor, B.Cu at (98.2, 119.3)
- added R13: 10k, SM0603_Resistor, B.Cu at (99.3, 139.6)
- added R14: 10k, SM0603_Resistor, B.Cu at (85.0, 133.0)
- added R15: 10k, SM0603_Resistor, B.Cu at (85.0, 131.7)
- added R16: 10k, SM0603_Resistor, B.Cu at (85.0, 130.4)
- added R17: 10k, SM0603_Resistor, B.Cu at (85.0, 129.2)
- added R18: 10k, SM0603_Resistor, B.Cu at (85.0, 127.9)
- added R19: 10k, SM0603_Resistor, B.Cu at (85.0, 126.6)
- added R2: 1k, SM0603_Resistor, B.Cu at (112.0, 157.7)
- added R20: 10k, SM0603_Resistor, B.Cu at (85.0, 125.3)
- added R21: 10k, SM0603_Resistor, B.Cu at (85.0, 124.1)
- added R22: 11.5k, SM0603_Resistor, B.Cu at (104.3, 106.3)
- added R23: 11.5k, SM0603_Resistor, B.Cu at (108.6, 106.3)
- added R24: 11.5k, SM0603_Resistor, B.Cu at (106.0, 106.3)
- added R25: 11.5k, SM0603_Resistor, B.Cu at (108.6, 101.7)
- added R26: 11.5k, SM0603_Resistor, B.Cu at (100.7, 93.3)
- added R27: 11k5, SM0603_Resistor, B.Cu at (103.8, 93.3)
- added R28: 11k5, SM0603_Resistor, B.Cu at (100.7, 91.6)
- added R29: R, SM0603_Resistor, B.Cu at (104.5, 90.3)
- added R3: 1k, SM0603_Resistor, B.Cu at (108.8, 150.1)
- added R30: 11.5k, SM0603_Resistor, B.Cu at (101.2, 111.1)
- added R31: 11.5k, SM0603_Resistor, B.Cu at (98.2, 90.8)
- added R32: 100k, SM0603_Resistor, B.Cu at (99.4, 111.1)
- added R33: 100k, SM0603_Resistor, B.Cu at (96.4, 90.8)
- added R34: 11.5k, SM0603_Resistor, B.Cu at (97.7, 111.1)
- added R35: 11.5k, SM0603_Resistor, B.Cu at (94.6, 90.8)
- added R36: 11.5k, SM0603_Resistor, B.Cu at (106.0, 110.1)
- added R37: R, SM0603_Resistor, B.Cu at (85.0, 83.7)
- added R38: R, SM0603_Resistor, B.Cu at (85.0, 82.4)
- added R39: R, SM0603_Resistor, B.Cu at (85.0, 81.2)
- added R4: R, SM0603_Resistor, B.Cu at (119.5, 144.1)
- added R40: R, SM0603_Resistor, B.Cu at (85.0, 79.9)
- added R41: R, SM0603_Resistor, B.Cu at (85.0, 78.6)
- added R42: R, SM0603_Resistor, B.Cu at (85.0, 77.3)
- added R43: R, SM0603_Resistor, B.Cu at (85.0, 76.1)
- added R44: R, SM0603_Resistor, B.Cu at (85.0, 74.5)
- added R45: 1, SM0603_Resistor, B.Cu at (94.4, 42.0)
- added R46: 10, SM0603_Resistor, B.Cu at (104.3, 62.9)
- added R47: 470, SM0603_Resistor, B.Cu at (104.3, 60.8)
- added R48: NC, SM0603_Resistor, B.Cu at (107.1, 61.6)
- added R49: R, SM0603_Resistor, B.Cu at (64.1, 146.7)
- added R5: R, SM0603_Resistor, B.Cu at (61.8, 144.1)
- added R50: R, SM0603_Resistor, B.Cu at (65.9, 146.7)
- added R51: R, SM0603_Resistor, B.Cu at (67.7, 146.7)
- added R52: R, SM0603_Resistor, B.Cu at (77.1, 150.2)
- added R53: R, SM0603_Resistor, B.Cu at (61.8, 142.1)
- added R54: R, SM0603_Resistor, B.Cu at (79.1, 150.2)
- added R55: 1k, SM0603_Resistor, B.Cu at (99.4, 66.7)
- added R56: 1k, SM0603_Resistor, B.Cu at (97.2, 66.7)
- added R57: 1k, SM0603_Resistor, B.Cu at (94.6, 66.7)
- added R58: 1k, SM0603_Resistor, B.Cu at (92.3, 66.7)
- added R59: 1k, SM0603_Resistor, B.Cu at (89.8, 66.7)
- added R6: 10k, SM0603_Resistor, B.Cu at (104.4, 137.0)
- added R60: 1k, SM0603_Resistor, B.Cu at (71.0, 165.0)
- added R61: 1k, SM0603_Resistor, B.Cu at (67.9, 165.0)
- added R7: 10k, SM0603_Resistor, B.Cu at (102.5, 137.0)
- added R8: 10k, SM0603_Resistor, B.Cu at (101.7, 119.3)
- added R9: 10k, SM0603_Resistor, B.Cu at (100.6, 137.0)
- added RVAR1: 100, POT_10T_T93YB, B.Cu at (101.9, 141.2)
- added U1: MF10, SO20L, B.Cu at (95.5, 128.1)
- added U10: TDA2003, TDA2003V, B.Cu at (111.1, 54.0)
- added U2: 74HC4059, SO24E, B.Cu at (76.7, 128.5)
- added U3: 74HC377, SO20L, B.Cu at (76.7, 111.4)
- added U4: 74HC74, SO14N, B.Cu at (79.1, 95.9)
- added U5: 16Mhz, XTAL_QUAD, B.Cu at (64.9, 95.6)
- added U6: MC33172, SO8E, B.Cu at (103.8, 99.7)
- added U7: MF10, SO20L, B.Cu at (92.3, 99.7)
- added U8: 74HC4059, SO24E, B.Cu at (76.8, 79.1)
- added U9: 74HC377, SO20L, B.Cu at (76.8, 60.8)
Routing:
- net (no net): track 2445.8 -> 4.78 mm, vias 4 -> 8
- net GND: track 740.6 -> 1481.2 mm, vias 22 -> 44
- net +5VD: track 431.5 -> 863.0 mm, vias 12 -> 24
- net +12V: track 269.9 -> 539.7 mm, vias 9 -> 18
- net +3.3V: track 186.9 -> 373.7 mm, vias 1 -> 2
- net +5VA: track 171.3 -> 342.6 mm, vias 4 -> 8
- net -5VA: track 163.5 -> 327.1 mm, vias 6 -> 12
- net /BD7: track 123.1 -> 246.3 mm, vias 2 -> 4
- net /HP/HP1: track 119.8 -> 239.6 mm, vias 1 -> 2
- net /BD0: track 114.9 -> 229.8 mm, vias 2 -> 4
- net /BD1: track 108.3 -> 216.6 mm, vias 2 -> 4
- net /BD6: track 102.9 -> 205.8 mm, vias 2 -> 4
- net /BD2: track 97.9 -> 195.7 mm, vias 2 -> 4
- net /BD4: track 97.1 -> 194.1 mm, vias 2 -> 4
- net /BD3: track 91.1 -> 182.2 mm, vias 2 -> 4
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