File: JK330-5-OL9/OL9Mhz.kicad_pcb (KiCad board)
At the start: 2 copper layers, 21 parts, among them K1 CONN_3, K2 CONN_2, K3 COLONETTE, K4 COLONETTE, K5 COLONETTE, K6 COLONETTE, P2 BNC, Q1 BSN20, X1 9Mhz, X2 9Mhz

Commit message: MAJ3D
Parts:
- removed the C15 at (65.3, 161.5)
- removed K1: CONN_3, SIL-3
- removed the K2 at (52.6, 177.4)
- removed the K3 at (65.3, 137.4)
- removed the K4 at (33.5, 175.5)
- removed the K5 at (33.5, 137.4)
- removed the K6 at (65.3, 175.5)
- removed the P2 at (69.7, 162.8)
- removed the Q1 at (59.6, 156.5)
- removed the X1 at (41.8, 141.2)
- removed the X2 at (32.3, 159.0)
- added ?: , SIL-3, F.Cu at (41.4, 37.8)
Routing:
- net GND: track 346.4 -> 173.2 mm, vias 2 -> 1
- net N-0000020: track 103.8 -> 51.9 mm, vias 4 -> 2
- net N-0000015: track 78.0 -> 39.0 mm, vias 2 -> 1
- net N-0000026: track 63.9 -> 31.9 mm
- net +12V: track 54.7 -> 27.4 mm, vias 2 -> 1
- net N-0000016: track 38.9 -> 19.5 mm, vias 2 -> 1
- net N-0000023: track 31.0 -> 15.5 mm
- net N-0000022: track 30.7 -> 15.4 mm
- net N-0000013: track 21.6 -> 10.8 mm
- net N-0000024: track 20.7 -> 10.3 mm
- net N-0000014: track 18.8 -> 9.40 mm, vias 2 -> 1
- net N-0000025: track 18.8 -> 9.40 mm
- net N-0000021: track 15.2 -> 7.58 mm
- net N-000005: track 13.7 -> 6.86 mm
- net N-0000019: track 13.7 -> 6.86 mm
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Other:
- board text removed: "OL 9MHZ"
- board text removed: "V0-10"
