File: LEDX4-12V/LEDX4-12V.kicad_pcb (KiCad board)
At the start: 2 copper layers, 22 parts, among them K1001 CONN_2, K1002 CONN_2

Commit message: Ajout carte power
Parts:
- moved K1002 253.9 mm to (26.7, 52.1), turned to 180 degrees
- moved K1001 250.6 mm to (31.8, 52.1), turned to 180 degrees
- moved D1001 234.1 mm to (27.9, 67.3), turned to 270 degrees
- moved R1005 221.7 mm to (24.1, 80.0), turned to 270 degrees
- moved R1001 219.7 mm to (26.7, 80.0), turned to 270 degrees
- moved R1006 217.8 mm to (29.2, 80.0), turned to 270 degrees
- moved R1007 215.9 mm to (31.8, 80.0), turned to 270 degrees
- moved D1002 203.8 mm to (27.9, 92.7), turned to 270 degrees
- moved R1010 192.7 mm to (24.1, 105.4), turned to 270 degrees
- moved R1008 190.5 mm to (26.7, 105.4), turned to 270 degrees
- moved R1002 188.2 mm to (29.2, 105.4), turned to 270 degrees
- moved R1009 186.1 mm to (31.8, 105.4), turned to 270 degrees
- moved D1003 175.6 mm to (27.9, 118.1), turned to 270 degrees
- moved R1013 166.5 mm to (24.1, 130.8), turned to 270 degrees
- moved R1012 163.9 mm to (26.7, 130.8), turned to 270 degrees
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