File: LEDX4-12V/LEDX4-12V.sch (KiCad schematic (older format))
At the start: 22 parts, among them K1001 CONN_2, K1002 CONN_2

Commit message: Ajout carte power
Parts:
- R1001, R1002, R1003, R1004, R1005, R1006, R1007, R1008, R1009, R1010, R1011, R1012, R1013, R1014, R1015, R1016: value R -> 10
Changed lines of the file:
@@
 U 1 1 51D1D70F
 P 3950 2950
-F 0 "R1001" V 3900 3050 50  0000 C CNN
-F 1 "R" V 4000 3050 50  0000 C CNN
+F 0 "R1001" V 4000 2850 50  0000 C CNN
+F 1 "10" V 3900 2850 50  0000 C CNN
 F 2 "" H 3950 2950 60  0000 C CNN
 F 3 "" H 3950 2950 60  0000 C CNN
@@
 U 1 1 51D1D71E
 P 4950 2950
-F 0 "R1002" V 4900 3050 50  0000 C CNN
-F 1 "R" V 5000 3050 50  0000 C CNN
+F 0 "R1002" V 5000 2850 50  0000 C CNN
+F 1 "10" V 4900 2850 50  0000 C CNN
 F 2 "" H 4950 2950 60  0000 C CNN
 F 3 "" H 4950 2950 60  0000 C CNN
@@
 U 1 1 51D1D72D
 P 5950 2950
-F 0 "R1003" V 5900 3050 50  0000 C CNN
-F 1 "R" V 6000 3050 50  0000 C CNN
+F 0 "R1003" V 6000 2850 50  0000 C CNN
+F 1 "10" V 5900 2850 50  0000 C CNN
 F 2 "" H 5950 2950 60  0000 C CNN
 F 3 "" H 5950 2950 60  0000 C CNN
@@
 U 1 1 51D1D75A
 P 7050 2950
-F 0 "R1004" V 7000 3050 50  0000 C CNN
-F 1 "R" V 7100 3050 50  0000 C CNN
+F 0 "R1004" V 7100 2850 50  0000 C CNN
+F 1 "10" V 7000 2850 50  0000 C CNN
 F 2 "" H 7050 2950 60  0000 C CNN
 F 3 "" H 7050 2950 60  0000 C CNN
@@
 U 1 1 51D32E65
 P 4950 2750
-F 0 "R1010" V 4900 2850 50  0000 C CNN
-F 1 "R" V 5000 2850 50  0000 C CNN
+F 0 "R1010" V 5000 2650 50  0000 C CNN
+F 1 "10" V 4900 2650 50  0000 C CNN
 F 2 "" H 4950 2750 60  0000 C CNN
 F 3 "" H 4950 2750 60  0000 C CNN
@@
 U 1 1 51D32E72
 P 4950 2550
-F 0 "R1009" V 4900 2650 50  0000 C CNN
-F 1 "R" V 5000 2650 50  0000 C CNN
+F 0 "R1009" V 5000 2450 50  0000 C CNN
+F 1 "10" V 4900 2450 50  0000 C CNN
 F 2 "" H 4950 2550 60  0000 C CNN
 F 3 "" H 4950 2550 60  0000 C CNN
@@
 U 1 1 51D32E78
 P 4950 2350
-F 0 "R1008" V 4900 2450 50  0000 C CNN
-F 1 "R" V 5000 2450 50  0000 C CNN
+F 0 "R1008" V 5000 2250 50  0000 C CNN
+F 1 "10" V 4900 2250 50  0000 C CNN
 F 2 "" H 4950 2350 60  0000 C CNN
 F 3 "" H 4950 2350 60  0000 C CNN
@@
 U 1 1 51D32E7E
 P 5950 2750
-F 0 "R1013" V 5900 2850 50  0000 C CNN
-F 1 "R" V 6000 2850 50  0000 C CNN
+F 0 "R1013" V 6000 2650 50  0000 C CNN
+F 1 "10" V 5900 2650 50  0000 C CNN
 F 2 "" H 5950 2750 60  0000 C CNN
 F 3 "" H 5950 2750 60  0000 C CNN
@@
 U 1 1 51D32E84
 P 5950 2550
-F 0 "R1012" V 5900 2650 50  0000 C CNN
-F 1 "R" V 6000 2650 50  0000 C CNN
+F 0 "R1012" V 6000 2450 50  0000 C CNN
+F 1 "10" V 5900 2450 50  0000 C CNN
 F 2 "" H 5950 2550 60  0000 C CNN
 F 3 "" H 5950 2550 60  0000 C CNN
@@
 U 1 1 51D32E8A
 P 3950 2750
-F 0 "R1007" V 3900 2850 50  0000 C CNN
-F 1 "R" V 4000 2850 50  0000 C CNN
+F 0 "R1007" V 4000 2650 50  0000 C CNN
+F 1 "10" V 3900 2650 50  0000 C CNN
 F 2 "" H 3950 2750 60  0000 C CNN
 F 3 "" H 3950 2750 60  0000 C CNN
@@
 U 1 1 51D32E90
 P 3950 2550
-F 0 "R1006" V 3900 2650 50  0000 C CNN
-F 1 "R" V 4000 2650 50  0000 C CNN
+F 0 "R1006" V 4000 2450 50  0000 C CNN
+F 1 "10" V 3900 2450 50  0000 C CNN
 F 2 "" H 3950 2550 60  0000 C CNN
 F 3 "" H 3950 2550 60  0000 C CNN
@@
 U 1 1 51D32E96
 P 3950 2350
-F 0 "R1005" V 3900 2450 50  0000 C CNN
-F 1 "R" V 4000 2450 50  0000 C CNN
+F 0 "R1005" V 4000 2250 50  0000 C CNN
+F 1 "10" V 3900 2250 50  0000 C CNN
 F 2 "" H 3950 2350 60  0000 C CNN
 F 3 "" H 3950 2350 60  0000 C CNN
@@
 U 1 1 51D32E9C
 P 5950 2350
-F 0 "R1011" V 5900 2450 50  0000 C CNN
-F 1 "R" V 6000 2450 50  0000 C CNN
+F 0 "R1011" V 6000 2250 50  0000 C CNN
+F 1 "10" V 5900 2250 50  0000 C CNN
 F 2 "" H 5950 2350 60  0000 C CNN
 F 3 "" H 5950 2350 60  0000 C CNN
@@
 U 1 1 51D32EA2
 P 7050 2750
-F 0 "R1016" V 7000 2850 50  0000 C CNN
-F 1 "R" V 7100 2850 50  0000 C CNN
+F 0 "R1016" V 7100 2650 50  0000 C CNN
+F 1 "10" V 7000 2650 50  0000 C CNN
 F 2 "" H 7050 2750 60  0000 C CNN
 F 3 "" H 7050 2750 60  0000 C CNN
@@
 U 1 1 51D32EA8
 P 7050 2550
-F 0 "R1015" V 7000 2650 50  0000 C CNN
-F 1 "R" V 7100 2650 50  0000 C CNN
+F 0 "R1015" V 7100 2450 50  0000 C CNN
+F 1 "10" V 7000 2450 50  0000 C CNN
 F 2 "" H 7050 2550 60  0000 C CNN
 F 3 "" H 7050 2550 60  0000 C CNN
@@
 U 1 1 51D32EAE
 P 7050 2350
-F 0 "R1014" V 7000 2450 50  0000 C CNN
-F 1 "R" V 7100 2450 50  0000 C CNN
+F 0 "R1014" V 7100 2250 50  0000 C CNN
+F 1 "10" V 7000 2250 50  0000 C CNN
 F 2 "" H 7050 2350 60  0000 C CNN
 F 3 "" H 7050 2350 60  0000 C CNN
