File: JK330-9-POWER/JK330-9-POWER.kicad_pcb (KiCad board)
At the start: 2 copper layers, 55 parts, among them P1001 CONN_6, P1002 CONN_6, P1003 CONN_6, P1004 CONN_6, P1005 CONN_6, P1006 CONN_6, P1007 CONN_6, P1008 CONN_6, P1009 CONN_6, P1010 CONN_6, P1011 CONN_6, P1012 CONN_6, U1001 EC3A04

Commit message: POWER
Parts:
- removed P1011, P1012: CONN_6, WEIDMULLER6
- added C1011: 10U/10V, SM1812L, F.Cu at (-58.7, 33.7)
- added C1012: 10n, SM0603_Capa, F.Cu at (0.00, 0.00)
- added K1001: CONN_2, WEIDMULLER2-508, F.Cu at (-38.9, 37.2)
- added K1002: CONN_2, KK-2, F.Cu at (-31.5, 70.2)
- added L1001: 10U/3.4A 30%, SELFCMS2, F.Cu at (12.3, 82.0)
- added L1002: 10U/3.4A 30%, SELFCMS2, F.Cu at (5.97, 72.5)
- added R1013, R1014, R1015, R1016: NC, SM0603_Resistor, F.Cu at (0.00, 0.00)
- added U1002: MP2307, SO8N, F.Cu at (82.7, 58.0)
- added U1003: MP2307, SO8N, F.Cu at (90.2, 58.4)
- added U1004: LM1117, DPAK2, F.Cu at (72.8, -0.51)
- C1003: value 10U/10V -> 10µ/16V; footprint SM1812L -> SM2112L
- C1004: value 100n -> 10µ/16V; footprint SM0603_Capa -> SM2112L
- C1005: value 100n -> 10U/10V; footprint SM0603_Capa -> SM1812L
- C1006, C1016: value 3.3n -> 100n
- C1007, C1025, C1026: value 10U/10V -> 100n; footprint SM1812L -> SM0603_Capa
- C1008, C1017: value 10n -> 100n
- C1009: value 100p -> 3.3n
- C1010: value 100n -> 3.3n
- C1013: value 10µ/16V -> 10n; footprint SM2112L -> SM0603_Capa
- C1014: value 10µ/16V -> 100p; footprint SM2112L -> SM0603_Capa
- C1015: value 100n -> 100p
- C1018: value 100p -> 100n
- C1019, C1020: value 22U/16V -> 10U/10V; footprint SM2112L -> SM1812L
- C1021, C1023: value 100n -> 22U/10V; footprint SM0603_Capa -> SM2112L
- C1022, C1024: value 100n -> 22U/16V; footprint SM0603_Capa -> SM2112L
- P1001, P1002, P1003, P1004, P1005, P1006, P1007, P1008, P1009, P1010: value CONN_6 -> CONN_7; footprint WEIDMULLER6 -> PHONCONT-7-D-3-81
- R1001: value 100k -> 3.3k; footprint WEIDMULLER8 -> SM0603_Resistor
- R1002: value 45.3k 1% -> 3.3k
- R1003: value 10k 1% -> 1k
- R1004, R1005: value 3.3k -> 1k
- R1006: value 1k -> 470
- R1007, R1008: value 1k -> 100k
- R1009: value 470 -> 45.3k 1%
- R1010: value 100k -> 10k 1%
- moved P1006 101.4 mm to (-28.8, 8.00)
- moved P1004 81.3 mm to (63.9, 27.7)
- moved P1008 74.7 mm to (95.5, -23.5)
- moved C1005 72.8 mm to (-60.7, 40.1)
- moved C1020 66.8 mm to (-60.7, 27.9)
- moved C1019 63.6 mm to (-59.7, 21.8)
- moved P1007 62.6 mm to (6.99, -29.2)
- moved P1005 60.6 mm to (-11.2, 39.2)
- moved R1001 57.1 mm to (0.00, 0.00)
- moved P1002 55.8 mm to (-31.1, -17.7)
- moved P1009 37.7 mm to (41.5, -5.08)
- moved P1010 37.4 mm to (31.9, 34.2)
- moved P1003 34.0 mm to (45.0, 55.4)
- moved U1001 29.2 mm to (88.4, 23.9)
- moved C1021 29.0 mm to (14.9, 24.9)
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Connections:
- C1003 pad 1: +5VD -> +BATT
- C1004 pad 1: N-0000019 -> +BATT
- C1006 pad 1: N-0000031 -> N-0000020
- C1007 pad 1: +3.3V -> N-0000028
- C1008 pad 1: N-0000015 -> +5VD
- C1008 pad 2: N-0000016 -> GND
- C1009 pad 1: N-0000031 -> N-0000012
- C1010 pad 1: +3.3V -> N-0000030
- C1013 pad 1: +BATT -> N-0000029
- C1013 pad 2: GND -> N-0000031
- C1014 pad 1: +BATT -> N-0000012
- C1015 pad 1: N-0000032 (its old number) -> N-0000030
- C1016 pad 1: N-0000027 -> +3.3V
- C1017 pad 1: N-0000030 -> +5VA
- C1017 pad 2: N-0000029 -> GND
- C1018 pad 1: N-0000027 -> GND
- C1018 pad 2: GND -> -5VA
- C1019 pad 1: +12V -> +5VA
- C1020 pad 1: +12V -> GND
- C1020 pad 2: GND -> -5VA
- C1023 pad 1: +5VA -> +5VD
- C1024 pad 1: GND -> +12V
- C1024 pad 2: -5VA -> GND
- C1025 pad 1: +5VA -> +5VD
- C1026 pad 1: GND -> +12V
- C1026 pad 2: -5VA -> GND
- D1001 pad 2: N-0000014 -> N-000008
- D1002 pad 2: N-000009 -> N-0000026
- D1003 pad 1: (no net) -> +5VA
- D1003 pad 2: N-0000010 -> N-0000027
- D1004 pad 2: N-000008 -> N-0000024
- D1005 pad 2: N-0000011 -> N-0000025
- D1006 pad 2: N-0000012 -> N-0000023
- R1001 pad 1: N-0000018 -> N-000008
- R1001 pad 2: +BATT -> GND
- R1002 pad 1: +5VD -> N-0000026
- R1002 pad 2: N-0000017 -> GND
- R1003 pad 1: N-0000017 -> N-0000027
- R1004 pad 1: N-0000014 -> N-0000024
- R1005 pad 1: N-000009 -> N-0000025
- R1006 pad 1: N-0000010 -> N-0000023
- R1007 pad 1: N-000008 -> N-0000022
- R1007 pad 2: GND -> +BATT
- R1008 pad 1: N-0000011 -> N-0000021
- R1008 pad 2: GND -> +BATT
- R1009 pad 1: N-0000012 -> +5VD
- R1009 pad 2: GND -> N-0000010
- R1010 pad 1: N-0000033 -> N-0000010
- R1010 pad 2: +BATT -> GND

Commit message: MAJ  mineur
Parts:
- removed K1002: CONN_2, KK-2
- added COLONETTE: VAL**, COLONETTE, F.Cu at (136.8, 137.5)
- added COLONETTE: VAL**, COLONETTE, F.Cu at (278.1, 138.2)
- added COLONETTE: VAL**, COLONETTE, F.Cu at (137.7, 79.9)
- added COLONETTE: VAL**, COLONETTE, F.Cu at (277.7, 79.5)
- added COLONETTE: VAL**, COLONETTE, F.Cu at (209.3, 79.2)
- added K1003: CONN_2, WEIDMULLER2-508, F.Cu at (239.1, 79.0)
- L1001, L1002: footprint SELFCMS2 -> SELF10
- U1002, U1003: footprint SO8N -> SO8_WITH_EP
- moved C1025 300.0 mm to (275.8, 117.9)
- moved R1014 298.0 mm to (271.9, 121.9), turned to 90 degrees
- moved R1013 296.5 mm to (270.3, 121.9), turned to 90 degrees
- moved R1009 294.9 mm to (268.5, 121.9), turned to 90 degrees
- moved R1010 294.3 mm to (269.4, 118.6), turned to 90 degrees
- moved K1001 293.9 mm to (252.1, 79.0), turned to 180 degrees
- moved C1023 288.1 mm to (278.4, 128.4)
- moved C1006 287.3 mm to (262.6, 116.5), turned to 90 degrees
- moved C1014 285.7 mm to (260.9, 116.5), turned to 90 degrees
- moved C1011 284.4 mm to (208.5, 131.1), turned to 90 degrees
- moved C1012 283.0 mm to (253.7, 125.2), turned to 180 degrees
- moved R1008 282.4 mm to (257.3, 116.5), turned to 90 degrees
- moved C1005 281.5 mm to (208.5, 122.2), turned to 270 degrees
- moved C1009 281.3 mm to (259.1, 116.5), turned to 90 degrees
- moved C1021 280.8 mm to (278.3, 122.3)
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Connections:
- K1001 pad 2: +BATT -> N-000009
Routing:
- net GND: track 0.00 -> 451.4 mm, vias 0 -> 23
- net +BATT: track 0.00 -> 332.5 mm, vias 0 -> 3
- net +3.3V: track 0.00 -> 281.7 mm, vias 0 -> 2
- net -5VA: track 0.00 -> 274.0 mm, vias 0 -> 3
- net +12V: track 0.00 -> 264.8 mm, vias 0 -> 2
- net +5VA: track 0.00 -> 256.7 mm, vias 0 -> 2
- net +5VD: track 0.00 -> 246.7 mm, vias 0 -> 1
- net N-0000032: track 0.00 -> 39.7 mm, vias 0 -> 2
- net N-0000033: track 0.00 -> 16.4 mm
- net N-0000030: track 0.00 -> 16.1 mm, vias 0 -> 2
- net N-0000023: track 0.00 -> 4.19 mm
- net N-0000029: track 0.00 -> 2.55 mm
- net N-0000031: track 0.00 -> 2.52 mm
- net N-000008: track 0.00 -> 1.66 mm
- net N-0000028: track 0.00 -> 1.66 mm
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- added copper zone on F.Cu, net +3.3V
Other:
- net class Default: via_dia 0.889 -> 1.3; via_drill 0.635 -> 0.6
- board text added: "ARRET URGENCE"
- board text added: "BATT"

Commit message: POWER PCB OK
Parts:
- moved C1023 79.0 mm to (211.8, 85.9)
- moved C1025 75.3 mm to (210.1, 81.3)
- moved C1021 72.9 mm to (211.8, 92.2)
- moved C1024 69.6 mm to (178.3, 117.9)
- moved L1002 69.3 mm to (167.9, 120.7)
- moved C1003 68.7 mm to (155.7, 114.3)
- moved C1001 68.6 mm to (155.7, 120.7)
- moved R1014 68.0 mm to (208.5, 97.3), turned to 180 degrees
- moved C1006 66.8 mm to (198.6, 97.4)
- moved C1002 66.8 mm to (187.7, 120.3)
- moved C1004 66.8 mm to (187.7, 114.3)
- moved C1008 66.8 mm to (140.5, 104.9)
- moved C1012 66.8 mm to (189.7, 106.2)
- moved C1014 66.8 mm to (196.8, 97.4)
- moved C1016 66.8 mm to (140.5, 110.2)
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Routing:
- net +5VD: track 246.7 -> 401.6 mm, vias 1 -> 3
- net GND: track 451.4 -> 562.4 mm, vias 23 -> 26
- net +BATT: track 332.5 -> 367.5 mm
- net +3.3V: track 281.7 -> 314.6 mm, vias 2 -> 3
- net N-0000010: track 0.00 -> 20.6 mm, vias 0 -> 2
- net +5VA: track 256.7 -> 276.8 mm, vias 2 -> 3
- net N-0000021: track 0.00 -> 18.7 mm, vias 0 -> 2
- net N-0000011: track 0.00 -> 15.3 mm
- net +12V: track 264.8 -> 279.5 mm
- net N-0000032: track 39.7 -> 28.6 mm
- net N-000009: track 0.00 -> 8.00 mm
- net N-0000012: track 0.00 -> 3.94 mm
- net N-0000022: track 0.00 -> 2.37 mm
- net N-0000013: track 0.00 -> 2.24 mm
- added copper zone on B.Cu, net +3.3V
- added copper zone on B.Cu, net GND
- added copper zone on F.Cu, net GND
Other:
- board text added: "+12V"
- board text added: "+3.3V"
- board text added: "+5VA"
- board text added: "+5VD"
- board text added: "+BATT"
- board text added: "-5VA"
- board text added: "GND"

Commit message: MAJ TEXTE PCB
Other:
- board text added: "F4DEB JK330-9 POWER 08/13 V0-10"
Changed lines of the file:
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@@
   (general
     (links 174)
-    (no_connects 1)
-    (area 128.7526 70.040499 286.1564 149.7584)
+    (no_connects 9)
+    (area 49.912001 50.990499 225.806001 138.336)
     (thickness 1.6)
-    (drawings 11)
+    (drawings 12)
     (tracks 430)
     (zones 0)
@@
   )
   (page A4)
+  (title_block
+    (title "JK330-9 POWER")
+    (rev V0-10)
+    (company F4DEB)
+  )
   (layers
     (15 Dessus.Cu signal)
@@
   )
   (setup
-    (last_trace_width 2)
+    (last_trace_width 0.254)
     (user_trace_width 0.3)
     (user_trace_width 0.35)
@@
     )
   )
+  (gr_text "F4DEB JK330-9 POWER  08/13     V0-10" (at 109.982 61.214) (layer Dessus.Cu)
+    (effects (font (size 1.5 1.5) (thickness 0.3)))
+  )
   (dimension 69.85 (width 0.3) (layer Contours.Ci)

Commit message: MAJ pour impression
Parts:
- added C1001: 10µ/16V, SM2112L, B.Cu at (243.8, 120.9)
- added C1002: 10µ/16V, SM2112L, B.Cu at (243.5, 152.9)
- added C1003: 10µ/16V, SM2112L, B.Cu at (237.5, 120.9)
- added C1004: 10µ/16V, SM2112L, B.Cu at (237.5, 152.9)
- added C1005: 10U/10V, SM1812L, B.Cu at (226.3, 109.7)
- added C1006: 100n, SM0603_Capa, B.Cu at (220.6, 163.8)
- added C1007: 100n, SM0603_Capa, B.Cu at (220.6, 130.9)
- added C1008: 100n, SM0603_Capa, B.Cu at (228.1, 105.7)
- added C1009: 3.3n, SM0603_Capa, B.Cu at (220.6, 160.3)
- added C1010: 3.3n, SM0603_Capa, B.Cu at (220.6, 127.1)
- added C1011: 10U/10V, SM1812L, B.Cu at (235.2, 109.7)
- added C1012: 10n, SM0603_Capa, B.Cu at (229.4, 154.9)
- added C1013: 10n, SM0603_Capa, B.Cu at (229.2, 121.4)
- added C1014: 100p, SM0603_Capa, B.Cu at (220.6, 162.1)
- added C1015: 100p, SM0603_Capa, B.Cu at (220.6, 129.0)
- added C1016: 100n, SM0603_Capa, B.Cu at (233.4, 105.7)
- added C1017: 100n, SM0603_Capa, B.Cu at (220.0, 66.8)
- added C1018: 100n, SM0603_Capa, B.Cu at (220.0, 55.4)
- added C1019: 10U/10V, SM1812L, B.Cu at (223.3, 66.8)
- added C1020: 10U/10V, SM1812L, B.Cu at (223.3, 55.4)
- added C1021: 22U/10V, SM2112L, B.Cu at (215.4, 177.0)
- added C1022: 22U/16V, SM2112L, B.Cu at (221.2, 142.2)
- added C1023: 22U/10V, SM2112L, B.Cu at (209.0, 177.0)
- added C1024: 22U/16V, SM2112L, B.Cu at (241.0, 143.5)
- added C1025: 100n, SM0603_Capa, B.Cu at (204.5, 175.3)
- added C1026: 100n, SM0603_Capa, B.Cu at (227.8, 141.4)
- added COLONETTE: VAL**, COLONETTE, B.Cu at (183.4, 110.5)
- added COLONETTE: VAL**, COLONETTE, B.Cu at (183.6, 178.9)
- added COLONETTE: VAL**, COLONETTE, B.Cu at (184.0, 38.9)
- added COLONETTE: VAL**, COLONETTE, B.Cu at (242.3, 179.3)
- added COLONETTE: VAL**, COLONETTE, B.Cu at (241.7, 38.0)
- added D1001: LED, LED-0603, B.Cu at (192.5, 39.5)
- added D1002: LED, LED-0603, B.Cu at (196.3, 39.5)
- added D1003: LED, LED-0603, B.Cu at (204.0, 39.5)
- added D1004: LED, LED-0603, B.Cu at (207.8, 39.5)
- added D1005: LED, LED-0603, B.Cu at (200.2, 39.5)
- added D1006: LED, LED-0603, B.Cu at (211.6, 39.5)
- added K1001: CONN_2, WEIDMULLER2-508, B.Cu at (183.1, 153.3)
- added K1003: CONN_2, WEIDMULLER2-508, B.Cu at (183.1, 140.3)
- added L1001: 10U/3.4A 30%, SELF10, B.Cu at (231.9, 166.8)
- added L1002: 10U/3.4A 30%, SELF10, B.Cu at (243.8, 133.1)
- added P1001: CONN_7, PHONCONT-7-D-3-81, B.Cu at (204.0, 46.5)
- added P1002: CONN_7, PHONCONT-7-D-3-81, B.Cu at (204.0, 59.2)
- added P1003: CONN_7, PHONCONT-7-D-3-81, B.Cu at (204.0, 71.9)
- added P1004: CONN_7, PHONCONT-7-D-3-81, B.Cu at (204.0, 84.6)
- added P1005: CONN_7, PHONCONT-7-D-3-81, B.Cu at (204.0, 97.3)
- added P1006: CONN_7, PHONCONT-7-D-3-81, B.Cu at (204.0, 110.0)
- added P1007: CONN_7, PHONCONT-7-D-3-81, B.Cu at (204.0, 122.7)
- added P1008: CONN_7, PHONCONT-7-D-3-81, B.Cu at (204.0, 135.4)
- added P1009: CONN_7, PHONCONT-7-D-3-81, B.Cu at (204.0, 148.1)
- added P1010: CONN_7, PHONCONT-7-D-3-81, B.Cu at (204.0, 160.8)
- added R1001: 3.3k, SM0603_Resistor, B.Cu at (192.5, 36.3)
- added R1002: 3.3k, SM0603_Resistor, B.Cu at (196.3, 36.3)
- added R1003: 1k, SM0603_Resistor, B.Cu at (204.0, 36.3)
- added R1004: 1k, SM0603_Resistor, B.Cu at (207.8, 36.3)
- added R1005: 1k, SM0603_Resistor, B.Cu at (200.2, 36.3)
- added R1006: 470, SM0603_Resistor, B.Cu at (211.6, 36.3)
- added R1007: 100k, SM0603_Resistor, B.Cu at (220.6, 125.2)
- added R1008: 100k, SM0603_Resistor, B.Cu at (220.6, 158.5)
- added R1009: 45.3k 1%, SM0603_Resistor, B.Cu at (224.0, 173.7)
- added R1010: 10k 1%, SM0603_Resistor, B.Cu at (222.8, 170.6)
- added R1011: 121k 1%, SM0603_Resistor, B.Cu at (227.8, 137.7)
- added R1012: 10k 1%, SM0603_Resistor, B.Cu at (222.6, 135.9)
- added R1013: NC, SM0603_Resistor, B.Cu at (222.2, 173.7)
- added R1014: NC, SM0603_Resistor, B.Cu at (220.5, 173.7)
- added R1015: NC, SM0603_Resistor, B.Cu at (227.8, 135.9)
- added R1016: NC, SM0603_Resistor, B.Cu at (227.8, 139.4)
- added U1001: EC3A04, EC3A, B.Cu at (236.2, 59.2)
- added U1002: MP2307, SO8_WITH_EP, B.Cu at (226.2, 159.6)
- added U1003: MP2307, SO8_WITH_EP, B.Cu at (226.3, 126.5)
- added U1004: LM1117, DPAK2, B.Cu at (230.4, 100.8)
- moved COLONETTE 164.9 mm to (50.5, 37.0), turned to 90 degrees
- moved C1025 144.5 mm to (71.4, 40.6), turned to 90 degrees
- moved C1023 143.8 mm to (75.9, 38.9), turned to 90 degrees
- moved C1021 140.1 mm to (82.3, 38.9), turned to 90 degrees
- moved K1001 138.1 mm to (50.0, 62.6), turned to 270 degrees
- moved COLONETTE 133.5 mm to (109.2, 36.6), turned to 90 degrees
- moved R1014 133.1 mm to (87.4, 42.2), turned to 270 degrees
- moved R1013 132.2 mm to (89.2, 42.2), turned to 270 degrees
- moved R1009 131.4 mm to (90.9, 42.2), turned to 270 degrees
- moved R1010 127.8 mm to (89.7, 45.3), turned to 180 degrees
- moved P1010 127.3 mm to (70.9, 55.1), turned to 180 degrees
- moved K1003 126.1 mm to (50.0, 75.6), turned to 270 degrees
- moved C1006 120.0 mm to (87.5, 52.1), turned to 180 degrees
- moved L1001 118.8 mm to (98.8, 49.1), turned to 90 degrees
- moved COLONETTE 118.4 mm to (50.9, 177.0), turned to 90 degrees
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Routing:
- net GND: track 562.4 -> 1124.7 mm, vias 26 -> 52
- net +5VD: track 401.6 -> 803.2 mm, vias 3 -> 6
- net +BATT: track 367.5 -> 735.1 mm, vias 3 -> 6
- net +3.3V: track 314.6 -> 629.3 mm, vias 3 -> 6
- net +12V: track 279.5 -> 559.1 mm, vias 2 -> 4
- net +5VA: track 276.8 -> 553.6 mm, vias 3 -> 6
- net -5VA: track 274.0 -> 548.0 mm, vias 3 -> 6
- net N-0000032: track 28.6 -> 57.2 mm, vias 2 -> 4
- net N-0000010: track 20.6 -> 41.2 mm, vias 2 -> 4
- net N-0000021: track 18.7 -> 37.3 mm, vias 2 -> 4
- net N-0000033: track 16.4 -> 32.7 mm
- net N-0000030: track 16.1 -> 32.3 mm, vias 2 -> 4
- net N-0000011: track 15.3 -> 30.6 mm
- net N-000009: track 8.00 -> 16.0 mm
- net N-0000023: track 4.19 -> 8.38 mm
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
Commit message: MAJ EMPREINTE SELF
Parts:
- moved COLONETTE 150.3 mm to (246.1, 175.8)
- moved COLONETTE 144.9 mm to (245.5, 34.4)
- moved COLONETTE 143.7 mm to (187.8, 35.3)
- moved COLONETTE 87.9 mm to (187.2, 106.9)
- moved COLONETTE 65.0 mm to (187.5, 175.4)
- moved P1004 6.28 mm to (72.4, 125.2)
- moved C1005 6.28 mm to (94.7, 100.1)
- moved C1006 6.28 mm to (89.0, 46.0)
- moved C1008 6.28 mm to (96.5, 104.1)
- moved C1011 6.28 mm to (103.6, 100.1)
- moved C1012 6.28 mm to (97.8, 54.9)
- moved C1013 6.28 mm to (97.7, 88.4)
- moved C1016 6.28 mm to (101.9, 104.1)
- moved C1017 6.28 mm to (88.4, 143.0)
- moved C1018 6.28 mm to (88.4, 154.4)
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