File: JK330-9-POWER/JK330-9-POWER.sch (KiCad schematic (older format))
At the start: 64 parts, among them K1001 CONN_2, K1002 CONN_2, P1001 CONN_6, P1002 CONN_6, P1003 CONN_6, P1004 CONN_6, P1005 CONN_6, P1006 CONN_6, P1007 CONN_6, P1008 CONN_6, P1009 CONN_6, P1010 CONN_6, P1011 CONN_6, P1012 CONN_6, U1001 EC3A04, U1002 MP2307, U1003 LM1117, U1004 MP2307

Commit message: POWER
Parts:
- removed P1001, P1002, P1003, P1004, P1005, P1006, P1007, P1008, P1009, P1010, P1011, P1012: CONN_6, symbol CONN_6
- added P1001, P1002, P1003, P1004, P1005, P1006, P1007, P1008, P1009, P1010: CONN_7, ~, symbol CONN_7
- added R1013, R1014, R1015, R1016: NC, ~, symbol R
- renumbered C1013 to C1001, C1001 to C1002, C1014 to C1003, C1002 to C1004, C1003 to C1005, C1004 to C1006, C1015 to C1007, C1005 to C1008, C1006 to C1009, C1016 to C1010, C1007 to C1011, C1008 to C1012, C1017 to C1013, C1009 to C1014, C1018 to C1015, C1010 to C1016, C1023 to C1017, C1024 to C1018, C1025 to C1019, C1026 to C1020, C1011 to C1021, C1019 to C1022, C1012 to C1023, C1020 to C1024, C1021 to C1025, C1022 to C1026, R1004 to R1001, R1005 to R1002, R1006 to R1003, R1007 to R1004, R1008 to R1005, R1009 to R1006, R1010 to R1007, R1001 to R1008, R1002 to R1009, R1003 to R1010, U1004 to U1003, U1003 to U1004
Connections:
- wire segments 185 -> 191
Other:
- moved on the sheet: C1001, C1002, C1003, C1004, C1006, C1007, C1009, C1010, C1012, C1013, C1014, C1015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

Commit message: MAJ  mineur
Parts:
- removed K1002: CONN_2, ~, symbol CONN_2
- added K1003: CONN_2, ~, symbol CONN_2
Connections:
- net +BATT: now also K1003.2 (PM); no longer K1001.2 (PM)
- new net: K1001.2 (PM), K1003.1 (P1)
Changed lines of the file:
@@
 Sheet 1 1
 Title "JK330-9 POWER"
-Date "9 aug 2013"
+Date "25 aug 2013"
 Rev "V0.10"
 Comp "F4DEB"
@@
 L +BATT #PWR06
 U 1 1 51E85EF4
-P 9950 1200
-F 0 "#PWR06" H 9950 1150 20  0001 C CNN
-F 1 "+BATT" H 9950 1300 30  0000 C CNN
-F 2 "" H 9950 1200 60  0000 C CNN
-F 3 "" H 9950 1200 60  0000 C CNN
-	1    9950 1200
-	1    0    0    -1
+P 10250 1150
+F 0 "#PWR06" H 10250 1100 20  0001 C CNN
+F 1 "+BATT" H 10250 1250 30  0000 C CNN
+F 2 "" H 10250 1150 60  0000 C CNN
+F 3 "" H 10250 1150 60  0000 C CNN
+	1    10250 1150
+	0    1    1    0
 $EndComp
 $Comp
@@
 $EndComp
 Wire Wire Line
-	9950 1200 9950 1300
+	10250 1150 10150 1150
 Wire Wire Line
 	9950 1400 9950 1550
@@
 Wire Wire Line
 	9500 3200 9400 3200
-Wire Wire Line
-	2100 1150 2100 1650
-Wire Wire Line
-	2100 1650 1700 1650
-Connection ~ 2100 1150
-$Comp
-L CONN_2 K1002
-U 1 1 51EB02DA
-P 1700 1750
-F 0 "K1002" H 2000 1900 50  0000 C CNN
-F 1 "CONN_2" H 2050 1850 40  0000 C CNN
-F 2 "~" H 1700 1750 60  0000 C CNN
-F 3 "~" H 1700 1750 60  0000 C CNN
-	1    1700 1750
-	-1   0    0    1
-$EndComp
-Wire Wire Line
-	1700 1750 1750 1750
-Wire Wire Line
-	1750 1750 1750 1850
-$Comp
-L GND #PWR043
-U 1 1 51EB03B5
-P 1750 1850
-F 0 "#PWR043" H 1750 1850 30  0001 C CNN
-F 1 "GND" H 1750 1780 30  0001 C CNN
-F 2 "" H 1750 1850 60  0000 C CNN
-F 3 "" H 1750 1850 60  0000 C CNN
-	1    1750 1850
-	1    0    0    -1
-$EndComp
 $Comp
 L R R1003
@@
 $EndComp
 $Comp
-L -5VA #PWR1095
+L -5VA #PWR1097
 U 1 1 5204B613
 P 10250 3000
-F 0 "#PWR1095" H 10250 3200 40  0001 C CNN
+F 0 "#PWR1097" H 10250 3200 40  0001 C CNN
 F 1 "-5VA" H 10250 3150 40  0000 C CNN
 F 2 "" H 10250 3000 60  0000 C CNN
@@
 $EndComp
 $Comp
-L -5VA #PWR1096
+L -5VA #PWR1098
 U 1 1 5204B681
 P 10250 3850
-F 0 "#PWR1096" H 10250 4050 40  0001 C CNN
+F 0 "#PWR1098" H 10250 4050 40  0001 C CNN
 F 1 "-5VA" H 10250 4000 40  0000 C CNN
 F 2 "" H 10250 3850 60  0000 C CNN
@@
 $EndComp
 $Comp
-L -5VA #PWR1097
+L -5VA #PWR1099
 U 1 1 5204B6EF
 P 10250 4700
-F 0 "#PWR1097" H 10250 4900 40  0001 C CNN
+F 0 "#PWR1099" H 10250 4900 40  0001 C CNN
 F 1 "-5VA" H 10250 4850 40  0000 C CNN
 F 2 "" H 10250 4700 60  0000 C CNN
@@
 $EndComp
 $Comp
-L -5VA #PWR1098
+L -5VA #PWR1100
 U 1 1 5204B75D
 P 10250 5550
-F 0 "#PWR1098" H 10250 5750 40  0001 C CNN
+F 0 "#PWR1100" H 10250 5750 40  0001 C CNN
 F 1 "-5VA" H 10250 5700 40  0000 C CNN
 F 2 "" H 10250 5550 60  0000 C CNN
@@
 $EndComp
 $Comp
-L -5VA #PWR1099
+L -5VA #PWR1101
 U 1 1 5204B7CB
 P 10250 6400
-F 0 "#PWR1099" H 10250 6600 40  0001 C CNN
+F 0 "#PWR1101" H 10250 6600 40  0001 C CNN
 F 1 "-5VA" H 10250 6550 40  0000 C CNN
 F 2 "" H 10250 6400 60  0000 C CNN
@@
 	4600 3000 4600 2950
 Connection ~ 4400 3000
+$Comp
+L CONN_2 K1003
+U 1 1 521A22D8
+P 10050 1150
+F 0 "K1003" H 10350 1300 50  0000 C CNN
+F 1 "CONN_2" H 10400 1250 40  0000 C CNN
+F 2 "~" H 10050 1150 60  0000 C CNN
+F 3 "~" H 10050 1150 60  0000 C CNN
+	1    10050 1150
+	0    -1   -1   0
+$EndComp
+Wire Wire Line
+	10050 1150 9950 1150
+Wire Wire Line
+	9950 1150 9950 1300
 $EndSCHEMATC

Commit message: DEBUT CPU
Parts:
- C1002, C1004: value 10µ/16V -> 33µ/16V
- C1005, C1011, C1019, C1020: value 10U/10V -> 47U/10V
- C1009, C1010: value 3.3n -> 4.7n
- C1012, C1013: value 10n -> 6.8n
- C1021: value 22U/10V -> 47U/10V
- C1022, C1024: value 22U/16V -> 33U/16V
- C1023: value 22U/10V -> NC
Connections:
- net -5VA: now also D1004.2 (K); no longer D1004.1 (A)
- net at R1004.1: now also D1004.1 (A); no longer D1004.2 (K)
