File: JK330-9-POWER/_autosave-JK330-9-POWER.kicad_pcb (KiCad board)
At the start: 2 copper layers, 142 parts, among them K1001 CONN_2, K1003 CONN_2, P1001 CONN_7, P1002 CONN_7, P1003 CONN_7, P1004 CONN_7, P1005 CONN_7, P1006 CONN_7, P1007 CONN_7, P1008 CONN_7, P1009 CONN_7, P1010 CONN_7, U1001 EC3A04, U1002 MP2307, U1003 MP2307, U1004 LM1117

Commit message: MAJ DOC TECHNIQUE
Parts:
- C1005, C1011, C1019, C1020: value 47U/10V -> 10U/10V
- C1009, C1010: value 4.7n -> 3.3n
- C1012, C1013: value 6.8n -> 10n
- C1021: value 47U/10V -> 22U/10V
- C1023: value NC -> 22U/10V
Connections:
- U1002 pad 9: (no net) -> GND
- U1003 pad 9: (no net) -> GND
Changed lines of the file:
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@@
 (kicad_pcb (version 3) (host pcbnew "(2013-07-07 BZR 4022)-stable")
   (general
-    (links 372)
+    (links 374)
     (no_connects 28)
     (area 27.717717 16.708 271.350285 189.390001)
@@
   (layers
     (15 Dessus.Cu signal)
-    (0 Dessous.Cu signal hide)
+    (0 Dessous.Cu signal)
     (16 Dessous.Adhes user)
     (17 Dessus.Adhes user)
@@
     (pad_to_mask_clearance 0)
     (aux_axis_origin 0 0)
-    (visible_elements 7FFFFBFF)
+    (visible_elements 7FFFFFFF)
     (pcbplotparams
       (layerselection 3178497)
-      (usegerberextensions true)
+      (usegerberextensions false)
       (excludeedgelayer true)
       (linewidth 0.150000)
-      (plotframeref false)
+      (plotframeref true)
       (viasonmask false)
       (mode 1)
@@
       (padsonsilk false)
       (subtractmaskfromsilk false)
-      (outputformat 1)
+      (outputformat 2)
       (mirror false)
-      (drillshape 1)
+      (drillshape 2)
       (scaleselection 1)
       (outputdirectory ""))
@@
     (pad 9 smd rect (at 0 0 270) (size 4.0005 2.79908)
       (layers Dessous.Cu Dessous.Pate Dessous.Masque)
+      (net 7 GND)
     )
     (model smd/cms_so8.wrl
@@
     (pad 9 smd rect (at 0 0 270) (size 4.0005 2.79908)
       (layers Dessous.Cu Dessous.Pate Dessous.Masque)
+      (net 7 GND)
     )
     (model smd/cms_so8.wrl
@@
       (effects (font (size 0.508 0.4572) (thickness 0.1143)) (justify mirror))
     )
-    (fp_text value 6.8n (at -1.651 0 360) (layer Dessous.SilkS)
+    (fp_text value 10n (at -1.651 0 360) (layer Dessous.SilkS)
       (effects (font (size 0.508 0.4572) (thickness 0.1143)) (justify mirror))
     )
@@
       (effects (font (size 0.508 0.4572) (thickness 0.1143)) (justify mirror))
     )
-    (fp_text value 4.7n (at -1.651 0 450) (layer Dessous.SilkS)
+    (fp_text value 3.3n (at -1.651 0 450) (layer Dessous.SilkS)
       (effects (font (size 0.508 0.4572) (thickness 0.1143)) (justify mirror))
     )
@@
       (effects (font (size 0.508 0.4572) (thickness 0.1143)) (justify mirror))
     )
-    (fp_text value 6.8n (at -1.651 0 360) (layer Dessous.SilkS)
+    (fp_text value 10n (at -1.651 0 360) (layer Dessous.SilkS)
       (effects (font (size 0.508 0.4572) (thickness 0.1143)) (justify mirror))
     )
@@
       (effects (font (size 0.508 0.4572) (thickness 0.1143)) (justify mirror))
     )
-    (fp_text value 4.7n (at -1.651 0 450) (layer Dessous.SilkS)
+    (fp_text value 3.3n (at -1.651 0 450) (layer Dessous.SilkS)
       (effects (font (size 0.508 0.4572) (thickness 0.1143)) (justify mirror))
     )
@@
       (effects (font (size 0.889 0.762) (thickness 0.127)) (justify mirror))
     )
-    (fp_text value 47U/10V (at 0.635 0 270) (layer Dessous.SilkS)
+    (fp_text value 10U/10V (at 0.635 0 270) (layer Dessous.SilkS)
       (effects (font (size 0.889 0.762) (thickness 0.127)) (justify mirror))
     )
@@
       (effects (font (size 0.889 0.762) (thickness 0.127)) (justify mirror))
     )
-    (fp_text value 47U/10V (at 0.635 0 450) (layer Dessous.SilkS)
+    (fp_text value 10U/10V (at 0.635 0 450) (layer Dessous.SilkS)
       (effects (font (size 0.889 0.762) (thickness 0.127)) (justify mirror))
     )
@@
       (effects (font (size 0.889 0.762) (thickness 0.127)) (justify mirror))
     )
-    (fp_text value 47U/10V (at 0.635 0 360) (layer Dessous.SilkS)
+    (fp_text value 10U/10V (at 0.635 0 360) (layer Dessous.SilkS)
       (effects (font (size 0.889 0.762) (thickness 0.127)) (justify mirror))
     )
@@
       (effects (font (size 0.889 0.762) (thickness 0.127)) (justify mirror))
     )
-    (fp_text value 47U/10V (at 0.635 0 360) (layer Dessous.SilkS)
+    (fp_text value 10U/10V (at 0.635 0 360) (layer Dessous.SilkS)
       (effects (font (size 0.889 0.762) (thickness 0.127)) (justify mirror))
     )
@@
       (effects (font (size 1.016 0.762) (thickness 0.2032)) (justify mirror))
     )
-    (fp_text value 47U/10V (at -0.889 0 540) (layer Dessous.SilkS)
+    (fp_text value 22U/10V (at -0.889 0 540) (layer Dessous.SilkS)
       (effects (font (size 0.762 0.762) (thickness 0.2032)) (justify mirror))
     )
@@
       (effects (font (size 1.016 0.762) (thickness 0.2032)) (justify mirror))
     )
-    (fp_text value NC (at -0.889 0 540) (layer Dessous.SilkS)
+    (fp_text value 22U/10V (at -0.889 0 540) (layer Dessous.SilkS)
       (effects (font (size 0.762 0.762) (thickness 0.2032)) (justify mirror))
     )
