File: jk330-8-CPU/5vto3v3.sch (KiCad schematic (older format))
At the start: 18 parts, among them U2 74LVCC3245, U3 74LVCC3245, U4 PCA9306, U5 PCA9306, U6 74LVCC3245

Commit message: MAJ CPU
Parts:
- removed R11, R12, R13, R14: 2.1k, symbol R
- removed R39: 200k, symbol R
- removed U5: PCA9306, symbol PCA9306
Connections:
- net labels added: /BCE, /BRD, /BWR, /CE, /RD, /WR, BC/D, C/D
- net labels removed: BE, BR/W, BRS, E, OC1, OC1-5V, OC2, OC2-5V, OC5, OC5-5V, R/W, RS, SCL4, SCL4-5V, SDA4, SDA4-5V, U5RX, U5RX-5V, U5TX, U5TX-5V, U6RX, U6RX-5V, U6TX, U6TX-5V
- wire segments 127 -> 107
Changed lines of the file:
@@
 LIBS:power
 LIBS:CEN-SCHEMA
+LIBS:ELECTRONICAL_MAIN_BOARD_32-cache
 EELAYER 27 0
 EELAYER END
 $Descr A4 11693 8268
 encoding utf-8
-Sheet 3 3
-Title "ELECTRONICAL_MAIN_BOARD_32"
-Date "16 sep 2013"
-Rev "V1-10"
-Comp "CYBERNETIQUE EN NORD"
+Sheet 2 4
+Title "JK330-CPU"
+Date "21 sep 2013"
+Rev "V1-00"
+Comp "F4DEB"
 Comment1 ""
 Comment2 ""
@@
 $EndDescr
 Wire Wire Line
-	9200 5500 9200 5650
-Wire Wire Line
-	9200 5200 9200 5150
-Wire Wire Line
 	9200 3900 9200 3850
 Wire Wire Line
@@
 Wire Wire Line
 	2500 4000 2850 4000
-Connection ~ 9350 5150
-Wire Wire Line
-	9350 5100 9350 5350
-Wire Wire Line
-	8050 5100 8050 5350
-Connection ~ 9350 5750
-Wire Wire Line
-	9350 5750 9350 5650
-Wire Wire Line
-	9100 5750 9650 5750
-Wire Wire Line
-	9100 5850 9650 5850
-Wire Wire Line
-	9450 5850 9450 5650
-Connection ~ 9450 5850
-Wire Wire Line
-	9450 5350 9450 5150
 Connection ~ 9450 4550
 Wire Wire Line
@@
 Wire Wire Line
 	8350 4250 8400 4250
-Wire Wire Line
-	8400 5550 8350 5550
-Wire Wire Line
-	9200 5650 9100 5650
 Wire Wire Line
 	9100 4350 9200 4350
@@
 Wire Bus Line
 	5750 4550 5750 7800
-Wire Wire Line
-	9200 5550 9100 5550
 Connection ~ 9200 4250
-Connection ~ 9200 5550
-Wire Wire Line
-	8400 5650 8200 5650
-Wire Wire Line
-	8350 5550 8350 5450
 Wire Wire Line
 	8400 4450 7800 4450
@@
 Connection ~ 7950 4550
 Wire Wire Line
-	7950 5350 7950 5150
-Connection ~ 7950 5850
-Wire Wire Line
-	7950 5850 7950 5650
-Connection ~ 8050 5750
-Wire Wire Line
-	8050 5750 8050 5650
-Wire Wire Line
-	8400 5750 7800 5750
-Wire Wire Line
-	8400 5850 7800 5850
-Wire Wire Line
 	9350 4450 9350 4350
 Connection ~ 9350 4450
-Wire Wire Line
-	7950 5150 8200 5150
-Connection ~ 8050 5150
-Wire Wire Line
-	9450 5150 9200 5150
-Wire Wire Line
-	8200 5150 8200 5650
 Wire Wire Line
 	8200 4350 8200 3850
@@
 Wire Wire Line
 	9200 4350 9200 4200
-$Comp
-L R R39
-U 1 1 500C6020
-P 9200 5250
-F 0 "R39" V 9150 5050 50  0000 C CNN
-F 1 "200k" V 9150 5250 50  0000 C CNN
-F 2 "" H 9200 5250 60  0001 C CNN
-F 3 "" H 9200 5250 60  0001 C CNN
-	1    9200 5250
-	1    0    0    -1
-$EndComp
 $Comp
 L R R38
@@
 	1    0    0    -1
 $EndComp
-Text HLabel 4000 4100 2    60   Input ~ 0
-U5RX-5V
 Text HLabel 4000 3900 2    60   Input ~ 0
 U1RX-5V
-Text HLabel 2500 4000 0    60   Input ~ 0
-U5RX
 Text HLabel 2500 3800 0    60   Input ~ 0
 U1RX
-Text HLabel 2500 2400 0    60   Input ~ 0
-U5TX
 Text HLabel 2500 2200 0    60   Input ~ 0
+C/D
+Text HLabel 2500 2300 0    60   Input ~ 0
 U1TX
-Text HLabel 4000 2500 2    60   Input ~ 0
-U5TX-5V
-Text HLabel 4000 2300 2    60   Input ~ 0
+Text HLabel 4000 2400 2    60   Input ~ 0
 U1TX-5V
-Text HLabel 2300 7200 0    60   Input ~ 0
+Text HLabel 4250 7200 2    60   Input ~ 0
 BD[0..7]
 Entry Wire Line
@@
 Entry Wire Line
 	2400 6100 2500 6000
-Text Label 2550 6000 0    60   ~ 0
+Text Label 3800 6100 0    60   ~ 0
 BD0
-Text Label 2550 6100 0    60   ~ 0
+Text Label 3800 6200 0    60   ~ 0
 BD1
-Text Label 2550 6200 0    60   ~ 0
+Text Label 3800 6300 0    60   ~ 0
 BD2
-Text Label 2550 6300 0    60   ~ 0
+Text Label 3800 6400 0    60   ~ 0
 BD3
-Text Label 2550 6400 0    60   ~ 0
+Text Label 3800 6500 0    60   ~ 0
 BD4
-Text Label 2550 6500 0    60   ~ 0
+Text Label 3800 6600 0    60   ~ 0
 BD5
-Text Label 2550 6600 0    60   ~ 0
+Text Label 3800 6700 0    60   ~ 0
 BD6
-Text Label 2550 6700 0    60   ~ 0
+Text Label 3800 6800 0    60   ~ 0
 BD7
 Text Notes 9150 3100 2    90   ~ 18
@@
 CONTRASTE
 Text HLabel 4000 2200 2    60   Input ~ 0
-BE
-Text HLabel 4000 2100 2    60   Input ~ 0
-BRS
-Text HLabel 4000 2000 2    60   Input ~ 0
-BR/W
-Text HLabel 4000 4600 2    60   Input ~ 0
-OC5-5V
-Text HLabel 4000 4400 2    60   Input ~ 0
-OC2-5V
-Text HLabel 4000 4300 2    60   Input ~ 0
-OC1-5V
-Text HLabel 2500 4500 0    60   Input ~ 0
-OC5
-Text HLabel 2500 4300 0    60   Input ~ 0
-OC2
-Text HLabel 2500 4200 0    60   Input ~ 0
-OC1
-Text HLabel 9650 5850 2    60   Input ~ 0
-SDA4-5V
-Text HLabel 9650 5750 2    60   Input ~ 0
-SCL4-5V
-Text HLabel 7800 5850 0    60   Input ~ 0
-SDA4
-Text HLabel 7800 5750 0    60   Input ~ 0
-SCL4
+/BCE
 $Comp
 L +5V #PWR054
@@
 SDA1
 $Comp
-L R R13
-U 1 1 4FC52EED
-P 9350 5400
-F 0 "R13" V 9300 5250 50  0000 C CNN
-F 1 "2.1k" V 9300 5450 50  0000 C CNN
-F 2 "" H 9350 5400 60  0001 C CNN
-F 3 "" H 9350 5400 60  0001 C CNN
-	1    9350 5400
-	1    0    0    -1
-$EndComp
-$Comp
-L R R14
-U 1 1 4FC52EEC
-P 9450 5400
-F 0 "R14" V 9400 5250 50  0000 C CNN
-F 1 "2.1k" V 9400 5450 50  0000 C CNN
-F 2 "" H 9450 5400 60  0001 C CNN
-F 3 "" H 9450 5400 60  0001 C CNN
-	1    9450 5400
-	1    0    0    -1
-$EndComp
-$Comp
 L R R10
 U 1 1 4FC52EDD
@@
 $EndComp
 $Comp
-L R R11
-U 1 1 4FC52EBF
-P 7950 5400
-F 0 "R11" V 7900 5300 50  0000 C CNN
-F 1 "2.1k" V 7900 5450 50  0000 C CNN
-F 2 "" H 7950 5400 60  0001 C CNN
-F 3 "" H 7950 5400 60  0001 C CNN
-	1    7950 5400
-	1    0    0    -1
-$EndComp
-$Comp
-L R R12
-U 1 1 4FC52EBE
-P 8050 5400
-F 0 "R12" V 8000 5300 50  0000 C CNN
-F 1 "2.1k" V 8000 5450 50  0000 C CNN
-F 2 "" H 8050 5400 60  0001 C CNN
-F 3 "" H 8050 5400 60  0001 C CNN
-	1    8050 5400
-	1    0    0    -1
-$EndComp
-$Comp
 L R R8
 U 1 1 4FC52EAB
@@
 	1    7950 4100
 	1    0    0    -1
-$EndComp
-$Comp
-L GND #PWR056
-U 1 1 4FC52E7D
-P 8350 5450
-F 0 "#PWR056" H 8350 5450 30  0001 C CNN
-F 1 "GND" H 8350 5380 30  0001 C CNN
-F 2 "" H 8350 5450 60  0001 C CNN
-F 3 "" H 8350 5450 60  0001 C CNN
-	1    8350 5450
-	-1   0    0    1
 $EndComp
 $Comp
@@
 	-1   0    0    1
 $EndComp
-$Comp
-L +3.3V #PWR058
-U 1 1 4FC52E68
-P 8050 5100
-F 0 "#PWR058" H 8050 5060 30  0001 C CNN
-F 1 "+3.3V" H 8050 5210 30  0000 C CNN
-F 2 "" H 8050 5100 60  0001 C CNN
-F 3 "" H 8050 5100 60  0001 C CNN
-	1    8050 5100
-	1    0    0    -1
-$EndComp
-$Comp
-L +5V #PWR059
-U 1 1 4FC52E41
-P 9350 5100
-F 0 "#PWR059" H 9350 5190 20  0001 C CNN
-F 1 "+5V" H 9350 5190 30  0000 C CNN
-F 2 "" H 9350 5100 60  0001 C CNN
-F 3 "" H 9350 5100 60  0001 C CNN
-	1    9350 5100
-	1    0    0    -1
-$EndComp
 Text Notes 3300 2650 1    60   ~ 0
 PORTA => PORTB\n\n
@@
 $EndComp
 Text HLabel 2500 1900 0    60   Input ~ 0
-R/W
+/WR
 Text HLabel 2500 2000 0    60   Input ~ 0
-RS
+/RD
 Text HLabel 2500 2100 0    60   Input ~ 0
-E
+/CE
 $Comp
 L GND #PWR060
@@
 Text HLabel 2500 3900 0    60   Input ~ 0
 U2RX
-Text HLabel 2500 4100 0    60   Input ~ 0
-U6RX
 Text HLabel 4000 4000 2    60   Input ~ 0
 U2RX-5V
-Text HLabel 4000 4200 2    60   Input ~ 0
-U6RX-5V
 $Comp
 L GND #PWR065
@@
 	0    1    1    0
 $EndComp
-Text HLabel 4000 2600 2    60   Input ~ 0
-U6TX-5V
-Text HLabel 4000 2400 2    60   Input ~ 0
+Text HLabel 4000 2500 2    60   Input ~ 0
 U2TX-5V
-Text HLabel 2500 2500 0    60   Input ~ 0
-U6TX
-Text HLabel 2500 2300 0    60   Input ~ 0
+Text HLabel 2500 2400 0    60   Input ~ 0
 U2TX
-$Comp
-L PCA9306 U5
-U 1 1 4FC529C0
-P 8400 5350
-F 0 "U5" H 9000 5350 60  0000 C CNN
-F 1 "PCA9306" H 8650 5350 60  0000 C CNN
-F 2 "" H 8400 5350 60  0001 C CNN
-F 3 "" H 8400 5350 60  0001 C CNN
-	1    8400 5350
-	1    0    0    -1
-$EndComp
 $Comp
 L PCA9306 U4
@@
 	1    0    0    -1
 $EndComp
-Text Label 3800 6800 0    60   ~ 0
+Text Label 2550 6700 0    60   ~ 0
 D7
-Text Label 3800 6700 0    60   ~ 0
+Text Label 2550 6600 0    60   ~ 0
 D6
-Text Label 3800 6600 0    60   ~ 0
+Text Label 2550 6500 0    60   ~ 0
 D5
-Text Label 3800 6400 0    60   ~ 0
+Text Label 2550 6300 0    60   ~ 0
 D3
-Text Label 3800 6500 0    60   ~ 0
+Text Label 2550 6400 0    60   ~ 0
 D4
-Text Label 3800 6300 0    60   ~ 0
+Text Label 2550 6200 0    60   ~ 0
 D2
-Text Label 3800 6200 0    60   ~ 0
+Text Label 2550 6100 0    60   ~ 0
 D1
-Text Label 3800 6100 0    60   ~ 0
+Text Label 2550 6000 0    60   ~ 0
 D0
-Text HLabel 4250 7200 2    60   Input ~ 0
+Text HLabel 2300 7200 0    60   Input ~ 0
 D[0..7]
 Entry Wire Line
@@
 $EndComp
 Text HLabel 1450 5900 0    60   Input ~ 0
-R/W
+/RD
 $Comp
 L +5V #PWR071
@@
 	1    0    0    -1
 $EndComp
+Connection ~ 5600 -100
+Text HLabel 4000 2000 2    60   Input ~ 0
+/BWR
+Text HLabel 4000 2100 2    60   Input ~ 0
+/BRD
+Text HLabel 4000 2300 2    60   Input ~ 0
+BC/D
+Wire Wire Line
+	2500 4400 2850 4400
+Wire Wire Line
+	3650 4500 4000 4500
 $EndSCHEMATC

Commit message: MAJ CPU
Parts:
- added U?: 74LVCC3245, symbol 74LVCC3245
Connections:
- net labels added: /BKOE, /KOE, BKAV, BKDA, BKDB, BKDC, BKDD, BKDE, BKDF, BOC1, BOC2, BOC3, BOC4, BOC5, KAV, KDA, KDB, KDC, KDD, KDE, KDF, OC1, OC2, OC3, OC4, OC5, U3RX, U3RX-5V, U3TX, U3TX-5V
- net labels removed: U1RX, U1RX-5V, U1TX, U1TX-5V
- wire segments 107 -> 132
Other:
- moved on the sheet: D6, R15, U2, U3, U6

Commit message: SCHEMA CPU 85%
Parts:
- added C4001, C4002, C4003, C4004, C4005, C4006, C4007, C4008, C4009, C4010: 100n, ~, symbol C
- gave numbers to parts that had none: 1
- renumbered D6 to D4001, R15 to R4001, R7 to R4002, R8 to R4003, R38 to R4004, R9 to R4005, R10 to R4006, RVAR1 to RVAR4001, U3 to U4002, U6 to U4003, U2 to U4004, U4 to U4005
Connections:
- net +3.3V: now also C4001.1, C4002.1, C4003.1, C4004.1, C4005.1
- net GND: now also C4001.2, C4002.2, C4003.2, C4004.2, C4005.2, C4006.2, C4007.2, C4008.2, C4009.2, C4010.2
- net +5V renamed +5VD
- net +5VD: now also C4006.1, C4007.1, C4008.1, C4009.1, C4010.1
Other:
- note added: "3.3V-5V CONVERTER"
- note removed: "LCD AND RS232 CONVERTER"

Commit message: CPU SCHEMA 100%
Parts:
- added Q4001, Q4002: BSS123, ~, symbol BSS123
- added R4002, R4003: 10k, ~, symbol R
- renumbered R4002 to R4004, R4003 to R4005, R4004 to R4006, R4005 to R4007, R4006 to R4008
Connections:
- net +3.3V: now also R4002.1
- net +5VD: now also R4003.1
- net GND: now also Q4001.1 (S), Q4002.1 (S)
- net U3RX: now also Q4001.3 (D), R4002.2
- net U3RX-5V: now also Q4002.2 (G)
- new net: Q4001.2 (G), Q4002.3 (D), R4003.2
- no-connect marks 0 -> 12
Other:
- moved on the sheet: D4001, R4001, U4002, U4003

Commit message: CPU EN TEST
Parts:
- RVAR4001: value 4.7K -> 4.7k; footprint (none) -> ~
Connections:
- net BC/D is gone; now on net /BCE: U4001.18 (B4)
- net C/D is gone; now on net /CE: U4001.6 (A4)
- net /BCE: no longer U4001.19 (B3)
- net /BRD: now also U4001.19 (B3); no longer U4001.20 (B2)
- net /BWR: now also U4001.20 (B2); no longer U4001.21 (B1)
- net /CE: no longer U4001.5 (A3)
- net /RD: now also U4001.5 (A3); no longer U4001.4 (A2)
- net /WR: now also U4001.4 (A2); no longer U4001.3 (A1)
- net BKDA: now also U4002.16 (B6); no longer U4002.19 (B3)
- net BKDB: now also U4002.17 (B5); no longer U4002.18 (B4)
- net BKDC: now also U4002.18 (B4); no longer U4002.17 (B5)
- net BKDD: now also U4002.19 (B3); no longer U4002.16 (B6)
- net KDA: now also U4002.8 (A6); no longer U4002.5 (A3)
- net KDB: now also U4002.7 (A5); no longer U4002.6 (A4)
- net KDC: now also U4002.6 (A4); no longer U4002.7 (A5)
- net KDD: now also U4002.5 (A3); no longer U4002.8 (A6)
- net U2TX: now also U4001.3 (A1); no longer U4001.8 (A6)
- net U2TX-5V: now also U4001.21 (B1); no longer U4001.16 (B6)
- net U3TX: now also U4001.8 (A6); no longer U4001.7 (A5)
- net U3TX-5V: now also U4001.16 (B6); no longer U4001.17 (B5)
- new net BCD: U4001.17 (B5)
- new net CD: U4001.7 (A5)
