File: jk330-8-CPU/ELECTRONICAL_MAIN_BOARD_32.sch (KiCad schematic (older format))
At the start: 33 parts, among them J1 SIL1, J2 SIL1, J3 SIL1, J4 SIL1, J5 RJ12, J6 SIL1, J7 SIL1, K1 CONN_3, K2 CONN_3, K3 CONN_3, K4 CONN_3, K5 CONN_3, K6 CONN_3, K7 CONN_3, P1 HE10-16, P2 CONN_4, P3 CONN_4, P4 CONN_4, P5 CONN_4, P6 CONN_4, P7 CONN_4, P8 CONN_2, P9 CONN_5, SW1 SWITCH_X_8, SW2 SW_PUSH_SMALL, SW3 SWITCH_X_8

Commit message: DEBUT CPU
Other:
- note added: "ELECTRONICAL_MAIN_BOARD_32 JK330-A"
- note removed: "ELECTRONICAL_MAIN_BOARD_32"

Commit message: MAJ CPU
Parts:
- removed K1, K2, K3, K4, K5, K6, K7: CONN_3, symbol CONN_3
- removed L1: 15uH, symbol INDUCTOR
- removed P1: HE10-16, symbol HE10-16
- removed P4, P5, P6: CONN_4, symbol CONN_4
- removed P8: CONN_2, symbol CONN_2
- removed P9: CONN_5, symbol CONN_5
- removed SW1, SW3: SWITCH_X_8, symbol SWITCH_X_8
- added P?: CONN_5, symbol CONN_5
- added P?: CONN_5X2, symbol CONN_5X2
- added P?: CONN_10X2, symbol CONN_10X2
- added P?: CAVALIER2, ~, symbol CAVALIER2
- added R?: R, ~, symbol R
Connections:
- net labels added: +5VA, +5VD, /BCE, /BRD, /BWR, /CE, /RD, /RST, /WR, BC/D, CONTRASTE, FS
- net labels removed: +5V, BE, BR/W, BRS, CONT
- wire segments 177 -> 101
Other:
- note added: "ALIM\n\n"
- note added: "CPU 32 BITS JK330-A"
- note added: "LCD GRAPHIQUE\nMGLS24064"
- note added: "UART-1\n\n"
- note added: "UART-2\n\n\n"
- note removed: "ALIM 3.3V \n5V / 12V\n"
- note removed: "CAN"
- note removed: "ELECTRONICAL_MAIN_BOARD_32 JK330-A"
- note removed: "GO"
- note removed: "I2C-4"
- note removed: "LCD 4 X 20"
- note removed: "S1"
- note removed: "S2"
- note removed: "S3"
- note removed: "SERVO MOTEUR"
- note removed: "UART-2\n"
- note removed: "UART-6\n"
- moved on the sheet: D1, D2, D3, D4, J1, J2, J3, J4, J5, J6, J7, P2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

Commit message: MAJ CPU
Parts:
- added P? (x2): CONN_5X2, symbol CONN_5X2
Connections:
- net labels added: LED1, LED2, LED3, LED4, LED5, LED6, LED7, LED8, SCL, SDA
- net labels removed: /CE, /RD, /WR
- wire segments 101 -> 108
Other:
- note added: "UART-3\n\n\n"
- note removed: "CONFIG"
- note removed: "UART-1\n\n"
- moved on the sheet: P?

Commit message: SCHEMA CPU 85%
Parts:
- added K1001, K1002, K1003, K1004, K1005, K1006, K1007, K1008, K1009, K1010, K1011, K1012, K1013, K1014: CONN_3, symbol CONN_3
- added R? (x2): R, ~, symbol R
- R1003: renamed from R?; value R -> 0
- gave numbers to parts that had none: 6
- renumbered D1 to D1001, D2 to D1002, D3 to D1003, D4 to D1004, J5 to J1001, J1 to J1002, J2 to J1003, J3 to J1004, J4 to J1005, J6 to J1006, J7 to J1007, P2 to P1002, P3 to P1003, P7 to P1004, R1 to R1001, R2 to R1002, SW2 to SW1001
Connections:
- net labels added: ADC1, ADC10, ADC11, ADC12, ADC13, ADC14, ADC2, ADC3, ADC4, ADC5, ADC6, ADC7, ADC8, ADC9, X1, X2, X3, X4, Y1, Y1A, Y1B, Y2, Y2A, Y2B, Y3, Y3A, Y3B, Y4, Y4A, Y4B
- wire segments 108 -> 212
Other:
- moved on the sheet: D1001, D1002, D1003, D1004, P1001, P1002, P1003, P1004, P1007, P1008, P1009, R1001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

Commit message: CPU SCHEMA 100%
Parts:
- added K1008, K1009, K1010, K1018, K1019: CONN_3, symbol CONN_3
- R1001: renamed from R?; value R -> 3.3k
- R1002: renamed from R?; value R -> 1k
- R1003: renamed from R1001; value R -> 1k
- R1004: renamed from R1002; value R -> 330
- renumbered K1008 to K1011, K1009 to K1012, K1010 to K1013, K1011 to K1014, K1012 to K1015, K1013 to K1016, K1014 to K1017, R1003 to R1005
Connections:
- net labels added: +BATT, BOC1, BOC2, BOC3, BOC4, BOC5, D[0..7]
- wire segments 212 -> 263
- no-connect marks 0 -> 7
Other:
- note added: "14 I/O or DAC\n"
- note added: "5 OUT 5V\n"
- note added: "KEYBOARD + LED"
- moved on the sheet: P1007, P1008, P1009

Commit message: CPU EN TEST
Parts:
- added K1020: CONN_3, symbol CONN_3
Connections:
- net labels added: +5V, BCD
- net labels removed: BC/D
- wire segments 263 -> 266
- no-connect marks 7 -> 5
Other:
- moved on the sheet: P1007, P1008, P1009
