File: jk330-8-CPU/INTERFACE BOARD.sch (KiCad schematic (older format))
At the start: 40 parts

Commit message: MAJ CPU
Parts:
- removed D? (x4): LED, symbol LED
- removed D? (x2): LED_BI_2, symbol LED_BI_2
- R?: value R -> 10k
Connections:
- net labels added: BKAV, BKDA, BKDB, BKDC, BKDD, BKDE, BKDF, BKOE\, LED1, LED2, LED3, LED4, LED5, LED6, LED7, LED8
- net labels removed: KAV, KDA, KDB, KDC, KDD, KDE, KDF, KOE\
- wire segments 152 -> 98

Commit message: SCHEMA CPU 85%
Parts:
- gave numbers to parts that had none: 33
Connections:
- wire segments 98 -> 100

Commit message: CPU SCHEMA 100%
Parts:
- C2001, C2003, C2004, C2005: value C -> 100n
- C2002: value C -> 1U
- R2002, R2003, R2004, R2005, R2006, R2007, R2008, R2009: value R -> 1k
- R2010, R2011, R2012, R2013, R2014, R2015, R2016, R2017: value R -> 10k
Other:
- moved on the sheet: U2003A, U2003B
