File: jk330-8-CPU/PIC32.sch (KiCad schematic (older format))
At the start: 42 parts, among them U1 PIC32MX795F512H

Commit message: MAJ CPU
Parts:
- removed D10, D5, D7, D8, D9: LED, symbol LED
- removed R16, R17, R18, R19, R20, R21, R22, R23, R24, R25, R26, R27, R28, R29, R5: 10K, symbol R
- removed R3, R4, R6: 1K, symbol R
- removed R30, R31, R32, R33, R34, R35, R36, R37: 470, symbol R
Connections:
- net SMETER: now reaches U1.14 (AN2/C2IN-/CN4/RB2)
- net E renamed /WR
- net GO: no longer names the net of U1.36 (D-/RG3)
- net OC1: no longer names the net of U1.46 (OC1/INT0/RD0)
- net OC2: no longer names the net of U1.49 (EMDIO/AEMDIO/SCK3/U4TX/U1RTS/OC2/RD1)
- net OC5: no longer names the net of U1.52 (OC5/IC5/PMWR/CN13/RD4)
- net R/W renamed /CE
- net RS renamed /RD
- net SCL4: no longer names the net of U1.6 (SCL4/SDO2/U3TX/PMA3/CN10/RG8)
- net SDA4: no longer names the net of U1.5 (SDA4/SDI2/U3RX/PMA4/CN9/RG7)
- net SW0: no longer names the net of U1.53 (PMRD/CN14/RD5)
- net SW1: no longer names the net of U1.54 (AETXEN/ETXERR/CN15/RD6)
- net SW10: no longer names the net of U1.28 (TDI/AN13/PMA10/RB13)
- net SW11: no longer names the net of U1.30 (AN15/EMDC/AEMDC/OCFB/PMALL/PMA0/CN12/RB15)
- net SW12: no longer names the net of U1.47 (SOSCI/CN1/RC13)
- net SW13: no longer names the net of U1.37 (D+/RG2)
- net SW2: no longer names the net of U1.55 (ETXCLK/AERXERR/CN16/RD7)
- net SW3 renamed C/D
- net SW4: no longer names the net of U1.17 (PGEC2/AN6/OCFA/RB6)
- net SW5: no longer names the net of U1.18 (PGED2/AN7/RB7)
- net SW6: no longer names the net of U1.22 (AN9/C2OUT/PMA7/RB9)
- net SW7: no longer names the net of U1.23 (TMS/AN10/CVREFOUT/PMA13/RB10)
- net SW8: no longer names the net of U1.24 (TDO/AN11/PMA12/RB11)
- net SW9: no longer names the net of U1.27 (TCK/AN12/PMA11/RB12)
- net U5RX: no longer names the net of U1.21 (AN8/C2TX/SS4/U5RX/U2CTS/C1OUT/RB8)
- net U5TX: no longer names the net of U1.29 (AN14/C2RX/SCK4/U5TX/U2RTS/PMALH/PMA1/RB14)
- net U6RX: no longer names the net of U1.8 (SS2/U6RX/U3CTS/PMA2/CN11/RG9)
- net U6TX: no longer names the net of U1.4 (SCK2/U6TX/U3RTS/PMA5/CN8/RG6)
Other:
- note added: "FILTER CAPACITOR"
- note removed: "FILTER CAPACITER"

Commit message: MAJ CPU
Parts:
- added C? (x2): C, ~, symbol C
- added X?: 32.768khz, ~, symbol CRYSTAL1
Connections:
- net GND: now also C?.2, C?.2
- net ADC4: now reaches U1.11 (AN5/C1IN+/Vbuson/CN7/RB5)
- net ADC3: now reaches U1.12 (AN4/C1IN-/CN6/RB4)
- net ADC2: now reaches U1.13 (AN3/C2IN+/CN5/RB3)
- net ADC5: now reaches U1.17 (PGEC2/AN6/OCFA/RB6)
- net ADC6: now reaches U1.18 (PGED2/AN7/RB7)
- net ADC7: now reaches U1.21 (AN8/C2TX/SS4/U5RX/U2CTS/C1OUT/RB8)
- net ADC8: now reaches U1.22 (AN9/C2OUT/PMA7/RB9)
- net ADC9: now reaches U1.23 (TMS/AN10/CVREFOUT/PMA13/RB10)
- net ADC10: now reaches U1.24 (TDO/AN11/PMA12/RB11)
- net ADC11: now reaches U1.27 (TCK/AN12/PMA11/RB12)
- net ADC12: now reaches U1.28 (TDI/AN13/PMA10/RB13)
- net ADC13: now reaches U1.29 (AN14/C2RX/SCK4/U5TX/U2RTS/PMALH/PMA1/RB14)
- net ADC14: now reaches U1.30 (AN15/EMDC/AEMDC/OCFB/PMALL/PMA0/CN12/RB15)
- net OC1: now reaches U1.46 (OC1/INT0/RD0)
- net at U1.47 (SOSCI/CN1/RC13): now also C?.1, X?.2
- net at U1.48 (SOSCO/T1CK/CN0/RC14): now also C?.1, X?.1
- net OC2: now reaches U1.49 (EMDIO/AEMDIO/SCK3/U4TX/U1RTS/OC2/RD1)
- net U3RX: now reaches U1.5 (SDA4/SDI2/U3RX/PMA4/CN9/RG7)
- net OC5: now reaches U1.52 (OC5/IC5/PMWR/CN13/RD4)
- net U3TX: now reaches U1.6 (SCL4/SDO2/U3TX/PMA3/CN10/RG8)
- net SMETER renamed ADC1
- net U1RX renamed OC3
- net U1TX renamed OC4
Other:
- note added: "MICROCONTROLLER\n"
- note removed: "MICRO-CONTROLLOR\n"
Changed lines of the file:
@@
 $Descr A4 11693 8268
 encoding utf-8
-Sheet 2 4
+Sheet 3 4
 Title "JK330-CPU"
-Date "21 sep 2013"
+Date "22 sep 2013"
 Rev "V1-00"
 Comp "F4DEB"
@@
 $EndDescr
 Wire Wire Line
-	10500 3950 9100 3950
+	9100 3950 10500 3950
 Connection ~ 9800 4850
 Wire Wire Line
@@
 Connection ~ 9800 4450
 Wire Wire Line
-	10500 4500 10500 4450
-Wire Wire Line
-	10500 4450 9100 4450
+	10500 4450 10500 4500
+Wire Wire Line
+	9100 4450 10500 4450
 Connection ~ 9800 3950
 Wire Wire Line
@@
 Connection ~ 9800 3550
 Wire Wire Line
-	10500 3600 10500 3550
+	10500 3550 10500 3600
 Wire Wire Line
 	7100 2500 7300 2500
@@
 Wire Wire Line
 	4550 5550 2650 5550
-Wire Wire Line
-	4550 4950 2650 4950
 Wire Wire Line
 	4550 2250 2600 2250
@@
 Connection ~ 9450 3950
 Wire Wire Line
-	9450 4050 9450 3900
+	9450 3900 9450 4050
 Wire Wire Line
 	9450 3450 9450 3600
@@
 	9100 4800 9100 4850
 Wire Wire Line
-	9450 4950 9450 4800
+	9450 4800 9450 4950
 Wire Wire Line
 	7100 4250 7650 4250
@@
 	7100 3650 7650 3650
 Wire Bus Line
-	7750 4150 7750 3400
+	7750 3400 7750 4150
 Wire Bus Line
 	7750 3400 8400 3400
@@
 Wire Wire Line
 	4550 2350 2600 2350
-Wire Wire Line
-	4550 4850 2650 4850
 Wire Notes Line
 	6750 3300 6750 2350
@@
 	7100 2400 7300 2400
 Wire Wire Line
-	10150 3600 10150 3550
+	10150 3550 10150 3600
 Connection ~ 10150 3550
 Wire Wire Line
@@
 	1    0    0    -1
 $EndComp
-Text HLabel 2650 4950 0    60   Input ~ 0
-U1TX
-Text HLabel 2650 4850 0    60   Input ~ 0
-U1RX
 Text HLabel 2600 2250 0    60   Input ~ 0
 PGED1
@@
 $EndComp
 Text Notes 4200 900  0    150  ~ 30
-MICRO-CONTROLLOR\n
+MICROCONTROLLER\n
 Text Notes 4650 1650 0    90   ~ 18
 PIC
@@
 Wire Wire Line
 	4550 2450 3850 2450
+Wire Wire Line
+	3850 2550 4550 2550
+Wire Wire Line
+	3850 2650 4550 2650
+Wire Wire Line
+	3850 2750 4550 2750
+Wire Wire Line
+	3850 2850 4550 2850
+Wire Wire Line
+	3850 2950 4550 2950
+Wire Wire Line
+	3850 3050 4550 3050
+Wire Wire Line
+	3850 3150 4550 3150
+Wire Wire Line
+	3850 3250 4550 3250
+Wire Wire Line
+	3850 3350 4550 3350
+Wire Wire Line
+	3850 3450 4550 3450
+Wire Wire Line
+	3850 3550 4550 3550
+Wire Wire Line
+	3850 3650 4550 3650
+Wire Wire Line
+	3850 3750 4550 3750
+Wire Wire Line
+	3350 3900 4550 3900
+Wire Notes Line
+	4350 4150 4350 4550
+Wire Notes Line
+	4350 4550 5200 4550
+Wire Notes Line
+	5200 4550 5200 4150
+Wire Notes Line
+	5200 4150 4350 4150
+Text Notes 4800 4250 2    60   ~ 0
+INTERNAL\n
 Text HLabel 3850 2450 0    60   Input ~ 0
-SMETER
+ADC1
+Text HLabel 3850 2550 0    60   Input ~ 0
+ADC2
+Text HLabel 3850 2650 0    60   Input ~ 0
+ADC3
+Text HLabel 3850 2750 0    60   Input ~ 0
+ADC4
+Text HLabel 3850 2850 0    60   Input ~ 0
+ADC5
+Text HLabel 3850 2950 0    60   Input ~ 0
+ADC6
+Text HLabel 3850 3050 0    60   Input ~ 0
+ADC7
+Text HLabel 3850 3150 0    60   Input ~ 0
+ADC8
+Text HLabel 3850 3250 0    60   Input ~ 0
+ADC9
+Text HLabel 3850 3350 0    60   Input ~ 0
+ADC10
+Text HLabel 3850 3550 0    60   Input ~ 0
+ADC12
+Text HLabel 3850 3450 0    60   Input ~ 0
+ADC11
+Text HLabel 3850 3650 0    60   Input ~ 0
+ADC13
+Text HLabel 3850 3750 0    60   Input ~ 0
+ADC14
+Wire Wire Line
+	2750 4050 4550 4050
+$Comp
+L CRYSTAL1 X?
+U 1 1 523F4EF1
+P 3150 3900
+F 0 "X?" H 3150 4050 60  0000 C CNN
+F 1 "32.768khz" H 3150 3750 60  0000 C CNN
+F 2 "~" H 3150 3900 60  0000 C CNN
+F 3 "~" H 3150 3900 60  0000 C CNN
+	1    3150 3900
+	1    0    0    -1
+$EndComp
+$Comp
+L C C?
+U 1 1 523F4F0A
+P 2750 4350
+F 0 "C?" H 2800 4450 50  0000 L CNN
+F 1 "C" H 2800 4250 50  0000 L CNN
+F 2 "~" H 2750 4350 60  0000 C CNN
+F 3 "~" H 2750 4350 60  0000 C CNN
+	1    2750 4350
+	1    0    0    -1
+$EndComp
+$Comp
+L C C?
+U 1 1 523F4F19
+P 3500 4350
+F 0 "C?" H 3550 4450 50  0000 L CNN
+F 1 "C" H 3550 4250 50  0000 L CNN
+F 2 "~" H 3500 4350 60  0000 C CNN
+F 3 "~" H 3500 4350 60  0000 C CNN
+	1    3500 4350
+	1    0    0    -1
+$EndComp
+Wire Wire Line
+	2750 4200 2750 3900
+Wire Wire Line
+	2750 3900 2950 3900
+Wire Wire Line
+	3500 4200 3500 3900
+Connection ~ 3500 3900
+Connection ~ 2750 4050
+Wire Wire Line
+	2750 4500 2750 4550
+Wire Wire Line
+	3500 4500 3500 4550
+$Comp
+L GND #PWR?
+U 1 1 523F514A
+P 2750 4550
+F 0 "#PWR?" H 2750 4550 30  0001 C CNN
+F 1 "GND" H 2750 4480 30  0001 C CNN
+F 2 "" H 2750 4550 60  0000 C CNN
+F 3 "" H 2750 4550 60  0000 C CNN
+	1    2750 4550
+	1    0    0    -1
+$EndComp
+$Comp
+L GND #PWR?
+U 1 1 523F5159
+P 3500 4550
+F 0 "#PWR?" H 3500 4550 30  0001 C CNN
+F 1 "GND" H 3500 4480 30  0001 C CNN
+F 2 "" H 3500 4550 60  0000 C CNN
+F 3 "" H 3500 4550 60  0000 C CNN
+	1    3500 4550
+	1    0    0    -1
+$EndComp
+Wire Wire Line
+	4550 4650 4250 4650
+Wire Wire Line
+	4550 4750 4250 4750
+Wire Wire Line
+	4550 5050 4250 5050
+Wire Wire Line
+	7100 5550 7600 5550
+Wire Wire Line
+	7100 5650 7600 5650
+Text HLabel 7600 5550 2    60   Input ~ 0
+U3RX
+Text HLabel 7600 5650 2    60   Input ~ 0
+U3TX
+Wire Wire Line
+	4250 4850 4550 4850
+Wire Wire Line
+	4250 4950 4550 4950
+Text HLabel 4250 4650 0    60   Input ~ 0
+OC1
+Text HLabel 4250 4750 0    60   Input ~ 0
+OC2
+Text HLabel 4250 4850 0    60   Input ~ 0
+OC3
+Text HLabel 4250 4950 0    60   Input ~ 0
+OC4
+Text HLabel 4250 5050 0    60   Input ~ 0
+OC5
 $EndSCHEMATC

Commit message: SCHEMA CPU 85%
Parts:
- removed C1, C10, C11, C2, C3, C4, C5, C6, C7, C8: 100n, symbol C
- gave numbers to parts that had none: 3
- renumbered U1 to U3001
Connections:
- net C/D: now also U3001.45 (ECRS/AEREFCLK/IC4/PMCS1/PMA14/INT4/RD11); no longer U3001.42 (RTCC/AERXD1/ETXD3/IC1/INT1/RD8)
- net KDE: now reaches U3001.36 (D-/RG3)
- net KDF: now reaches U3001.37 (D+/RG2)
- net KAV: now reaches U3001.4 (SCK2/U6TX/U3RTS/PMA5/CN8/RG6)
- net KDA: now reaches U3001.53 (PMRD/CN14/RD5)
- net KDB: now reaches U3001.54 (AETXEN/ETXERR/CN15/RD6)
- net KDC: now reaches U3001.55 (ETXCLK/AERXERR/CN16/RD7)
- net /KOE: now reaches U3001.8 (SS2/U6RX/U3CTS/PMA2/CN11/RG9)
- new net KDD: U3001.42 (RTCC/AERXD1/ETXD3/IC1/INT1/RD8)
Other:
- note removed: "FILTER CAPACITOR"

Commit message: CPU SCHEMA 100%
Parts:
- C3001, C3002: value C -> 22p
Connections:
- no-connect marks 0 -> 12
Changed lines of the file:
@@
 Sheet 3 4
 Title "JK330-CPU"
-Date "23 sep 2013"
+Date "24 sep 2013"
 Rev "V1-00"
 Comp "F4DEB"
@@
 	7100 2400 7300 2400
 $Comp
-L GND #PWR3004
+L GND #PWR093
 U 1 1 4FD220E7
 P 7300 2500
-F 0 "#PWR3004" H 7300 2500 30  0001 C CNN
+F 0 "#PWR093" H 7300 2500 30  0001 C CNN
 F 1 "GND" H 7300 2430 30  0001 C CNN
 F 2 "" H 7300 2500 60  0001 C CNN
@@
 $EndComp
 $Comp
-L +3.3V #PWR3003
+L +3.3V #PWR094
 U 1 1 4FD220DF
 P 7300 2400
-F 0 "#PWR3003" H 7300 2360 30  0001 C CNN
+F 0 "#PWR094" H 7300 2360 30  0001 C CNN
 F 1 "+3.3V" H 7300 2510 30  0000 C CNN
 F 2 "" H 7300 2400 60  0001 C CNN
@@
 P 2750 4350
 F 0 "C3001" H 2800 4450 50  0000 L CNN
-F 1 "C" H 2800 4250 50  0000 L CNN
+F 1 "22p" H 2800 4250 50  0000 L CNN
 F 2 "~" H 2750 4350 60  0000 C CNN
 F 3 "~" H 2750 4350 60  0000 C CNN
@@
 P 3500 4350
 F 0 "C3002" H 3550 4450 50  0000 L CNN
-F 1 "C" H 3550 4250 50  0000 L CNN
+F 1 "22p" H 3550 4250 50  0000 L CNN
 F 2 "~" H 3500 4350 60  0000 C CNN
 F 3 "~" H 3500 4350 60  0000 C CNN
@@
 	3500 4500 3500 4550
 $Comp
-L GND #PWR3001
+L GND #PWR095
 U 1 1 523F514A
 P 2750 4550
-F 0 "#PWR3001" H 2750 4550 30  0001 C CNN
+F 0 "#PWR095" H 2750 4550 30  0001 C CNN
 F 1 "GND" H 2750 4480 30  0001 C CNN
 F 2 "" H 2750 4550 60  0000 C CNN
@@
 $EndComp
 $Comp
-L GND #PWR3002
+L GND #PWR096
 U 1 1 523F5159
 P 3500 4550
-F 0 "#PWR3002" H 3500 4550 30  0001 C CNN
+F 0 "#PWR096" H 3500 4550 30  0001 C CNN
 F 1 "GND" H 3500 4480 30  0001 C CNN
 F 2 "" H 3500 4550 60  0000 C CNN
@@
 Text HLabel 7500 5450 2    60   Input ~ 0
 KAV
+NoConn ~ 4550 4300
+NoConn ~ 4550 4450
+NoConn ~ 7100 2600
+NoConn ~ 7100 2700
+NoConn ~ 7100 2800
+NoConn ~ 7100 2900
+NoConn ~ 7100 3000
+NoConn ~ 7100 3150
+NoConn ~ 7100 3250
+NoConn ~ 7100 3400
+NoConn ~ 7100 4950
+NoConn ~ 7100 5050
 $EndSCHEMATC

Commit message: CPU EN TEST
Connections:
- net at C3002.1, X3001.2: now also U3001.48 (SOSCO/T1CK/CN0/RC14); no longer U3001.47 (SOSCI/CN1/RC13)
- net at C3001.1, X3001.1: now also U3001.47 (SOSCI/CN1/RC13); no longer U3001.48 (SOSCO/T1CK/CN0/RC14)
- net C/D renamed CD
Other:
- moved on the sheet: C3001, C3002, X3001
Changed lines of the file:
@@
 Sheet 3 4
 Title "JK330-CPU"
-Date "24 sep 2013"
+Date "19 oct 2013"
 Rev "V1-00"
 Comp "F4DEB"
@@
 	7100 2400 7300 2400
 $Comp
-L GND #PWR093
+L GND #PWR094
 U 1 1 4FD220E7
 P 7300 2500
-F 0 "#PWR093" H 7300 2500 30  0001 C CNN
+F 0 "#PWR094" H 7300 2500 30  0001 C CNN
 F 1 "GND" H 7300 2430 30  0001 C CNN
 F 2 "" H 7300 2500 60  0001 C CNN
@@
 $EndComp
 $Comp
-L +3.3V #PWR094
+L +3.3V #PWR095
 U 1 1 4FD220DF
 P 7300 2400
-F 0 "#PWR094" H 7300 2360 30  0001 C CNN
+F 0 "#PWR095" H 7300 2360 30  0001 C CNN
 F 1 "+3.3V" H 7300 2510 30  0000 C CNN
 F 2 "" H 7300 2400 60  0001 C CNN
@@
 	4550 5750 4300 5750
 Text HLabel 4300 5750 0    60   Input ~ 0
-C/D
+CD
 Wire Wire Line
 	4550 2450 3850 2450
@@
 Wire Wire Line
 	3850 3750 4550 3750
-Wire Wire Line
-	3350 3900 4550 3900
 Wire Notes Line
 	4350 4150 4350 4550
@@
 Text HLabel 3850 3750 0    60   Input ~ 0
 ADC14
-Wire Wire Line
-	2750 4050 4550 4050
 $Comp
 L CRYSTAL1 X3001
 U 1 1 523F4EF1
-P 3150 3900
-F 0 "X3001" H 3150 4050 60  0000 C CNN
-F 1 "32.768khz" H 3200 4150 60  0000 C CNN
-F 2 "~" H 3150 3900 60  0000 C CNN
-F 3 "~" H 3150 3900 60  0000 C CNN
-	1    3150 3900
+P 3150 4050
+F 0 "X3001" H 3150 4200 60  0000 C CNN
+F 1 "32.768khz" H 3200 4300 60  0000 C CNN
+F 2 "~" H 3150 4050 60  0000 C CNN
+F 3 "~" H 3150 4050 60  0000 C CNN
+	1    3150 4050
 	1    0    0    -1
 $EndComp
@@
 L C C3001
 U 1 1 523F4F0A
-P 2750 4350
-F 0 "C3001" H 2800 4450 50  0000 L CNN
-F 1 "22p" H 2800 4250 50  0000 L CNN
-F 2 "~" H 2750 4350 60  0000 C CNN
-F 3 "~" H 2750 4350 60  0000 C CNN
-	1    2750 4350
+P 2750 4500
+F 0 "C3001" H 2800 4600 50  0000 L CNN
+F 1 "22p" H 2800 4400 50  0000 L CNN
+F 2 "~" H 2750 4500 60  0000 C CNN
+F 3 "~" H 2750 4500 60  0000 C CNN
+	1    2750 4500
 	1    0    0    -1
 $EndComp
@@
 L C C3002
 U 1 1 523F4F19
-P 3500 4350
-F 0 "C3002" H 3550 4450 50  0000 L CNN
-F 1 "22p" H 3550 4250 50  0000 L CNN
-F 2 "~" H 3500 4350 60  0000 C CNN
-F 3 "~" H 3500 4350 60  0000 C CNN
-	1    3500 4350
-	1    0    0    -1
-$EndComp
-Wire Wire Line
-	2750 3900 2750 4200
-Wire Wire Line
-	2750 3900 2950 3900
-Wire Wire Line
-	3500 4200 3500 3900
-Connection ~ 3500 3900
-Connection ~ 2750 4050
-Wire Wire Line
-	2750 4500 2750 4550
-Wire Wire Line
-	3500 4500 3500 4550
-$Comp
-L GND #PWR095
+P 3500 4500
+F 0 "C3002" H 3550 4600 50  0000 L CNN
+F 1 "22p" H 3550 4400 50  0000 L CNN
+F 2 "~" H 3500 4500 60  0000 C CNN
+F 3 "~" H 3500 4500 60  0000 C CNN
+	1    3500 4500
+	1    0    0    -1
+$EndComp
+Wire Wire Line
+	2750 3900 2750 4350
+Wire Wire Line
+	2750 4050 2950 4050
+Wire Wire Line
+	3500 4350 3500 4050
+Wire Wire Line
+	2750 4650 2750 4700
+Wire Wire Line
+	3500 4650 3500 4700
+$Comp
+L GND #PWR096
 U 1 1 523F514A
-P 2750 4550
-F 0 "#PWR095" H 2750 4550 30  0001 C CNN
-F 1 "GND" H 2750 4480 30  0001 C CNN
-F 2 "" H 2750 4550 60  0000 C CNN
-F 3 "" H 2750 4550 60  0000 C CNN
-	1    2750 4550
-	1    0    0    -1
-$EndComp
-$Comp
-L GND #PWR096
+P 2750 4700
+F 0 "#PWR096" H 2750 4700 30  0001 C CNN
+F 1 "GND" H 2750 4630 30  0001 C CNN
+F 2 "" H 2750 4700 60  0000 C CNN
+F 3 "" H 2750 4700 60  0000 C CNN
+	1    2750 4700
+	1    0    0    -1
+$EndComp
+$Comp
+L GND #PWR097
 U 1 1 523F5159
-P 3500 4550
-F 0 "#PWR096" H 3500 4550 30  0001 C CNN
-F 1 "GND" H 3500 4480 30  0001 C CNN
-F 2 "" H 3500 4550 60  0000 C CNN
-F 3 "" H 3500 4550 60  0000 C CNN
-	1    3500 4550
+P 3500 4700
+F 0 "#PWR097" H 3500 4700 30  0001 C CNN
+F 1 "GND" H 3500 4630 30  0001 C CNN
+F 2 "" H 3500 4700 60  0000 C CNN
+F 3 "" H 3500 4700 60  0000 C CNN
+	1    3500 4700
 	1    0    0    -1
 $EndComp
@@
 NoConn ~ 7100 4950
 NoConn ~ 7100 5050
+Wire Wire Line
+	3350 4050 4550 4050
+Connection ~ 3500 4050
+Wire Wire Line
+	4550 3900 2750 3900
+Connection ~ 2750 4050
 $EndSCHEMATC
