File: jk330-8-CPU/ELECTRONICAL_MAIN_BOARD_32.kicad_pcb (KiCad board)
At the start: 2 copper layers, 85 parts, among them J1001 RJ12, J1002 SIL1, J1003 SIL1, J1004 SIL1, J1005 SIL1, J1006 SIL1, J1007 SIL1, K1001 CONN_3, K1002 CONN_3, K1003 CONN_3, K1004 CONN_3, K1005 CONN_3, K1006 CONN_3, K1007 CONN_3, K1008 CONN_3, K1009 CONN_3, K1010 CONN_3, K1011 CONN_3, K1012 CONN_3, K1013 CONN_3, K1014 CONN_3, K1015 CONN_3, K1016 CONN_3, K1017 CONN_3, K1018 CONN_3, K1019 CONN_3, K1020 CONN_3, P1001 CONN_5, P1002 CONN_4, P1003 CONN_4, P1004 CONN_4, P1005 CAVALIER2, P1006 CONN_10X2, P1007 CONN_5X2, P1008 CONN_5X2, P1009 CONN_5X2, Q4001 BSS123, Q4002 BSS123, SW1001 SW_PUSH_SMALL, U2001 74C922, U3001 PIC32MX795F512H, X3001 32.768khz

Commit message: LCD HD77480
Parts:
- removed the J1001 at (105.7, 35.1)
- removed the J1002 at (130.0, 172.6)
- removed the J1003 at (129.9, 25.8)
- removed the J1004 at (130.2, 119.6)
- removed the J1005 at (29.0, 185.2)
- removed the J1006 at (28.3, 25.8)
- removed the J1007 at (28.2, 119.0)
- removed the K1001 at (127.4, 63.1)
- removed the K1002 at (127.4, 69.5)
- removed the K1003 at (127.4, 75.8)
- removed the K1004 at (127.4, 82.2)
- removed the K1005 at (127.4, 88.5)
- removed the K1006 at (127.4, 94.9)
- removed the K1007 at (127.4, 101.2)
- removed the K1008 at (30.7, 38.7)
- removed the K1009 at (30.7, 45.1)
- removed the K1010 at (30.7, 51.4)
- removed the K1011 at (127.5, 129.8)
- removed the K1012 at (127.5, 136.1)
- removed the K1013 at (127.5, 142.5)
- removed the K1014 at (127.5, 181.4)
- removed the K1015 at (127.5, 148.8)
- removed the K1016 at (121.2, 181.4)
- removed the K1017 at (114.8, 181.4)
- removed the K1018 at (30.7, 57.8)
- removed the K1019 at (30.7, 64.1)
- removed the K1020 at (31.0, 107.2)
- removed the P1001 at (92.3, 25.1)
- removed the P1005 at (53.6, 176.9)
- removed the P1006 at (71.6, 184.4)
- removed the P1007 at (28.4, 86.1)
- removed the P1008 at (28.4, 140.5)
- removed the P1009 at (28.2, 167.1)
- removed the Q4001 at (96.6, 89.3)
- removed the Q4002 at (96.8, 83.3)
- removed the R4001 at (83.8, 169.4)
- removed the RVAR4001 at (100.5, 184.3)
- removed the SW1001 at (122.3, 24.9)
- removed the U2001 at (52.6, 81.0)
- removed the U3001 at (93.7, 105.9)
- removed the X3001 at (90.0, 153.9)
- added C2001: 100n, SM0603_Capa, F.Cu at (171.2, 145.0)
- added C2002: 1U, SM1206, F.Cu at (178.1, 143.8)
- added C2003: 100n, SM0603_Capa, F.Cu at (218.1, 104.6)
- added C2004: 100n, SM0603_Capa, B.Cu at (98.8, 152.1)
- added C2005: 100n, SM0603_Capa, F.Cu at (176.4, 117.3)
- added C3001: 22p, SM1206, B.Cu at (99.2, 100.2)
- added C3002: 22p, SM1206, B.Cu at (99.2, 90.0)
- added C4001: 100n, SM0603_Capa, F.Cu at (88.8, 110.6)
- added C4002: 100n, SM0603_Capa, F.Cu at (88.8, 121.2)
- added C4003: 100n, SM0603_Capa, F.Cu at (176.4, 106.3)
- added C4004: 100n, SM0603_Capa, F.Cu at (212.6, 133.1)
- added C4005: 100n, SM0603_Capa, F.Cu at (209.3, 108.0)
- added C4006: 100n, SM0603_Capa, F.Cu at (83.4, 121.2)
- added C4007: 100n, SM0603_Capa, B.Cu at (150.6, 134.1)
- added C4008: 100n, SM0603_Capa, F.Cu at (83.3, 110.6)
- added C4009: 100n, SM0603_Capa, F.Cu at (213.1, 141.4)
- added C4010: 100n, SM0603_Capa, B.Cu at (171.3, 133.6)
- added D1001: LED, SM0603, F.Cu at (211.7, 101.5)
- added D1002: LED, SM0603, F.Cu at (211.7, 98.9)
- added D1003: LED, SM0603, F.Cu at (211.7, 96.4)
- added D1004: LED, SM0603, F.Cu at (211.7, 93.9)
- added D2001: DIODE, SM0805, F.Cu at (104.6, 138.7)
- added D2002: DIODE, SM0805, F.Cu at (106.7, 138.7)
- added D2003: DIODE, SM0805, F.Cu at (108.7, 138.7)
- added D2004: DIODE, SM0805, F.Cu at (110.7, 138.7)
- added D2005: DIODE, SM0805, F.Cu at (86.9, 139.7)
- added D2006: DIODE, SM0805, F.Cu at (88.9, 139.7)
- added D2007: DIODE, SM0805, F.Cu at (90.9, 139.7)
- added D2008: DIODE, SM0805, F.Cu at (93.0, 139.7)
- added D4001: LED, SM0603, F.Cu at (84.7, 102.4)
- added R1001: 3.3k, SM0603_Resistor, F.Cu at (214.9, 101.5)
- added R1002: 1k, SM0603_Resistor, F.Cu at (214.9, 98.9)
- added R1003: 1k, SM0603_Resistor, F.Cu at (214.9, 96.4)
- added R1004: 330, SM0603_Resistor, F.Cu at (214.9, 93.9)
- added R1005: 0, SM0603_Resistor, F.Cu at (78.1, 103.1)
- added R2001: 10k, SM0603_Resistor, B.Cu at (134.1, 134.1)
- added R2002: 1k, SM0603_Resistor, B.Cu at (178.6, 159.0)
- added R2003: 1k, SM0603_Resistor, B.Cu at (178.6, 156.5)
- added R2004: 1k, SM0603_Resistor, B.Cu at (124.0, 160.7)
- added R2005: 1k, SM0603_Resistor, B.Cu at (124.0, 158.9)
- added R2006: 1k, SM0603_Resistor, B.Cu at (96.8, 159.3)
- added R2007: 1k, SM0603_Resistor, B.Cu at (96.8, 156.7)
- added R2008: 1k, SM0603_Resistor, B.Cu at (150.9, 157.7)
- added R2009: 1k, SM0603_Resistor, B.Cu at (150.9, 160.3)
- added R2010: 10k, SM0603_Resistor, F.Cu at (113.3, 146.8)
- added R2011: 10k, SM0603_Resistor, F.Cu at (113.3, 145.0)
- added R2012: 10k, SM0603_Resistor, F.Cu at (113.3, 143.3)
- added R2013: 10k, SM0603_Resistor, F.Cu at (113.3, 141.5)
- added R2014: 10k, SM0603_Resistor, F.Cu at (80.0, 141.0)
- added R2015: 10k, SM0603_Resistor, F.Cu at (80.0, 142.7)
- added R2016: 10k, SM0603_Resistor, F.Cu at (80.0, 144.5)
- added R2017: 10k, SM0603_Resistor, F.Cu at (80.0, 146.3)
- added R4002: 10k, SM0603_Resistor, F.Cu at (161.8, 85.1)
- added R4003: 10k, SM0603_Resistor, F.Cu at (164.1, 85.1)
- added R4004: 2.1k, SM0603_Resistor, F.Cu at (209.3, 114.0)
- added R4005: 2.1k, SM0603_Resistor, F.Cu at (209.3, 111.0)
- added R4006: 200k, SM1206, F.Cu at (217.2, 107.4)
- added R4007: 2.1k, SM0603_Resistor, F.Cu at (218.9, 111.0)
- added R4008: 2.1k, SM0603_Resistor, F.Cu at (218.9, 114.0)
- added U2002: PCF8574T, SO16W, B.Cu at (142.5, 138.4)
- added U2003: 74LS20, SO14N, B.Cu at (98.8, 145.3)
- added U4001: 74LVCC3245, SSOP24, B.Cu at (86.1, 110.4)
- added U4002: 74LVCC3245, SSOP24, F.Cu at (170.7, 111.8)
- added U4003: 74LVCC3245, SSOP24, B.Cu at (86.1, 121.4)
- added U4004: 74LVCC3245, SSOP24, F.Cu at (207.3, 138.4)
- added U4005: PCA9306, VSSOP-8, F.Cu at (213.9, 111.8)
- J1001: footprint RJ12_E -> RJ12
- P1002, P1003: footprint SIL-3 -> KK-4
- P1004: footprint SIL-3 -> KK-4; moved to F.Cu
- P1007, P1008, P1009: footprint he10-10d -> he10-10D
- moved K1014 206.3 mm to (70.9, 58.7), turned to 180 degrees
- moved K1016 201.1 mm to (70.9, 65.0), turned to 180 degrees
- moved J1002 198.8 mm to (79.6, 56.1), turned to 180 degrees
- moved K1017 196.1 mm to (70.9, 71.4), turned to 180 degrees
- moved RVAR4001 189.6 mm to (67.9, 85.7), turned to 180 degrees
- moved P1006 175.3 mm to (67.8, 114.6), turned to 270 degrees
- moved K1015 171.7 mm to (103.4, 58.7), turned to 90 degrees
- moved J1005 171.4 mm to (67.1, 157.2), turned to 180 degrees
- moved P1004 170.0 mm to (227.1, 107.7), turned to 270 degrees
- moved K1013 165.6 mm to (109.7, 58.7), turned to 90 degrees
- moved R4001 160.7 mm to (82.8, 102.4), turned to 270 degrees
- moved P1005 160.1 mm to (75.3, 132.6), turned to 270 degrees
- moved K1012 159.8 mm to (116.1, 58.7), turned to 90 degrees
- moved K1011 154.2 mm to (122.4, 58.7), turned to 90 degrees
- moved J1004 149.3 mm to (132.6, 56.0), turned to 180 degrees
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Routing:
- net GND: track 2542.1 -> 1271.0 mm, vias 54 -> 27
- net +5VD: track 1340.1 -> 670.1 mm, vias 26 -> 13
- net +3.3V: track 1113.8 -> 556.9 mm, vias 32 -> 16
- net /PIC32/RST: track 564.3 -> 282.1 mm, vias 4 -> 2
- net /5vto3v3/U2TX-5V: track 394.7 -> 197.4 mm, vias 8 -> 4
- net /5vto3v3/U3TX-5V: track 347.3 -> 173.7 mm, vias 4 -> 2
- net /5vto3v3/OC1: track 331.4 -> 165.7 mm, vias 2 -> 1
- net /INTERFACE BOARD/X1: track 323.0 -> 161.5 mm, vias 8 -> 4
- net /INTERFACE BOARD/X2: track 315.1 -> 157.6 mm, vias 8 -> 4
- net /5vto3v3/SCL1: track 289.9 -> 145.0 mm, vias 6 -> 3
- net /5vto3v3/SDA1: track 286.2 -> 143.1 mm, vias 6 -> 3
- net /INTERFACE BOARD/X3: track 277.5 -> 138.8 mm, vias 8 -> 4
- net /5vto3v3/OC2: track 268.9 -> 134.4 mm, vias 2 -> 1
- net /5vto3v3//BKOE: track 268.7 -> 134.3 mm, vias 8 -> 4
- net /INTERFACE BOARD/Y4: track 261.0 -> 130.5 mm, vias 8 -> 4
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