File: Chargeur-Max712/CHARGEUR.sch (KiCad schematic (older format))
At the start: 17 parts

Commit message: MAJ
Parts:
- C? (x2): value C -> 10n
- C?: value C -> 1U
- D?: value DIODE -> 1N4001
- R?: value R -> 150
- R?: value R -> 0.68
- R?: value R -> 22k
- R?: value R -> 68k
- R?: value R -> 680
- R?: value 1k -> 470
Other:
- note added: "LOAD"
Changed lines of the file:
@@
 Sheet 1 1
 Title ""
-Date "7 oct 2013"
+Date "29 dec 2013"
 Rev ""
 Comp ""
@@
 U 1 1 52530D25
 P 6100 2450
-F 0 "Q?" H 6100 2300 60  0000 R CNN
-F 1 "PNP" H 6100 2600 60  0000 R CNN
+F 0 "Q?" V 6350 2600 60  0000 R CNN
+F 1 "PNP" V 6350 2400 60  0000 R CNN
 F 2 "~" H 6100 2450 60  0000 C CNN
 F 3 "~" H 6100 2450 60  0000 C CNN
@@
 U 1 1 52531D7D
 P 5750 2700
-F 0 "R?" V 5700 2800 50  0000 C CNN
-F 1 "R" V 5800 2800 50  0000 C CNN
+F 0 "R?" V 5700 2600 50  0000 C CNN
+F 1 "150" V 5800 2600 50  0000 C CNN
 F 2 "~" H 5750 2700 60  0000 C CNN
 F 3 "~" H 5750 2700 60  0000 C CNN
@@
 U 1 1 52531D96
 P 5550 2600
-F 0 "C?" H 5600 2700 50  0000 L CNN
-F 1 "C" H 5600 2500 50  0000 L CNN
+F 0 "C?" H 5450 2700 50  0000 L CNN
+F 1 "10n" H 5400 2500 50  0000 L CNN
 F 2 "~" H 5550 2600 60  0000 C CNN
 F 3 "~" H 5550 2600 60  0000 C CNN
@@
 P 6550 2900
 F 0 "D?" H 6550 3000 40  0000 C CNN
-F 1 "DIODE" H 6550 2800 40  0000 C CNN
+F 1 "1N4001" H 6550 2800 40  0000 C CNN
 F 2 "~" H 6550 2900 60  0000 C CNN
 F 3 "~" H 6550 2900 60  0000 C CNN
@@
 U 1 1 52532AE8
 P 5900 4600
-F 0 "R?" V 5850 4700 50  0000 C CNN
-F 1 "R" V 5950 4700 50  0000 C CNN
+F 0 "R?" V 5850 4500 50  0000 C CNN
+F 1 "0.68" V 5950 4500 50  0000 C CNN
 F 2 "~" H 5900 4600 60  0000 C CNN
 F 3 "~" H 5900 4600 60  0000 C CNN
@@
 P 5300 5050
 F 0 "C?" H 5350 5150 50  0000 L CNN
-F 1 "C" H 5350 4950 50  0000 L CNN
+F 1 "10n" H 5350 4950 50  0000 L CNN
 F 2 "~" H 5300 5050 60  0000 C CNN
 F 3 "~" H 5300 5050 60  0000 C CNN
@@
 U 1 1 52532ED8
 P 4750 4950
-F 0 "R?" V 4700 5050 50  0000 C CNN
-F 1 "R" V 4800 5050 50  0000 C CNN
+F 0 "R?" V 4700 4850 50  0000 C CNN
+F 1 "22k" V 4800 4850 50  0000 C CNN
 F 2 "~" H 4750 4950 60  0000 C CNN
 F 3 "~" H 4750 4950 60  0000 C CNN
@@
 U 1 1 52532F33
 P 4650 4200
-F 0 "R?" V 4600 4300 50  0000 C CNN
-F 1 "R" V 4700 4300 50  0000 C CNN
+F 0 "R?" V 4600 4100 50  0000 C CNN
+F 1 "68k" V 4700 4100 50  0000 C CNN
 F 2 "~" H 4650 4200 60  0000 C CNN
 F 3 "~" H 4650 4200 60  0000 C CNN
@@
 U 1 1 5253301A
 P 4100 2500
-F 0 "R?" V 4050 2600 50  0000 C CNN
-F 1 "R" V 4150 2600 50  0000 C CNN
+F 0 "R?" V 4050 2400 50  0000 C CNN
+F 1 "680" V 4150 2400 50  0000 C CNN
 F 2 "~" H 4100 2500 60  0000 C CNN
 F 3 "~" H 4100 2500 60  0000 C CNN
@@
 P 4100 5050
 F 0 "C?" H 4150 5150 50  0000 L CNN
-F 1 "C" H 4150 4950 50  0000 L CNN
+F 1 "1U" H 4150 4950 50  0000 L CNN
 F 2 "~" H 4100 5050 60  0000 C CNN
 F 3 "~" H 4100 5050 60  0000 C CNN
@@
 U 1 1 525333D7
 P 4400 2900
-F 0 "R?" V 4350 3000 50  0000 C CNN
-F 1 "1k" V 4450 3000 50  0000 C CNN
+F 0 "R?" V 4350 2800 50  0000 C CNN
+F 1 "470" V 4450 2800 50  0000 C CNN
 F 2 "~" H 4400 2900 60  0000 C CNN
 F 3 "~" H 4400 2900 60  0000 C CNN
@@
 Wire Wire Line
 	5850 3500 5700 3500
+Text Notes 7350 5200 0    60   ~ 12
+LOAD
 $EndSCHEMATC
