File: INTEFACE SON/INTERFACE SON.sch (KiCad schematic (older format))
At the start: 21 parts, among them IC1 PC817, J1 RJ12, J2 JACK_MONO_F, J3 JACK_MONO_F, J4 DB9, K1 CONN_2, P1 CAVALIER, P2 CAVALIER, P3 CAVALIER, T1 TRANSFO2, T2 TRANSFO2

Commit message: MAJ???
Parts:
- IC1: symbol PC817 -> PC817-RESCUE-INTERFACE_SON
Changed lines of the file:
@@
 EESchema Schematic File Version 2
+LIBS:INTERFACE SON-rescue
 LIBS:power
-LIBS:CEN-SCHEMA
 LIBS:analog_switches
 LIBS:opto
+LIBS:CEN-SCHEMA
 LIBS:INTERFACE SON-cache
-EELAYER 27 0
+EELAYER 25 0
 EELAYER END
 $Descr A4 11693 8268
@@
 Connection ~ 6450 4700
 $Comp
-L PC817 IC1
+L PC817-RESCUE-INTERFACE_SON IC1
 U 1 1 532DDD33
 P 5550 6000
